File: Circuit_layout/isolators.sch (KiCad schematic (older format))
At the start: 29 parts

Commit message: KiCad BOM
Parts:
- gave numbers to parts that had none: 28
Connections:
- net Throttle_HV: now also U16.8; no longer U16.1
- net V_Measure: now also U16.7; no longer U16.1
- net at R60.1, R65.2: now also U16.9 (-); no longer U16.2 (-)
- net at R59.1, R62.1: now also U16.10 (+); no longer U16.3 (+)
- net at R53.1, R56.2: now also U16.6 (-); no longer U16.2 (-)
- net at R54.1, R55.2: now also U16.5 (+); no longer U16.3 (+)
Changed lines of the file:
@@
 EESchema Schematic File Version 2
 LIBS:Circuit_layout-rescue
+LIBS:TSI_KiCad_Lib
 LIBS:TSI_HV_Isolater-cache
 LIBS:74xgxx
@@
 encoding utf-8
 Sheet 7 7
-Title ""
+Title "Tractive System Interface"
 Date ""
-Rev ""
-Comp ""
-Comment1 ""
-Comment2 ""
+Rev "0.0"
+Comp "Lafayette College"
+Comment1 "Spring 2017"
+Comment2 "Jack Plumb and Adam Ness"
 Comment3 ""
-Comment4 ""
+Comment4 "DEVELOPMENT ONLY"
 $EndDescr
 $Comp
-L ACPL-C870 U?
+L ACPL-C870 U17
 U 1 1 58B06069
 P 5450 1250
-F 0 "U?" H 5450 1450 60  0000 C CNN
+F 0 "U17" H 5450 1450 60  0000 C CNN
 F 1 "ACPL-C870" H 5450 1350 60  0000 C CNN
 F 2 "" H 5450 1450 60  0000 C CNN
@@
 	4950 1900 4950 1600
 $Comp
-L MCP6004 U?
-U 1 1 58B06078
+L MCP6004 U16
+U 3 1 58B06078
 P 7300 1550
-F 0 "U?" H 7350 1750 50  0000 C CNN
+F 0 "U16" H 7350 1750 50  0000 C CNN
 F 1 "MCP6004" H 7450 1350 50  0000 C CNN
 F 2 "" H 7250 1650 50  0000 C CNN
 F 3 "" H 7350 1750 50  0000 C CNN
-	1    7300 1550
+	3    7300 1550
 	1    0    0    -1
 $EndComp
@@
 	7600 1550 7800 1550
 $Comp
-L C C?
+L C C26
 U 1 1 58B060A1
 P 6100 1950
-F 0 "C?" H 6125 2050 50  0000 L CNN
+F 0 "C26" H 6125 2050 50  0000 L CNN
 F 1 "0.1u" H 6125 1850 50  0000 L CNN
 F 2 "" H 6138 1800 50  0000 C CNN
@@
 $EndComp
 $Comp
-L C C?
+L C C27
 U 1 1 58B060A8
 P 6250 1150
-F 0 "C?" H 6275 1250 50  0000 L CNN
+F 0 "C27" H 6275 1250 50  0000 L CNN
 F 1 "0.1u" H 6275 1050 50  0000 L CNN
 F 2 "" H 6288 1000 50  0000 C CNN
@@
 Throttle
 $Comp
-L ACPL-C870 U?
+L ACPL-C870 U18
 U 1 1 58B06729
 P 5450 3100
-F 0 "U?" H 5450 3300 60  0000 C CNN
+F 0 "U18" H 5450 3300 60  0000 C CNN
 F 1 "ACPL-C870" H 5450 3200 60  0000 C CNN
 F 2 "" H 5450 3300 60  0000 C CNN
@@
 $EndComp
 $Comp
-L MCP6004 U?
-U 1 1 58B06732
+L MCP6004 U16
+U 2 1 58B06732
 P 3600 3400
-F 0 "U?" H 3650 3600 50  0000 C CNN
+F 0 "U16" H 3650 3600 50  0000 C CNN
 F 1 "MCP6004" H 3750 3200 50  0000 C CNN
 F 2 "" H 3550 3500 50  0000 C CNN
 F 3 "" H 3650 3600 50  0000 C CNN
-	1    3600 3400
+	2    3600 3400
 	-1   0    0    -1
 $EndComp
@@
 	2600 3400 3300 3400
 $Comp
-L C C?
+L C C25
 U 1 1 58B06756
 P 4800 3800
-F 0 "C?" H 4825 3900 50  0000 L CNN
+F 0 "C25" H 4825 3900 50  0000 L CNN
 F 1 "0.1u" H 4825 3700 50  0000 L CNN
 F 2 "" H 4838 3650 50  0000 C CNN
@@
 $EndComp
 $Comp
-L C C?
+L C C24
 U 1 1 58B0675C
 P 4650 3000
-F 0 "C?" H 4675 3100 50  0000 L CNN
+F 0 "C24" H 4675 3100 50  0000 L CNN
 F 1 "0.1u" H 4675 2900 50  0000 L CNN
 F 2 "" H 4688 2850 50  0000 C CNN
@@
 Voltage Measurement
 $Comp
-L C C?
+L C C28
 U 1 1 58B086CD
 P 6400 3500
-F 0 "C?" H 6425 3600 50  0000 L CNN
+F 0 "C28" H 6425 3600 50  0000 L CNN
 F 1 "DNP" H 6425 3400 50  0000 L CNN
 F 2 "Capacitors_SMD:C_0805_HandSoldering" H 6438 3350 50  0001 C CNN
@@
 	3250 3950 3500 3950
 $Comp
-L +5V #PWR?
+L +5V #PWR088
 U 1 1 58B246C4
 P 4650 2700
-F 0 "#PWR?" H 4650 2550 50  0001 C CNN
+F 0 "#PWR088" H 4650 2550 50  0001 C CNN
 F 1 "+5V" H 4650 2840 50  0000 C CNN
 F 2 "" H 4650 2700 50  0000 C CNN
@@
 $EndComp
 $Comp
-L +5V #PWR?
+L +5V #PWR089
 U 1 1 58B24710
 P 4950 2900
-F 0 "#PWR?" H 4950 2750 50  0001 C CNN
+F 0 "#PWR089" H 4950 2750 50  0001 C CNN
 F 1 "+5V" H 4950 3040 50  0000 C CNN
 F 2 "" H 4950 2900 50  0000 C CNN
@@
 $EndComp
 $Comp
-L +5V #PWR?
+L +5V #PWR090
 U 1 1 58B2475C
 P 3700 3100
-F 0 "#PWR?" H 3700 2950 50  0001 C CNN
+F 0 "#PWR090" H 3700 2950 50  0001 C CNN
 F 1 "+5V" H 3700 3240 50  0000 C CNN
 F 2 "" H 3700 3100 50  0000 C CNN
@@
 $EndComp
 $Comp
-L GND #PWR?
+L GND #PWR091
 U 1 1 58B247A8
 P 3700 3700
-F 0 "#PWR?" H 3700 3450 50  0001 C CNN
+F 0 "#PWR091" H 3700 3450 50  0001 C CNN
 F 1 "GND" H 3700 3550 50  0000 C CNN
 F 2 "" H 3700 3700 50  0000 C CNN
@@
 $EndComp
 $Comp
-L GND #PWR?
+L GND #PWR092
 U 1 1 58B2480E
 P 4800 4100
-F 0 "#PWR?" H 4800 3850 50  0001 C CNN
+F 0 "#PWR092" H 4800 3850 50  0001 C CNN
 F 1 "GND" H 4800 3950 50  0000 C CNN
 F 2 "" H 4800 4100 50  0000 C CNN
@@
 	4650 1900 4950 1900
 $Comp
-L GND #PWR?
+L GND #PWR093
 U 1 1 58B25770
 P 4650 2000
-F 0 "#PWR?" H 4650 1750 50  0001 C CNN
+F 0 "#PWR093" H 4650 1750 50  0001 C CNN
 F 1 "GND" H 4650 1850 50  0000 C CNN
 F 2 "" H 4650 2000 50  0000 C CNN
@@
 $EndComp
 $Comp
-L +5V #PWR?
+L +5V #PWR094
 U 1 1 58B257CF
 P 4950 1050
-F 0 "#PWR?" H 4950 900 50  0001 C CNN
+F 0 "#PWR094" H 4950 900 50  0001 C CNN
 F 1 "+5V" H 4950 1190 50  0000 C CNN
 F 2 "" H 4950 1050 50  0000 C CNN
@@
 HV-
 $Comp
-L C C?
+L C C23
 U 1 1 58B52862
 P 1200 1550
-F 0 "C?" H 1225 1650 50  0000 L CNN
+F 0 "C23" H 1225 1650 50  0000 L CNN
 F 1 "0.1u" H 1225 1450 50  0000 L CNN
 F 2 "" H 1238 1400 50  0000 C CNN
@@
 HV-
 $Comp
-L R R?
+L R R64
 U 1 1 58B6DFCC
 P 7100 3700
-F 0 "R?" V 7180 3700 50  0000 C CNN
+F 0 "R64" V 7180 3700 50  0000 C CNN
 F 1 "10k" V 7100 3700 50  0000 C CNN
 F 2 "Resistors_SMD:R_0805_HandSoldering" V 7030 3700 50  0001 C CNN
@@
 $EndComp
 $Comp
-L R R?
+L R R61
 U 1 1 58B6F112
 P 6700 3500
-F 0 "R?" V 6780 3500 50  0000 C CNN
+F 0 "R61" V 6780 3500 50  0000 C CNN
 F 1 "1k" V 6700 3500 50  0000 C CNN
 F 2 "Resistors_SMD:R_0805_HandSoldering" V 6630 3500 50  0001 C CNN
@@
 $EndComp
 $Comp
-L R R?
+L R R67
 U 1 1 58B6FA2F
 P 7600 3700
-F 0 "R?" V 7680 3700 50  0000 C CNN
+F 0 "R67" V 7680 3700 50  0000 C CNN
 F 1 "10k" V 7600 3700 50  0000 C CNN
 F 2 "Resistors_SMD:R_0805_HandSoldering" V 7530 3700 50  0001 C CNN
@@
 $EndComp
 $Comp
-L R R?
+L R R69
 U 1 1 58B6FAB1
 P 8100 3700
-F 0 "R?" V 8180 3700 50  0000 C CNN
+F 0 "R69" V 8180 3700 50  0000 C CNN
 F 1 "10k" V 8100 3700 50  0000 C CNN
 F 2 "Resistors_SMD:R_0805_HandSoldering" V 8030 3700 50  0001 C CNN
@@
 $EndComp
 $Comp
-L R R?
+L R R71
 U 1 1 58B6FB30
 P 8600 3700
-F 0 "R?" V 8680 3700 50  0000 C CNN
+F 0 "R71" V 8680 3700 50  0000 C CNN
 F 1 "10k" V 8600 3700 50  0000 C CNN
 F 2 "Resistors_SMD:R_0805_HandSoldering" V 8530 3700 50  0001 C CNN
@@
 $EndComp
 $Comp
-L R R?
+L R R68
 U 1 1 58B6FBB6
 P 8100 3300
-F 0 "R?" V 8180 3300 50  0000 C CNN
+F 0 "R68" V 8180 3300 50  0000 C CNN
 F 1 "10k" V 8100 3300 50  0000 C CNN
 F 2 "Resistors_SMD:R_0805_HandSoldering" V 8030 3300 50  0001 C CNN
@@
 $EndComp
 $Comp
-L R R?
+L R R70
 U 1 1 58B6FCAC
 P 8600 3300
-F 0 "R?" V 8680 3300 50  0000 C CNN
+F 0 "R70" V 8680 3300 50  0000 C CNN
 F 1 "10k" V 8600 3300 50  0000 C CNN
 F 2 "Resistors_SMD:R_0805_HandSoldering" V 8530 3300 50  0001 C CNN
@@
 $EndComp
 $Comp
-L R R?
+L R R66
 U 1 1 58B6FD36
 P 7600 3300
-F 0 "R?" V 7680 3300 50  0000 C CNN
+F 0 "R66" V 7680 3300 50  0000 C CNN
 F 1 "10k" V 7600 3300 50  0000 C CNN
 F 2 "Resistors_SMD:R_0805_HandSoldering" V 7530 3300 50  0001 C CNN
@@
 $EndComp
 $Comp
-L R R?
+L R R63
 U 1 1 58B6FDD3
 P 7100 3300
-F 0 "R?" V 7180 3300 50  0000 C CNN
+F 0 "R63" V 7180 3300 50  0000 C CNN
 F 1 "10k" V 7100 3300 50  0000 C CNN
 F 2 "Resistors_SMD:R_0805_HandSoldering" V 7030 3300 50  0001 C CNN
@@
 $EndComp
 $Comp
-L R R?
+L R R53
 U 1 1 58B70343
 P 3650 3950
-F 0 "R?" V 3730 3950 50  0000 C CNN
+F 0 "R53" V 3730 3950 50  0000 C CNN
 F 1 "4.99k" V 3650 3950 50  0000 C CNN
 F 2 "Resistors_SMD:R_0805_HandSoldering" V 3580 3950 50  0001 C CNN
@@
 $EndComp
 $Comp
-L R R?
+L R R54
 U 1 1 58B703E2
 P 4000 3000
-F 0 "R?" V 4080 3000 50  0000 C CNN
+F 0 "R54" V 4080 3000 50  0000 C CNN
 F 1 "4.99k" V 4000 3000 50  0000 C CNN
 F 2 "Resistors_SMD:R_0805_HandSoldering" V 3930 3000 50  0001 C CNN
@@
 $EndComp
 $Comp
-L R R?
+L R R56
 U 1 1 58B704D7
 P 4300 3500
-F 0 "R?" V 4380 3500 50  0000 C CNN
+F 0 "R56" V 4380 3500 50  0000 C CNN
 F 1 "2k" V 4300 3500 50  0000 C CNN
 F 2 "Resistors_SMD:R_0805_HandSoldering" V 4230 3500 50  0001 C CNN
@@
 $EndComp
 $Comp
-L R R?
+L R R55
 U 1 1 58B70594
 P 4300 3300
-F 0 "R?" V 4380 3300 50  0000 C CNN
+F 0 "R55" V 4380 3300 50  0000 C CNN
 F 1 "2k" V 4300 3300 50  0000 C CNN
 F 2 "Resistors_SMD:R_0805_HandSoldering" V 4230 3300 50  0001 C CNN
@@
 $EndComp
 $Comp
-L R R?
+L R R57
 U 1 1 58B7068E
 P 4350 1450
-F 0 "R?" V 4430 1450 50  0000 C CNN
+F 0 "R57" V 4430 1450 50  0000 C CNN
 F 1 "3k" V 4350 1450 50  0000 C CNN
 F 2 "Resistors_SMD:R_0805_HandSoldering" V 4280 1450 50  0001 C CNN
@@
 $EndComp
 $Comp
-L R R?
+L R R58
 U 1 1 58B70843
 P 4650 1700
-F 0 "R?" V 4730 1700 50  0000 C CNN
+F 0 "R58" V 4730 1700 50  0000 C CNN
 F 1 "2k" V 4650 1700 50  0000 C CNN
 F 2 "Resistors_SMD:R_0805_HandSoldering" V 4580 1700 50  0001 C CNN
@@
 $EndComp
 $Comp
-L R R?
+L R R59
 U 1 1 58B70974
 P 6600 1450
-F 0 "R?" V 6680 1450 50  0000 C CNN
+F 0 "R59" V 6680 1450 50  0000 C CNN
 F 1 "2k" V 6600 1450 50  0000 C CNN
 F 2 "Resistors_SMD:R_0805_HandSoldering" V 6530 1450 50  0001 C CNN
@@
 $EndComp
 $Comp
-L R R?
+L R R60
 U 1 1 58B70AF9
 P 6600 1650
-F 0 "R?" V 6680 1650 50  0000 C CNN
+F 0 "R60" V 6680 1650 50  0000 C CNN
 F 1 "2k" V 6600 1650 50  0000 C CNN
 F 2 "Resistors_SMD:R_0805_HandSoldering" V 6530 1650 50  0001 C CNN
@@
 $EndComp
 $Comp
-L R R?
+L R R65
 U 1 1 58B70BD4
 P 7250 2000
-F 0 "R?" V 7330 2000 50  0000 C CNN
+F 0 "R65" V 7330 2000 50  0000 C CNN
 F 1 "4.99k" V 7250 2000 50  0000 C CNN
 F 2 "Resistors_SMD:R_0805_HandSoldering" V 7180 2000 50  0001 C CNN
@@
 $EndComp
 $Comp
-L R R?
+L R R62
 U 1 1 58B70CB0
 P 6900 1150
-F 0 "R?" V 6980 1150 50  0000 C CNN
+F 0 "R62" V 6980 1150 50  0000 C CNN
 F 1 "4.99k" V 6900 1150 50  0000 C CNN
 F 2 "Resistors_SMD:R_0805_HandSoldering" V 6830 1150 50  0001 C CNN
