File: Circuit_layout/Circuit_layout.sch (KiCad schematic (older format))
At the start: 19 parts

Commit message: KiCad BOM
Parts:
- U9: renamed from U?; Field5 http://www.digikey.com/product-detail/en/toshiba-semiconduc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 -> (none); Man P/N TLP293(GB-TPL,E -> TLP293(GB-TPLE; URL (none) -> http://www.digikey.com/product-detail/en/toshiba-semiconduc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
- Y1: renamed from Y?; DigiKey P/N (none) -> 887-1741-1-ND; Field4 887-1741-1-ND -> (none); Man P/N (none) -> 7A-10.000MAAE-T
- gave numbers to parts that had none: 16
Connections:
- net IMD: now also U4.6 (-), U4.7; no longer U4.1, U4.2 (-)
- net at C4.2, R5.2: now also U4.5 (+); no longer U4.3 (+)
Changed lines of the file:
@@
 EESchema Schematic File Version 2
 LIBS:Circuit_layout-rescue
+LIBS:TSI_KiCad_Lib
 LIBS:TSI_HV_Isolater-cache
 LIBS:74xgxx
@@
 Comp "Lafayette College"
 Comment1 "Spring 2017"
-Comment2 "Jack Plumb"
+Comment2 "Jack Plumb and Adam Ness"
 Comment3 ""
 Comment4 "DEVELOPMENT ONLY"
@@
 $EndSheet
 $Comp
-L AT90CAN128-A U?
+L AT90CAN128-A U7
 U 1 1 58A74D86
 P 5250 3700
-F 0 "U?" H 4100 5600 50  0000 L BNN
+F 0 "U7" H 4100 5600 50  0000 L BNN
 F 1 "AT90CAN128-A" H 6400 1750 50  0000 R BNN
 F 2 "TQFP64" H 5300 3700 50  0000 C CNN
@@
 $EndComp
 $Comp
-L Crystal Y?
+L Crystal Y1
 U 1 1 58A86763
 P 2900 2550
-F 0 "Y?" H 2900 2700 50  0000 C CNN
+F 0 "Y1" H 2900 2700 50  0000 C CNN
 F 1 "10MHz" H 2900 2400 50  0000 C CNN
 F 2 "" H 2900 2550 50  0000 C CNN
 F 3 "" H 2900 2550 50  0000 C CNN
-F 4 "887-1741-1-ND" H 2900 2550 60  0001 C CNN "Field4"
+F 4 "887-1741-1-ND" H 2900 2550 60  0001 C CNN "DigiKey P/N"
 F 5 "http://www.digikey.com/product-search/en?pv7=2&k=7A-10.000MAAE-T&mnonly=0&newproducts=0&ColumnSort=0&page=1&quantity=0&ptm=0&fid=0&pageSize=25" H 2900 2550 60  0001 C CNN "URL"
+F 6 "7A-10.000MAAE-T" H 2900 2550 60  0001 C CNN "Man P/N"
 	1    2900 2550
 	1    0    0    -1
@@
 Connection ~ 3050 2550
 $Comp
-L C C?
+L C C5
 U 1 1 58A868A1
 P 2750 2900
-F 0 "C?" H 2775 3000 50  0000 L CNN
+F 0 "C5" H 2775 3000 50  0000 L CNN
 F 1 "10p" H 2775 2800 50  0000 L CNN
 F 2 "" H 2788 2750 50  0000 C CNN
@@
 $EndComp
 $Comp
-L C C?
+L C C6
 U 1 1 58A86A84
 P 3050 2900
-F 0 "C?" H 3075 3000 50  0000 L CNN
+F 0 "C6" H 3075 3000 50  0000 L CNN
 F 1 "10p" H 3075 2800 50  0000 L CNN
 F 2 "" H 3088 2750 50  0000 C CNN
@@
 $EndSheet
 $Sheet
-S 8300 1550 1750 950
+S 8200 2200 1750 950
 U 58ADE5BC
 F0 "Power System" 60
@@
 	700  3750 1350 3750
 $Comp
-L C C?
+L C C1
 U 1 1 58B0B5F8
 P 1150 3250
-F 0 "C?" H 1175 3350 50  0000 L CNN
+F 0 "C1" H 1175 3350 50  0000 L CNN
 F 1 "0.1u" H 1175 3150 50  0000 L CNN
 F 2 "Capacitors_SMD:C_0805_HandSoldering" H 1188 3100 50  0001 C CNN
@@
 I_Measure
 $Sheet
-S 8600 5300 1700 1250
+S 8200 5250 1700 1250
 U 58A289D2
 F0 "ThrottlePlausibility" 60
 F1 "ThrottlePlausibility.sch" 60
-F2 "GND" I L 8600 6450 60
-F3 "RTN_GLV" O L 8600 5700 60
-F4 "APPS1" O L 8600 5850 60
-F5 "APPS2" O L 8600 6000 60
-F6 "APPS1_10" O L 8600 5400 60
-F7 "APPS2_5" O L 8600 5550 60
-F8 "+12LV" I L 8600 6300 60
-F9 "Throttle_SEL" I R 10300 5700 60
-F10 "Throttle_uC" I R 10300 5550 60
-F11 "Throttle_LV" O R 10300 5400 60
-F12 "+5LV" I L 8600 6150 60
-F13 "BP" I R 10300 6150 60
-F14 "BRAKE_5" O R 10300 6450 60
-F15 "BP_uC" I R 10300 6300 60
+F2 "GND" I L 8200 6400 60
+F3 "RTN_GLV" O L 8200 5650 60
+F4 "APPS1" O L 8200 5800 60
+F5 "APPS2" O L 8200 5950 60
+F6 "APPS1_10" O L 8200 5350 60
+F7 "APPS2_5" O L 8200 5500 60
+F8 "+12LV" I L 8200 6250 60
+F9 "Throttle_SEL" I R 9900 5650 60
+F10 "Throttle_uC" I R 9900 5500 60
+F11 "Throttle_LV" O R 9900 5350 60
+F12 "+5LV" I L 8200 6100 60
+F13 "BP" I R 9900 6100 60
+F14 "BRAKE_5" O R 9900 6400 60
+F15 "BP_uC" I R 9900 6250 60
 $EndSheet
 Text Notes 1350 2900 0    99   ~ 0
 Current \nMeasurement
 $Comp
-L C C?
+L C C3
 U 1 1 58B21260
 P 1700 1500
-F 0 "C?" H 1725 1600 50  0000 L CNN
+F 0 "C3" H 1725 1600 50  0000 L CNN
 F 1 "0.47u" H 1725 1400 50  0000 L CNN
 F 2 "Capacitors_SMD:C_0805_HandSoldering" H 1738 1350 50  0001 C CNN
@@
 $EndComp
 $Comp
-L C C?
+L C C4
 U 1 1 58B21267
 P 2700 900
-F 0 "C?" H 2725 1000 50  0000 L CNN
+F 0 "C4" H 2725 1000 50  0000 L CNN
 F 1 "0.47u" H 2725 800 50  0000 L CNN
 F 2 "Capacitors_SMD:C_0805_HandSoldering" H 2738 750 50  0001 C CNN
@@
 Sallen-Key Filter\nIntended for 10Hz PWM\n2Hz fc - breadboarded - still osc
 $Comp
-L MCP6004 U?
-U 1 1 58B21292
+L MCP6004 U4
+U 2 1 58B21292
 P 2600 1350
-F 0 "U?" H 2650 1550 50  0000 C CNN
+F 0 "U4" H 2650 1550 50  0000 C CNN
 F 1 "MCP6004" H 2750 1150 50  0000 C CNN
 F 2 "" H 2550 1450 50  0000 C CNN
 F 3 "" H 2650 1550 50  0000 C CNN
-	1    2600 1350
+	2    2600 1350
 	1    0    0    -1
 $EndComp
@@
 IMD
 $Comp
-L MCP6004 U?
+L MCP6004 U4
 U 1 1 58B2253B
 P 2200 3650
-F 0 "U?" H 2250 3850 50  0000 C CNN
+F 0 "U4" H 2250 3850 50  0000 C CNN
 F 1 "MCP6004" H 2350 3450 50  0000 C CNN
 F 2 "" H 2150 3750 50  0000 C CNN
@@
 Spare_Blue
 $Comp
-L TLP291 U?
+L TLP291 U9
 U 1 1 58B3A5D9
 P 7050 1200
-F 0 "U?" H 6850 1400 50  0000 L CNN
+F 0 "U9" H 6850 1400 50  0000 L CNN
 F 1 "TLP293" H 7050 1400 50  0000 L CNN
 F 2 "SOP-4" H 6850 1000 50  0000 L CIN
 F 3 "" H 7050 1200 50  0000 L CNN
 F 4 "TLP293(GB-TPLECT-ND" H 7050 1200 60  0001 C CNN "DigiKey P/N"
-F 5 "http://www.digikey.com/product-detail/en/toshiba-semiconductor-and-storage/TLP293(GB-TPL,E/TLP293(GB-TPLECT-ND/4562965" H 7050 1200 60  0001 C CNN "Field5"
-F 6 "TLP293(GB-TPL,E" H 7050 1200 60  0001 C CNN "Man P/N"
+F 5 "http://www.digikey.com/product-detail/en/toshiba-semiconductor-and-storage/TLP293(GB-TPL,E/TLP293(GB-TPLECT-ND/4562965" H 7050 1200 60  0001 C CNN "URL"
+F 6 "TLP293(GB-TPLE" H 7050 1200 60  0001 C CNN "Man P/N"
 F 7 "http://www.digikey.com/product-detail/en/toshiba-semiconductor-and-storage/TLP291(GB-TP,SE/TLP291(GB-TPSECT-ND/4562949" H 7050 1200 60  0001 C CNN "TLP291"
 	1    7050 1200
@@
 AIRs-_in
 $Comp
-L R R?
+L R R7
 U 1 1 58B4C950
 P 6500 1100
-F 0 "R?" V 6580 1100 50  0000 C CNN
+F 0 "R7" V 6580 1100 50  0000 C CNN
 F 1 "1k" V 6500 1100 50  0000 C CNN
 F 2 "Resistors_SMD:R_0805_HandSoldering" V 6430 1100 50  0001 C CNN
@@
 $EndComp
 $Comp
-L +5V #PWR?
+L +5V #PWR04
 U 1 1 58B52706
 P 7800 950
-F 0 "#PWR?" H 7800 800 50  0001 C CNN
+F 0 "#PWR04" H 7800 800 50  0001 C CNN
 F 1 "+5V" H 7800 1090 50  0000 C CNN
 F 2 "" H 7800 950 50  0000 C CNN
@@
 $EndComp
 $Comp
-L R R?
+L R R9
 U 1 1 58B530A6
 P 7550 1100
-F 0 "R?" V 7630 1100 50  0000 C CNN
+F 0 "R9" V 7630 1100 50  0000 C CNN
 F 1 "1k" V 7550 1100 50  0000 C CNN
 F 2 "Resistors_SMD:R_0805_HandSoldering" V 7480 1100 50  0001 C CNN
@@
 Safety_Loop
 $Comp
-L GND #PWR?
+L GND #PWR05
 U 1 1 58B230AC
 P 2100 3950
-F 0 "#PWR?" H 2100 3700 50  0001 C CNN
+F 0 "#PWR05" H 2100 3700 50  0001 C CNN
 F 1 "GND" H 2100 3800 50  0000 C CNN
 F 2 "" H 2100 3950 50  0000 C CNN
@@
 	1150 4200 1150 4250
 $Comp
-L GND #PWR?
+L GND #PWR06
 U 1 1 58B23714
 P 1150 4250
-F 0 "#PWR?" H 1150 4000 50  0001 C CNN
+F 0 "#PWR06" H 1150 4000 50  0001 C CNN
 F 1 "GND" H 1150 4100 50  0000 C CNN
 F 2 "" H 1150 4250 50  0000 C CNN
@@
 $EndComp
 $Comp
-L GND #PWR?
+L GND #PWR07
 U 1 1 58B237F4
 P 1150 2950
-F 0 "#PWR?" H 1150 2700 50  0001 C CNN
+F 0 "#PWR07" H 1150 2700 50  0001 C CNN
 F 1 "GND" H 1150 2800 50  0000 C CNN
 F 2 "" H 1150 2950 50  0000 C CNN
@@
 $EndComp
 $Comp
-L +5V #PWR?
+L +5V #PWR08
 U 1 1 58B238C3
 P 2100 3350
-F 0 "#PWR?" H 2100 3200 50  0001 C CNN
+F 0 "#PWR08" H 2100 3200 50  0001 C CNN
 F 1 "+5V" H 2100 3490 50  0000 C CNN
 F 2 "" H 2100 3350 50  0000 C CNN
@@
 $EndComp
 $Comp
-L +5V #PWR?
+L +5V #PWR09
 U 1 1 58B25F48
 P 2500 700
-F 0 "#PWR?" H 2500 550 50  0001 C CNN
+F 0 "#PWR09" H 2500 550 50  0001 C CNN
 F 1 "+5V" H 2500 840 50  0000 C CNN
 F 2 "" H 2500 700 50  0000 C CNN
@@
 $EndComp
 $Comp
-L GND #PWR?
+L GND #PWR010
 U 1 1 58B26028
 P 2500 1900
-F 0 "#PWR?" H 2500 1650 50  0001 C CNN
+F 0 "#PWR010" H 2500 1650 50  0001 C CNN
 F 1 "GND" H 2500 1750 50  0000 C CNN
 F 2 "" H 2500 1900 50  0000 C CNN
@@
 IMD PWM LPF
 $Comp
-L C C?
+L C C2
 U 1 1 58B54F3B
 P 1150 4050
-F 0 "C?" H 1175 4150 50  0000 L CNN
+F 0 "C2" H 1175 4150 50  0000 L CNN
 F 1 "0.1u" H 1175 3950 50  0000 L CNN
 F 2 "Capacitors_SMD:C_0805_HandSoldering" H 1188 3900 50  0001 C CNN
@@
 $EndComp
 $Comp
-L R R?
+L R R1
 U 1 1 58B56CDA
 P 1400 1250
-F 0 "R?" V 1480 1250 50  0000 C CNN
+F 0 "R1" V 1480 1250 50  0000 C CNN
 F 1 "160k" V 1400 1250 50  0000 C CNN
 F 2 "Resistors_SMD:R_0805_HandSoldering" V 1330 1250 50  0001 C CNN
@@
 $EndComp
 $Comp
-L R R?
+L R R5
 U 1 1 58B66CC7
 P 2000 1250
-F 0 "R?" V 2080 1250 50  0000 C CNN
+F 0 "R5" V 2080 1250 50  0000 C CNN
 F 1 "160k" V 2000 1250 50  0000 C CNN
 F 2 "Resistors_SMD:R_0805_HandSoldering" V 1930 1250 50  0001 C CNN
@@
 $EndComp
 $Comp
-L R R?
+L R R2
 U 1 1 58B681E6
 P 1500 3550
-F 0 "R?" V 1580 3550 50  0000 C CNN
+F 0 "R2" V 1580 3550 50  0000 C CNN
 F 1 "1k" V 1500 3550 50  0000 C CNN
 F 2 "Resistors_SMD:R_0805_HandSoldering" V 1430 3550 50  0001 C CNN
@@
 $EndComp
 $Comp
-L R R?
+L R R3
 U 1 1 58B68338
 P 1500 3750
-F 0 "R?" V 1580 3750 50  0000 C CNN
+F 0 "R3" V 1580 3750 50  0000 C CNN
 F 1 "1k" V 1500 3750 50  0000 C CNN
 F 2 "Resistors_SMD:R_0805_HandSoldering" V 1430 3750 50  0001 C CNN
@@
 $EndComp
 $Comp
-L R R?
+L R R6
 U 1 1 58B68415
 P 2150 4250
-F 0 "R?" V 2230 4250 50  0000 C CNN
+F 0 "R6" V 2230 4250 50  0000 C CNN
 F 1 "1k" V 2150 4250 50  0000 C CNN
 F 2 "Resistors_SMD:R_0805_HandSoldering" V 2080 4250 50  0001 C CNN
@@
 $EndComp
 $Comp
-L R R?
+L R R4
 U 1 1 58B68515
 P 1800 3250
-F 0 "R?" V 1880 3250 50  0000 C CNN
+F 0 "R4" V 1880 3250 50  0000 C CNN
 F 1 "1k" V 1800 3250 50  0000 C CNN
 F 2 "Resistors_SMD:R_0805_HandSoldering" V 1730 3250 50  0001 C CNN

Commit message: finished adding footprints/info to all parts that I can
Parts:
- removed C1, C2: 0.1u, Capacitors_SMD:C_0805_HandSoldering, symbol C
- removed C4: 0.47u, Capacitors_SMD:C_0805_HandSoldering, symbol C
- removed C5: 10p, symbol C
- removed U4: MCP6004, symbol MCP6004
- added C? (x2): 0.1u, Capacitors_SMD:C_0805_HandSoldering, symbol C
- added C?: 0.47u, Capacitors_SMD:C_0805_HandSoldering, symbol C
- added C?: 10p, Capacitors_SMD:C_0805_HandSoldering, symbol C
- added U? (x2): MCP6004, Housings_SOIC:SOIC-14_3.9x8.7mm_Pitch1.27mm, symbol MCP6004
- C3: Digikey P/N (none) -> 399-8100-1-ND; Man P/N (none) -> C0805C474K5RACTU; URL (none) -> http://www.digikey.com/product-detail/en/kemet/C0805C474K5R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
- C6: footprint (none) -> Capacitors_SMD:C_0805_HandSoldering; Man P/N (none) -> C0805C100J5GACTU
- Y1: footprint (none) -> Crystals:Crystal_SMD_HC49-SD_HandSoldering; DigiKey P/N 887-1741-1-ND -> 535-9065-1-ND; Man P/N 7A-10.000MAAE-T -> ABLS-10.000MHZ-B2-T; URL http://www.digikey.com/product-search/en?pv7=2&k=7A-10.000M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 -> http://www.digikey.com/product-detail/en/abracon-llc/ABLS-1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
Connections:
- net +5V: now also U?.4 (V+), U?.4 (V+)
- net A1_LV: now also C?.2
- net A2_LV: now also C?.1
- net GND: now also C?.1, C?.2, C?.2, U?.11 (V-), U?.11 (V-)
- net IMD: now also C?.1, U?.1, U?.2 (-)
- net I_Measure: now also U?.1
- net Throttle_SEL: now reaches U7.17 ((OC0A/OC1C)PB7)
- net at U7.24 (XTAL1), Y1.1: now also C?.1
- net at R5.2: now also C?.2, U?.3 (+)
- net at R3.1, R6.2: now also U?.2 (-)
- net at R2.1, R4.1: now also U?.3 (+)
- net BP renamed BP_uC
- net THROTTLE_SEL renamed Throttle_PL
- net uC_THROTTLE renamed Throttle_uC
Changed lines of the file:
@@
 EESchema Schematic File Version 2
 LIBS:Circuit_layout-rescue
-LIBS:TSI_KiCad_Lib
 LIBS:TSI_HV_Isolater-cache
 LIBS:74xgxx
@@
 F 0 "Y1" H 2900 2700 50  0000 C CNN
 F 1 "10MHz" H 2900 2400 50  0000 C CNN
-F 2 "" H 2900 2550 50  0000 C CNN
-F 3 "" H 2900 2550 50  0000 C CNN
-F 4 "887-1741-1-ND" H 2900 2550 60  0001 C CNN "DigiKey P/N"
-F 5 "http://www.digikey.com/product-search/en?pv7=2&k=7A-10.000MAAE-T&mnonly=0&newproducts=0&ColumnSort=0&page=1&quantity=0&ptm=0&fid=0&pageSize=25" H 2900 2550 60  0001 C CNN "URL"
-F 6 "7A-10.000MAAE-T" H 2900 2550 60  0001 C CNN "Man P/N"
+F 2 "Crystals:Crystal_SMD_HC49-SD_HandSoldering" H 2900 2550 50  0001 C CNN
+F 3 "http://www.abracon.com/Resonators/abls.pdf" H 2900 2550 50  0001 C CNN
+F 4 "535-9065-1-ND" H 2900 2550 60  0001 C CNN "DigiKey P/N"
+F 5 "http://www.digikey.com/product-detail/en/abracon-llc/ABLS-10.000MHZ-B2-T/535-9065-1-ND/675582" H 2900 2550 60  0001 C CNN "URL"
+F 6 "ABLS-10.000MHZ-B2-T" H 2900 2550 60  0001 C CNN "Man P/N"
 	1    2900 2550
 	1    0    0    -1
@@
 Connection ~ 2750 2550
 Connection ~ 3050 2550
-$Comp
-L C C5
-U 1 1 58A868A1
-P 2750 2900
-F 0 "C5" H 2775 3000 50  0000 L CNN
-F 1 "10p" H 2775 2800 50  0000 L CNN
-F 2 "" H 2788 2750 50  0000 C CNN
-F 3 "" H 2750 2900 50  0000 C CNN
-F 4 "399-1108-1-ND" H 2750 2900 60  0001 C CNN "DigiKey P/N"
-F 5 "http://www.digikey.com/product-detail/en/kemet/C0805C100J5GACTU/399-1108-1-ND/411383" H 2750 2900 60  0001 C CNN "URL"
-	1    2750 2900
-	1    0    0    -1
-$EndComp
 Wire Wire Line
 	2750 3050 3050 3050
@@
 F 0 "C6" H 3075 3000 50  0000 L CNN
 F 1 "10p" H 3075 2800 50  0000 L CNN
-F 2 "" H 3088 2750 50  0000 C CNN
-F 3 "" H 3050 2900 50  0000 C CNN
+F 2 "Capacitors_SMD:C_0805_HandSoldering" H 3088 2750 50  0001 C CNN
+F 3 "" H 3050 2900 50  0001 C CNN
 F 4 "399-1108-1-ND" H 3050 2900 60  0001 C CNN "DigiKey P/N"
 F 5 "http://www.digikey.com/product-detail/en/kemet/C0805C100J5GACTU/399-1108-1-ND/411383" H 3050 2900 60  0001 C CNN "URL"
+F 6 "C0805C100J5GACTU" H 3050 2900 60  0001 C CNN "Man P/N"
 	1    3050 2900
 	1    0    0    -1
@@
 F2 "D_LED_CTRL" I L 8150 3850 60
 F3 "RTDS_CTRL" I L 8150 4150 60
+F4 "BP_uC" I R 9950 3800 60
+F5 "Brake_Light" O R 9950 4000 60
 $EndSheet
 $Sheet
@@
 	6550 3500 7200 3500
 Text Label 7200 3500 2    60   ~ 0
-uC_THROTTLE
+Throttle_uC
 Wire Wire Line
 	3950 3800 3300 3800
@@
 	6550 3400 7200 3400
 Text Label 7200 3400 2    60   ~ 0
-THROTTLE_SEL
+Throttle_PL
 Wire Wire Line
 	6550 3300 7200 3300
 Text Label 7200 3300 2    60   ~ 0
-BP
+BP_uC
 Wire Wire Line
 	6550 2300 7150 2300
@@
 Wire Wire Line
 	700  3750 1350 3750
-$Comp
-L C C1
-U 1 1 58B0B5F8
-P 1150 3250
-F 0 "C1" H 1175 3350 50  0000 L CNN
-F 1 "0.1u" H 1175 3150 50  0000 L CNN
-F 2 "Capacitors_SMD:C_0805_HandSoldering" H 1188 3100 50  0001 C CNN
-F 3 "" H 1150 3250 50  0000 C CNN
-	1    1150 3250
-	1    0    0    -1
-$EndComp
 Wire Wire Line
 	1800 3750 1800 4250
@@
 F0 "ThrottlePlausibility" 60
 F1 "ThrottlePlausibility.sch" 60
-F2 "GND" I L 8200 6400 60
-F3 "RTN_GLV" O L 8200 5650 60
-F4 "APPS1" O L 8200 5800 60
-F5 "APPS2" O L 8200 5950 60
-F6 "APPS1_10" O L 8200 5350 60
-F7 "APPS2_5" O L 8200 5500 60
-F8 "+12LV" I L 8200 6250 60
-F9 "Throttle_SEL" I R 9900 5650 60
-F10 "Throttle_uC" I R 9900 5500 60
-F11 "Throttle_LV" O R 9900 5350 60
-F12 "+5LV" I L 8200 6100 60
-F13 "BP" I R 9900 6100 60
-F14 "BRAKE_5" O R 9900 6400 60
-F15 "BP_uC" I R 9900 6250 60
+F2 "RTN_GLV" O L 8200 5650 60
+F3 "APPS1" O L 8200 5800 60
+F4 "APPS2" O L 8200 5950 60
+F5 "APPS1_10" O L 8200 5350 60
+F6 "APPS2_5" O L 8200 5500 60
+F7 "Throttle_SEL" I R 9900 5650 60
+F8 "Throttle_uC" I R 9900 5500 60
+F9 "Throttle_LV" O R 9900 5350 60
+F10 "BP" I R 9900 6100 60
+F11 "BRAKE_5" O R 9900 6400 60
+F12 "BP_uC" I R 9900 6250 60
+F13 "Throttle_PL" O R 9900 5800 60
 $EndSheet
 Text Notes 1350 2900 0    99   ~ 0
@@
 F 1 "0.47u" H 1725 1400 50  0000 L CNN
 F 2 "Capacitors_SMD:C_0805_HandSoldering" H 1738 1350 50  0001 C CNN
-F 3 "" H 1700 1500 50  0000 C CNN
+F 3 "http://www.kemet.com/Lists/ProductCatalog/Attachments/53/KEM_C1002_X7R_SMD.pdf" H 1700 1500 50  0001 C CNN
+F 4 "399-8100-1-ND" H 1700 1500 60  0001 C CNN "Digikey P/N"
+F 5 "http://www.digikey.com/product-detail/en/kemet/C0805C474K5RACTU/399-8100-1-ND/3471823" H 1700 1500 60  0001 C CNN "URL"
+F 6 "C0805C474K5RACTU" H 1700 1500 60  0001 C CNN "Man P/N"
 	1    1700 1500
 	1    0    0    -1
-$EndComp
-$Comp
-L C C4
-U 1 1 58B21267
-P 2700 900
-F 0 "C4" H 2725 1000 50  0000 L CNN
-F 1 "0.47u" H 2725 800 50  0000 L CNN
-F 2 "Capacitors_SMD:C_0805_HandSoldering" H 2738 750 50  0001 C CNN
-F 3 "" H 2700 900 50  0000 C CNN
-	1    2700 900
-	0    1    1    0
 $EndComp
 Wire Wire Line
@@
 Text Notes 600  2050 0    60   ~ 0
 Sallen-Key Filter\nIntended for 10Hz PWM\n2Hz fc - breadboarded - still osc
-$Comp
-L MCP6004 U4
-U 2 1 58B21292
-P 2600 1350
-F 0 "U4" H 2650 1550 50  0000 C CNN
-F 1 "MCP6004" H 2750 1150 50  0000 C CNN
-F 2 "" H 2550 1450 50  0000 C CNN
-F 3 "" H 2650 1550 50  0000 C CNN
-	2    2600 1350
-	1    0    0    -1
-$EndComp
 Text Label 650  1250 0    60   ~ 0
 IMD_PWM
@@
 Text Label 3100 1350 0    60   ~ 0
 IMD
-$Comp
-L MCP6004 U4
-U 1 1 58B2253B
-P 2200 3650
-F 0 "U4" H 2250 3850 50  0000 C CNN
-F 1 "MCP6004" H 2350 3450 50  0000 C CNN
-F 2 "" H 2150 3750 50  0000 C CNN
-F 3 "" H 2250 3850 50  0000 C CNN
-	1    2200 3650
-	1    0    0    -1
-$EndComp
 Wire Wire Line
 	6550 3900 7200 3900
@@
 F1 "isolators.sch" 60
 F2 "Throttle_LV" I L 850 4850 60
-F3 "+5HV" I R 2450 5300 60
-F4 "HV+" I R 2450 5450 60
-F5 "HV-" I R 2450 5600 60
+F3 "+5HV" I R 2450 5150 60
+F4 "HV+" I R 2450 5500 60
+F5 "HV-" I R 2450 5650 60
 F6 "Throttle_HV" O R 2450 4850 60
 F7 "V_Measure" I L 850 5000 60
+F8 "I/O_Ground" I R 2450 5300 60
 $EndSheet
 Text Notes 950  1050 0    99   ~ 0
 IMD PWM LPF
-$Comp
-L C C2
-U 1 1 58B54F3B
-P 1150 4050
-F 0 "C2" H 1175 4150 50  0000 L CNN
-F 1 "0.1u" H 1175 3950 50  0000 L CNN
-F 2 "Capacitors_SMD:C_0805_HandSoldering" H 1188 3900 50  0001 C CNN
-F 3 "" H 1150 4050 50  0000 C CNN
-	1    1150 4050
-	1    0    0    -1
-$EndComp
 $Comp
 L R R1
@@
 	-1   0    0    1
 $EndComp
+$Comp
+L MCP6004 U?
+U 1 1 58B3FEE2
+P 2200 3650
+F 0 "U?" H 2250 3850 50  0000 C CNN
+F 1 "MCP6004" H 2350 3450 50  0000 C CNN
+F 2 "Housings_SOIC:SOIC-14_3.9x8.7mm_Pitch1.27mm" H 2150 3750 50  0001 C CNN
+F 3 "http://ww1.microchip.com/downloads/en/DeviceDoc/21733j.pdf" H 2250 3850 50  0001 C CNN
+F 4 "MCP6004T-I/SLCT-ND" H 2200 3650 60  0001 C CNN "Digikey P/N"
+F 5 "http://www.digikey.com/product-detail/en/microchip-technology/MCP6004T-I-SL/MCP6004T-I-SLCT-ND/5013527" H 2200 3650 60  0001 C CNN "URL"
+F 6 "MCP6004T-I/SL" H 2200 3650 60  0001 C CNN "Man P/N"
+	1    2200 3650
+	1    0    0    -1
+$EndComp
+$Comp
+L C C?
+U 1 1 58B40314
+P 1150 4050
+F 0 "C?" H 1175 4150 50  0000 L CNN
+F 1 "0.1u" H 1175 3950 50  0000 L CNN
+F 2 "Capacitors_SMD:C_0805_HandSoldering" H 1188 3900 50  0001 C CNN
+F 3 "http://www.kemet.com/Lists/ProductCatalog/Attachments/53/KEM_C1002_X7R_SMD.pdf" H 1150 4050 50  0001 C CNN
+F 4 "399-1168-1-ND" H 1150 4050 60  0001 C CNN "Digikey P/N"
+F 5 "http://www.digikey.com/product-detail/en/kemet/C0805C104K3RACTU/399-1168-1-ND/411443" H 1150 4050 60  0001 C CNN "URL"
+F 6 "C0805C104K3RACTU" H 1150 4050 60  0001 C CNN "Man P/N"
+	1    1150 4050
+	1    0    0    -1
+$EndComp
+$Comp
+L C C?
+U 1 1 58B40445
+P 1150 3250
+F 0 "C?" H 1175 3350 50  0000 L CNN
+F 1 "0.1u" H 1175 3150 50  0000 L CNN
+F 2 "Capacitors_SMD:C_0805_HandSoldering" H 1188 3100 50  0001 C CNN
+F 3 "http://www.kemet.com/Lists/ProductCatalog/Attachments/53/KEM_C1002_X7R_SMD.pdf" H 1150 3250 50  0001 C CNN
+F 4 "399-1168-1-ND" H 1150 3250 60  0001 C CNN "Digikey P/N"
+F 5 "http://www.digikey.com/product-detail/en/kemet/C0805C104K3RACTU/399-1168-1-ND/411443" H 1150 3250 60  0001 C CNN "URL"
+F 6 "C0805C104K3RACTU" H 1150 3250 60  0001 C CNN "Man P/N"
+	1    1150 3250
+	1    0    0    -1
+$EndComp
+$Comp
+L MCP6004 U?
+U 1 1 58B40627
+P 2600 1350
+F 0 "U?" H 2650 1550 50  0000 C CNN
+F 1 "MCP6004" H 2750 1150 50  0000 C CNN
+F 2 "Housings_SOIC:SOIC-14_3.9x8.7mm_Pitch1.27mm" H 2550 1450 50  0001 C CNN
+F 3 "http://ww1.microchip.com/downloads/en/DeviceDoc/21733j.pdf" H 2650 1550 50  0001 C CNN
+F 4 "MCP6004T-I/SLCT-ND" H 2600 1350 60  0001 C CNN "Digikey P/N"
+F 5 "http://www.digikey.com/product-detail/en/microchip-technology/MCP6004T-I-SL/MCP6004T-I-SLCT-ND/5013527" H 2600 1350 60  0001 C CNN "URL"
+F 6 "MCP6004T-I/SL" H 2600 1350 60  0001 C CNN "Man P/N"
+	1    2600 1350
+	1    0    0    -1
+$EndComp
+$Comp
+L C C?
+U 1 1 58B40E21
+P 2700 900
+F 0 "C?" H 2725 1000 50  0000 L CNN
+F 1 "0.47u" H 2725 800 50  0000 L CNN
+F 2 "Capacitors_SMD:C_0805_HandSoldering" H 2738 750 50  0001 C CNN
+F 3 "http://www.kemet.com/Lists/ProductCatalog/Attachments/53/KEM_C1002_X7R_SMD.pdf" H 2700 900 50  0001 C CNN
+F 4 "399-8100-1-ND" H 2700 900 60  0001 C CNN "Digikey P/N"
+F 5 "http://www.digikey.com/product-detail/en/kemet/C0805C474K5RACTU/399-8100-1-ND/3471823" H 2700 900 60  0001 C CNN "URL"
+F 6 "C0805C474K5RACTU" H 2700 900 60  0001 C CNN "Man P/N"
+	1    2700 900
+	0    1    1    0
+$EndComp
+$Comp
+L C C?
+U 1 1 58B423A5
+P 2750 2900
+F 0 "C?" H 2775 3000 50  0000 L CNN
+F 1 "10p" H 2775 2800 50  0000 L CNN
+F 2 "Capacitors_SMD:C_0805_HandSoldering" H 2788 2750 50  0001 C CNN
+F 3 "" H 2750 2900 50  0001 C CNN
+F 4 "399-1108-1-ND" H 2750 2900 60  0001 C CNN "DigiKey P/N"
+F 5 "http://www.digikey.com/product-detail/en/kemet/C0805C100J5GACTU/399-1108-1-ND/411383" H 2750 2900 60  0001 C CNN "URL"
+F 6 "C0805C100J5GACTU" H 2750 2900 60  0001 C CNN "Man P/N"
+	1    2750 2900
+	1    0    0    -1
+$EndComp
+Wire Wire Line
+	6550 3600 7200 3600
+Text Label 7200 3600 2    60   ~ 0
+Throttle_SEL
 $EndSCHEMATC

Commit message: working on schematic
Changed lines of the file:
@@
 EESchema Schematic File Version 2
 LIBS:Circuit_layout-rescue
+LIBS:TSI_KiCad_Lib
 LIBS:TSI_HV_Isolater-cache
 LIBS:74xgxx
@@
 $EndComp
 $Sheet
-S 8150 3600 1800 1050
+S 8150 3600 1550 850
 U 58ADE509
 F0 "Status Lights" 60
@@
 F2 "D_LED_CTRL" I L 8150 3850 60
 F3 "RTDS_CTRL" I L 8150 4150 60
-F4 "BP_uC" I R 9950 3800 60
-F5 "Brake_Light" O R 9950 4000 60
+F4 "BP_uC" I R 9700 3800 60
+F5 "Brake_Light" O R 9700 4000 60
 $EndSheet
 $Sheet
@@
 Text Label 7200 3600 2    60   ~ 0
 Throttle_SEL
+Text GLabel 9850 4000 2    60   Input ~ 0
+Brake_Light
+Wire Wire Line
+	9850 4000 9700 4000
 $EndSCHEMATC
