File: Circuit_layout/Ext_Connectors.sch (KiCad schematic (older format))
At the start: 14 parts, among them CON1 AVR-JTAG-10, J10 CONN_01X02, J11 CONN_8, J3 CONN_01X02, J4 CONN_01X04, J5 RJ12, J7 CONN_01X06, P1 CONN_01X02, P2 CONN_01X02, P3 CONN_01X03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

Commit message: took notes on nadovich's proposed changes
Other:
- note removed: "Need to see how this was done an pacman. Used to try and eliminate errors.\n"
- moved on the sheet: CON1, J5
Changed lines of the file:
@@
 L RJ12 J5
 U 1 1 58A76FD9
-P 1000 1100
-F 0 "J5" H 1200 1600 50  0000 C CNN
-F 1 "RJ12" H 850 1600 50  0000 C CNN
-F 2 "" H 1000 1100 50  0000 C CNN
-F 3 "" H 1000 1100 50  0000 C CNN
-F 4 "WM3789CT-ND" H 1000 1100 60  0001 C CNN "DigiKey P/N"
-F 5 "http://www.digikey.com/product-search/en?keywords=WM3789CT-ND" H 1000 1100 60  0001 C CNN "URL"
-	1    1000 1100
-	1    0    0    -1
-$EndComp
-NoConn ~ 1500 700
-NoConn ~ 1500 800
+P 1500 1100
+F 0 "J5" H 1700 1600 50  0000 C CNN
+F 1 "RJ12" H 1350 1600 50  0000 C CNN
+F 2 "" H 1500 1100 50  0000 C CNN
+F 3 "" H 1500 1100 50  0000 C CNN
+F 4 "WM3789CT-ND" H 1500 1100 60  0001 C CNN "DigiKey P/N"
+F 5 "http://www.digikey.com/product-search/en?keywords=WM3789CT-ND" H 1500 1100 60  0001 C CNN "URL"
+	1    1500 1100
+	1    0    0    -1
+$EndComp
+NoConn ~ 2000 700
+NoConn ~ 2000 800
+NoConn ~ 1800 1550
 NoConn ~ 1300 1550
-NoConn ~ 800  1550
 $Comp
 L CONN_01X02 P1
@@
 L AVR-JTAG-10 CON1
 U 1 1 58A7E9A9
-P 5850 5600
-F 0 "CON1" H 5680 5930 50  0000 C CNN
-F 1 "AVR-JTAG-10" H 5510 5270 50  0000 L BNN
-F 2 "AVR-JTAG-10" V 5280 5620 50  0001 C CNN
-F 3 "" H 5850 5600 50  0000 C CNN
-	1    5850 5600
-	1    0    0    -1
-$EndComp
-NoConn ~ 5900 5700
-NoConn ~ 5650 5700
-Text GLabel 5200 5350 0    60   Input ~ 0
+P 5300 4200
+F 0 "CON1" H 5130 4530 50  0000 C CNN
+F 1 "AVR-JTAG-10" H 4960 3870 50  0000 L BNN
+F 2 "AVR-JTAG-10" V 4730 4220 50  0001 C CNN
+F 3 "" H 5300 4200 50  0000 C CNN
+	1    5300 4200
+	1    0    0    -1
+$EndComp
+NoConn ~ 5350 4300
+NoConn ~ 5100 4300
+Text GLabel 4650 3950 0    60   Input ~ 0
 TCK
-Text GLabel 5200 5500 0    60   Input ~ 0
+Text GLabel 4650 4100 0    60   Input ~ 0
 TDO
-Text GLabel 5200 5650 0    60   Input ~ 0
+Text GLabel 4650 4250 0    60   Input ~ 0
 TMS
-Text GLabel 5200 5800 0    60   Input ~ 0
+Text GLabel 4650 4400 0    60   Input ~ 0
 TDI
 $Comp
 L GND #PWR23
 U 1 1 58A81278
-P 6250 5900
-F 0 "#PWR23" H 6250 5650 50  0001 C CNN
-F 1 "GND" H 6250 5750 50  0000 C CNN
-F 2 "" H 6250 5900 50  0000 C CNN
-F 3 "" H 6250 5900 50  0000 C CNN
-	1    6250 5900
-	1    0    0    -1
-$EndComp
-Text GLabel 6400 5600 2    60   Input ~ 0
+P 5700 4500
+F 0 "#PWR23" H 5700 4250 50  0001 C CNN
+F 1 "GND" H 5700 4350 50  0000 C CNN
+F 2 "" H 5700 4500 50  0000 C CNN
+F 3 "" H 5700 4500 50  0000 C CNN
+	1    5700 4500
+	1    0    0    -1
+$EndComp
+Text GLabel 5850 4200 2    60   Input ~ 0
 ~RESET_AVR
 $Comp
 L +5V #PWR24
 U 1 1 58A81530
-P 6400 5400
-F 0 "#PWR24" H 6400 5250 50  0001 C CNN
-F 1 "+5V" H 6400 5540 50  0000 C CNN
-F 2 "" H 6400 5400 50  0000 C CNN
-F 3 "" H 6400 5400 50  0000 C CNN
-	1    6400 5400
+P 5850 4000
+F 0 "#PWR24" H 5850 3850 50  0001 C CNN
+F 1 "+5V" H 5850 4140 50  0000 C CNN
+F 2 "" H 5850 4000 50  0000 C CNN
+F 3 "" H 5850 4000 50  0000 C CNN
+	1    5850 4000
 	1    0    0    -1
 $EndComp
@@
 +24V_RTN
 $Comp
-L +24V #PWR21
+L +24V #PWR19
 U 1 1 58AF1C5B
 P 1350 2600
-F 0 "#PWR21" H 1350 2450 50  0001 C CNN
+F 0 "#PWR19" H 1350 2450 50  0001 C CNN
 F 1 "+24V" H 1350 2740 50  0000 C CNN
 F 2 "" H 1350 2600 50  0000 C CNN
@@
 Drive_LED
 $Comp
-L +5V #PWR27
+L +5V #PWR26
 U 1 1 58B1052B
-P 7750 3950
-F 0 "#PWR27" H 7750 3800 50  0001 C CNN
-F 1 "+5V" H 7750 4090 50  0000 C CNN
-F 2 "" H 7750 3950 50  0000 C CNN
-F 3 "" H 7750 3950 50  0000 C CNN
-	1    7750 3950
+P 7650 4000
+F 0 "#PWR26" H 7650 3850 50  0001 C CNN
+F 1 "+5V" H 7650 4140 50  0000 C CNN
+F 2 "" H 7650 4000 50  0000 C CNN
+F 3 "" H 7650 4000 50  0000 C CNN
+	1    7650 4000
 	1    0    0    -1
 $EndComp
@@
 Brake_Light_RTN
 $Comp
-L GND #PWR25
+L GND #PWR27
 U 1 1 58B4A72F
 P 7750 3150
-F 0 "#PWR25" H 7750 2900 50  0001 C CNN
+F 0 "#PWR27" H 7750 2900 50  0001 C CNN
 F 1 "GND" H 7750 3000 50  0000 C CNN
 F 2 "" H 7750 3150 50  0000 C CNN
@@
 	8500 4100 9550 4100
 Wire Wire Line
-	7750 4000 9550 4000
+	7650 4000 9550 4000
 Wire Wire Line
 	8500 3900 9550 3900
@@
 	1150 6650 1550 6650
 Wire Wire Line
-	1100 1550 1100 1900
-Wire Wire Line
-	1000 1550 1000 1900
-Wire Wire Line
-	900  1550 900  1900
+	1600 1550 1600 1900
+Wire Wire Line
+	1500 1550 1500 1900
+Wire Wire Line
+	1400 1550 1400 1900
 Wire Wire Line
 	9550 5000 9400 5000
@@
 	4300 5300 4300 7800
 Wire Wire Line
-	5200 5800 5650 5800
-Wire Wire Line
-	5650 5600 5200 5600
-Wire Wire Line
-	5650 5500 5200 5500
-Wire Wire Line
-	5200 5400 5650 5400
-Wire Wire Line
-	5200 5600 5200 5650
-Wire Wire Line
-	5900 5800 6250 5800
-Wire Wire Line
-	6250 5400 6250 5900
-Wire Wire Line
-	5900 5400 6250 5400
-Connection ~ 6250 5800
-Wire Wire Line
-	5900 5500 6400 5500
-Wire Wire Line
-	6400 5500 6400 5400
-Wire Wire Line
-	5900 5600 6400 5600
-Wire Wire Line
-	5200 5400 5200 5350
+	4650 4400 5100 4400
+Wire Wire Line
+	5100 4200 4650 4200
+Wire Wire Line
+	5100 4100 4650 4100
+Wire Wire Line
+	4650 4000 5100 4000
+Wire Wire Line
+	4650 4200 4650 4250
+Wire Wire Line
+	5350 4400 5700 4400
+Wire Wire Line
+	5700 4000 5700 4500
+Wire Wire Line
+	5350 4000 5700 4000
+Connection ~ 5700 4400
+Wire Wire Line
+	5350 4100 5850 4100
+Wire Wire Line
+	5850 4100 5850 4000
+Wire Wire Line
+	5350 4200 5850 4200
+Wire Wire Line
+	4650 4000 4650 3950
 Wire Wire Line
 	1100 5750 1850 5750
@@
 	7750 2650 9550 2650
 $Comp
-L +5V #PWR20
+L +5V #PWR22
 U 1 1 58BB5596
-P 1200 1750
-F 0 "#PWR20" H 1200 1600 50  0001 C CNN
-F 1 "+5V" H 1200 1890 50  0000 C CNN
-F 2 "" H 1200 1750 50  0000 C CNN
-F 3 "" H 1200 1750 50  0000 C CNN
-	1    1200 1750
+P 1700 1750
+F 0 "#PWR22" H 1700 1600 50  0001 C CNN
+F 1 "+5V" H 1700 1890 50  0000 C CNN
+F 2 "" H 1700 1750 50  0000 C CNN
+F 3 "" H 1700 1750 50  0000 C CNN
+	1    1700 1750
 	-1   0    0    1
 $EndComp
 $Comp
-L GND #PWR19
+L GND #PWR21
 U 1 1 58BB55DD
-P 1100 1900
-F 0 "#PWR19" H 1100 1650 50  0001 C CNN
-F 1 "GND" H 1100 1750 50  0000 C CNN
-F 2 "" H 1100 1900 50  0000 C CNN
-F 3 "" H 1100 1900 50  0000 C CNN
-	1    1100 1900
-	1    0    0    -1
-$EndComp
-Wire Wire Line
-	1200 1550 1200 1750
-Text GLabel 1000 1900 3    60   Input ~ 0
+P 1600 1900
+F 0 "#PWR21" H 1600 1650 50  0001 C CNN
+F 1 "GND" H 1600 1750 50  0000 C CNN
+F 2 "" H 1600 1900 50  0000 C CNN
+F 3 "" H 1600 1900 50  0000 C CNN
+	1    1600 1900
+	1    0    0    -1
+$EndComp
+Wire Wire Line
+	1700 1550 1700 1750
+Text GLabel 1500 1900 3    60   Input ~ 0
 A2_LV
-Text GLabel 900  1900 3    60   Input ~ 0
+Text GLabel 1400 1900 3    60   Input ~ 0
 A1_LV
 $Comp
@@
 CH_GND
 $Comp
-L GND #PWR26
+L GND #PWR25
 U 1 1 58B7A0E8
-P 7750 3700
-F 0 "#PWR26" H 7750 3450 50  0001 C CNN
-F 1 "GND" H 7750 3550 50  0000 C CNN
-F 2 "" H 7750 3700 50  0000 C CNN
-F 3 "" H 7750 3700 50  0000 C CNN
-	1    7750 3700
-	-1   0    0    1
+P 7500 3800
+F 0 "#PWR25" H 7500 3550 50  0001 C CNN
+F 1 "GND" H 7500 3650 50  0000 C CNN
+F 2 "" H 7500 3800 50  0000 C CNN
+F 3 "" H 7500 3800 50  0000 C CNN
+	1    7500 3800
+	1    0    0    -1
 $EndComp
 Text GLabel 1200 3000 0    60   Input ~ 0
 CH_GND
 $Comp
-L GND #PWR22
+L GND #PWR20
 U 1 1 58B888D9
 P 1400 3250
-F 0 "#PWR22" H 1400 3000 50  0001 C CNN
+F 0 "#PWR20" H 1400 3000 50  0001 C CNN
 F 1 "GND" H 1400 3100 50  0000 C CNN
 F 2 "" H 1400 3250 50  0000 C CNN
@@
 HVPL
 Wire Wire Line
-	7750 3800 9550 3800
-Text Notes 1600 2950 0    60   ~ 0
-Need to see how this was done an pacman. Used to try and eliminate errors.\n
-Text GLabel 1450 4800 2    60   Input ~ 0
+	7500 3800 9550 3800
+Text GLabel 1750 4800 2    60   Input ~ 0
 CANH
-Text GLabel 1450 4900 2    60   Input ~ 0
+Text GLabel 1750 4900 2    60   Input ~ 0
 CANL
 Wire Wire Line
@@
 $EndComp
 Wire Wire Line
-	7750 3800 7750 3700
-Wire Wire Line
-	7750 4000 7750 3950
-Wire Wire Line
 	8500 4200 9550 4200
