File: Circuit_layout/PowerSystem.sch (KiCad schematic (older format))
At the start: 6 parts, among them U13 PDQ10-D, U14 PDQ15-D

Commit message: working on schematic
Parts:
- removed C10, C8: 10uF, Capacitors_SMD:C_0805_HandSoldering, symbol C
- removed C11: 6.8uF, Capacitors_SMD:C_0805_HandSoldering, symbol C
- added C?: 6.8uF, Capacitors_SMD:C_0805_HandSoldering, symbol C
- added C? (x4): 10uF, Capacitors_SMD:C_0805_HandSoldering, symbol C
- added R? (x10): R, symbol R
- added U?: PDQ6-D, symbol PDQ6-D
- C9: DigiKey P/N 445-14366-1-ND -> 445-14433-1-ND; Man P/N C2012X5R1A685K085AB -> C2012X5R1V685K125AC; URL http://www.digikey.com/product-detail/en/tdk-corporation/C2012X5R1A685K085AB/445-14366-1-ND/3956032 -> http://www.digikey.com/product-detail/en/tdk-corporation/C2012X5R1V685K125AC/445-14433-1-ND/3956099
Connections:
- net labels added: HV+, HV-, HVPL, HVPL_RTN
- wire segments 20 -> 44
- no-connect marks 4 -> 5
Other:
- note added: "Datasheet recommends 100uF, but I can't find one that has a high enough voltage threshold"

Commit message: took notes w/ greg
Parts:
- gave numbers to parts that had none: 16
Connections:
- net labels removed: Earth
- wire segments 44 -> 37
Other:
- moved on the sheet: R36, R37
Changed lines of the file:
@@
 	4550 4200 4550 4100
 Wire Wire Line
-	4550 4100 4200 4100
-Wire Wire Line
-	4200 4100 3800 4100
-Wire Wire Line
-	3800 4100 3350 4100
+	4550 4100 3350 4100
 Connection ~ 4200 4100
 Connection ~ 3800 4100
@@
 	4550 4300 4550 4400
 Wire Wire Line
-	4550 4400 4200 4400
-Wire Wire Line
-	4200 4400 3800 4400
-Wire Wire Line
-	3800 4400 3350 4400
+	4550 4400 3350 4400
 Connection ~ 4200 4400
 Connection ~ 3800 4400
@@
 	4500 2150 4500 2100
 Wire Wire Line
-	4500 2100 4150 2100
-Wire Wire Line
-	4150 2100 3800 2100
-Wire Wire Line
-	3800 2100 3350 2100
+	4500 2100 3350 2100
 Wire Wire Line
 	4650 2250 4500 2250
@@
 	4500 2250 4500 2400
 Wire Wire Line
-	4500 2400 4150 2400
-Wire Wire Line
-	4150 2400 3800 2400
-Wire Wire Line
-	3800 2400 3350 2400
+	4500 2400 3350 2400
 Connection ~ 4150 2100
 Connection ~ 4150 2400
@@
 Connection ~ 3800 2100
 $Comp
-L +24V #PWR032
+L +24V #PWR036
 U 1 1 58AF1DB3
 P 3350 4100
-F 0 "#PWR032" H 3350 3950 50  0001 C CNN
+F 0 "#PWR036" H 3350 3950 50  0001 C CNN
 F 1 "+24V" H 3350 4240 50  0000 C CNN
 F 2 "" H 3350 4100 50  0000 C CNN
@@
 $EndComp
 $Comp
-L +24V #PWR033
+L +24V #PWR037
 U 1 1 58AF1DD3
 P 3350 2100
-F 0 "#PWR033" H 3350 1950 50  0001 C CNN
+F 0 "#PWR037" H 3350 1950 50  0001 C CNN
 F 1 "+24V" H 3350 2240 50  0000 C CNN
 F 2 "" H 3350 2100 50  0000 C CNN
@@
 	6550 2150 6550 2050
 $Comp
-L +5V #PWR034
+L +5V #PWR038
 U 1 1 58AF2067
 P 6550 2050
-F 0 "#PWR034" H 6550 1900 50  0001 C CNN
+F 0 "#PWR038" H 6550 1900 50  0001 C CNN
 F 1 "+5V" H 6550 2190 50  0000 C CNN
 F 2 "" H 6550 2050 50  0000 C CNN
@@
 $EndComp
 $Comp
-L +12V #PWR035
+L +12V #PWR039
 U 1 1 58AF208D
 P 6600 4100
-F 0 "#PWR035" H 6600 3950 50  0001 C CNN
+F 0 "#PWR039" H 6600 3950 50  0001 C CNN
 F 1 "+12V" H 6600 4240 50  0000 C CNN
 F 2 "" H 6600 4100 50  0000 C CNN
@@
 	6550 2350 6550 2450
 $Comp
-L GND #PWR036
+L GND #PWR040
 U 1 1 58AF2561
 P 6550 2450
-F 0 "#PWR036" H 6550 2200 50  0001 C CNN
+F 0 "#PWR040" H 6550 2200 50  0001 C CNN
 F 1 "GND" H 6550 2300 50  0000 C CNN
 F 2 "" H 6550 2450 50  0000 C CNN
@@
 	6600 4400 6600 4550
 $Comp
-L GND #PWR037
+L GND #PWR041
 U 1 1 58AF25AA
 P 6600 4550
-F 0 "#PWR037" H 6600 4300 50  0001 C CNN
+F 0 "#PWR041" H 6600 4300 50  0001 C CNN
 F 1 "GND" H 6600 4400 50  0000 C CNN
 F 2 "" H 6600 4550 50  0000 C CNN
@@
 	1    0    0    -1
 $EndComp
-$Comp
-L Earth #PWR038
-U 1 1 58AF26C0
-P 6300 2350
-F 0 "#PWR038" H 6300 2100 50  0001 C CNN
-F 1 "Earth" H 6300 2200 50  0001 C CNN
-F 2 "" H 6300 2350 50  0000 C CNN
-F 3 "" H 6300 2350 50  0000 C CNN
-	1    6300 2350
-	1    0    0    -1
-$EndComp
-$Comp
-L Earth #PWR039
-U 1 1 58AF28A2
-P 6350 4400
-F 0 "#PWR039" H 6350 4150 50  0001 C CNN
-F 1 "Earth" H 6350 4250 50  0001 C CNN
-F 2 "" H 6350 4400 50  0000 C CNN
-F 3 "" H 6350 4400 50  0000 C CNN
-	1    6350 4400
-	1    0    0    -1
-$EndComp
 Text Notes 3700 7250 0    60   ~ 0
 DC DC Converter\n9V-36V to 12V
@@
 	3200 6600 3200 6500
 Wire Wire Line
-	3200 6500 3000 6500
-Wire Wire Line
-	3000 6500 2800 6500
+	3200 6500 2800 6500
 Connection ~ 3000 6500
-Wire Wire Line
-	2800 6800 3000 6800
-Wire Wire Line
-	3000 6800 3300 6800
 Connection ~ 3000 6800
 Wire Wire Line
@@
 	4050 5750 4050 7800
 $Comp
-L R R?
+L R R37
 U 1 1 58B4D9F5
-P 1150 6500
-F 0 "R?" V 1230 6500 50  0000 C CNN
-F 1 "R" V 1150 6500 50  0000 C CNN
-F 2 "" V 1080 6500 50  0000 C CNN
-F 3 "" H 1150 6500 50  0000 C CNN
-	1    1150 6500
-	0    1    1    0
-$EndComp
-$Comp
-L R R?
+P 1100 6500
+F 0 "R37" V 1180 6500 50  0000 C CNN
+F 1 "R" V 1100 6500 50  0000 C CNN
+F 2 "" V 1030 6500 50  0000 C CNN
+F 3 "" H 1100 6500 50  0000 C CNN
+	1    1100 6500
+	0    1    1    0
+$EndComp
+$Comp
+L R R39
 U 1 1 58B4DA62
 P 1450 6500
-F 0 "R?" V 1530 6500 50  0000 C CNN
+F 0 "R39" V 1530 6500 50  0000 C CNN
 F 1 "R" V 1450 6500 50  0000 C CNN
 F 2 "" V 1380 6500 50  0000 C CNN
@@
 $EndComp
 $Comp
-L R R?
+L R R72
 U 1 1 58B4DA9B
 P 1750 6500
-F 0 "R?" V 1830 6500 50  0000 C CNN
+F 0 "R72" V 1830 6500 50  0000 C CNN
 F 1 "R" V 1750 6500 50  0000 C CNN
 F 2 "" V 1680 6500 50  0000 C CNN
@@
 $EndComp
 $Comp
-L R R?
+L R R73
 U 1 1 58B4DAE3
 P 2050 6500
-F 0 "R?" V 2130 6500 50  0000 C CNN
+F 0 "R73" V 2130 6500 50  0000 C CNN
 F 1 "R" V 2050 6500 50  0000 C CNN
 F 2 "" V 1980 6500 50  0000 C CNN
@@
 $EndComp
 $Comp
-L R R?
+L R R75
 U 1 1 58B4DB4B
 P 2350 6500
-F 0 "R?" V 2430 6500 50  0000 C CNN
+F 0 "R75" V 2430 6500 50  0000 C CNN
 F 1 "R" V 2350 6500 50  0000 C CNN
 F 2 "" V 2280 6500 50  0000 C CNN
@@
 $EndComp
 $Comp
-L R R?
+L R R36
 U 1 1 58B4DB95
-P 850 6500
-F 0 "R?" V 930 6500 50  0000 C CNN
-F 1 "R" V 850 6500 50  0000 C CNN
-F 2 "" V 780 6500 50  0000 C CNN
-F 3 "" H 850 6500 50  0000 C CNN
-	1    850  6500
-	0    1    1    0
-$EndComp
-$Comp
-L R R?
+P 800 6500
+F 0 "R36" V 880 6500 50  0000 C CNN
+F 1 "R" V 800 6500 50  0000 C CNN
+F 2 "" V 730 6500 50  0000 C CNN
+F 3 "" H 800 6500 50  0000 C CNN
+	1    800  6500
+	0    1    1    0
+$EndComp
+$Comp
+L R R77
 U 1 1 58B4DC07
 P 2650 6500
-F 0 "R?" V 2730 6500 50  0000 C CNN
+F 0 "R77" V 2730 6500 50  0000 C CNN
 F 1 "R" V 2650 6500 50  0000 C CNN
 F 2 "" V 2580 6500 50  0000 C CNN
@@
 $EndComp
 $Comp
-L R R?
+L R R78
 U 1 1 58B4DCDF
 P 2650 6800
-F 0 "R?" V 2730 6800 50  0000 C CNN
+F 0 "R78" V 2730 6800 50  0000 C CNN
 F 1 "R" V 2650 6800 50  0000 C CNN
 F 2 "" V 2580 6800 50  0000 C CNN
@@
 $EndComp
 $Comp
-L R R?
+L R R76
 U 1 1 58B4DD5E
 P 2350 6800
-F 0 "R?" V 2430 6800 50  0000 C CNN
+F 0 "R76" V 2430 6800 50  0000 C CNN
 F 1 "R" V 2350 6800 50  0000 C CNN
 F 2 "" V 2280 6800 50  0000 C CNN
@@
 $EndComp
 $Comp
-L R R?
+L R R74
 U 1 1 58B4DDAC
 P 2050 6800
-F 0 "R?" V 2130 6800 50  0000 C CNN
+F 0 "R74" V 2130 6800 50  0000 C CNN
 F 1 "R" V 2050 6800 50  0000 C CNN
 F 2 "" V 1980 6800 50  0000 C CNN
@@
 $EndComp
 Wire Wire Line
-	700  6500 700  6850
-Wire Wire Line
-	1900 6800 1500 6800
+	650  6500 650  6850
+Wire Wire Line
+	1500 6800 1900 6800
 Text Label 1500 6800 0    60   ~ 0
 HV-
-Text Label 700  6850 0    60   ~ 0
+Text Label 650  6850 0    60   ~ 0
 HV+
 $Comp
-L PDQ6-D U?
+L PDQ6-D U18
 U 1 1 58B515A4
 P 4050 6700
-F 0 "U?" H 4050 6600 50  0000 C CNN
+F 0 "U18" H 4050 6600 50  0000 C CNN
 F 1 "PDQ6-D" H 4050 6800 50  0000 C CNN
 F 2 "" H 4050 6300 50  0001 C CNN
@@
 $EndComp
 $Comp
-L C C?
+L C C21
 U 1 1 58B52AED
 P 4200 4250
-F 0 "C?" H 4225 4350 50  0000 L CNN
+F 0 "C21" H 4225 4350 50  0000 L CNN
 F 1 "6.8uF" H 4225 4150 50  0000 L CNN
 F 2 "Capacitors_SMD:C_0805_HandSoldering" H 4238 4100 50  0001 C CNN
@@
 	1    0    0    -1
 $EndComp
-$Comp
-L Earth #PWR?
-U 1 1 58B4CD4F
-P 4950 6800
-F 0 "#PWR?" H 4950 6550 50  0001 C CNN
-F 1 "Earth" H 4950 6650 50  0001 C CNN
-F 2 "" H 4950 6800 50  0000 C CNN
-F 3 "" H 4950 6800 50  0000 C CNN
-	1    4950 6800
-	1    0    0    -1
-$EndComp
 Wire Wire Line
 	5100 6600 5100 6550
 Wire Wire Line
-	5100 6550 5300 6550
-Wire Wire Line
-	5300 6550 6000 6550
+	5100 6550 6000 6550
 Wire Wire Line
 	5100 6800 5100 6850
 Wire Wire Line
-	5100 6850 5300 6850
-Wire Wire Line
-	5300 6850 6000 6850
+	5100 6850 6000 6850
 Connection ~ 5300 6550
 Connection ~ 5300 6850
@@
 HVPL_RTN
 $Comp
-L C C?
+L C C8
 U 1 1 58B5815B
 P 3000 6650
-F 0 "C?" H 3025 6750 50  0000 L CNN
+F 0 "C8" H 3025 6750 50  0000 L CNN
 F 1 "10uF" H 3025 6550 50  0000 L CNN
 F 2 "Capacitors_SMD:C_0805_HandSoldering" H 3038 6500 50  0001 C CNN
@@
 $EndComp
 $Comp
-L C C?
+L C C23
 U 1 1 58B5825D
 P 5300 6700
-F 0 "C?" H 5325 6800 50  0000 L CNN
+F 0 "C23" H 5325 6800 50  0000 L CNN
 F 1 "10uF" H 5325 6600 50  0000 L CNN
 F 2 "Capacitors_SMD:C_0805_HandSoldering" H 5338 6550 50  0001 C CNN
@@
 Datasheet recommends 100uF, but I can't find one that has a high enough voltage threshold
 $Comp
-L C C?
+L C C10
 U 1 1 58B58FF4
 P 3800 2250
-F 0 "C?" H 3825 2350 50  0000 L CNN
+F 0 "C10" H 3825 2350 50  0000 L CNN
 F 1 "10uF" H 3825 2150 50  0000 L CNN
 F 2 "Capacitors_SMD:C_0805_HandSoldering" H 3838 2100 50  0001 C CNN
@@
 $EndComp
 $Comp
-L C C?
+L C C11
 U 1 1 58B59092
 P 4150 2250
-F 0 "C?" H 4175 2350 50  0000 L CNN
+F 0 "C11" H 4175 2350 50  0000 L CNN
 F 1 "10uF" H 4175 2150 50  0000 L CNN
 F 2 "Capacitors_SMD:C_0805_HandSoldering" H 4188 2100 50  0001 C CNN
@@
 	1    0    0    -1
 $EndComp
+Wire Wire Line
+	3000 6800 3300 6800
+Wire Wire Line
+	3000 6800 3000 7000
+Wire Wire Line
+	3000 7000 1700 7000
+Wire Wire Line
+	1700 7000 1700 6800
+Connection ~ 1700 6800
+Wire Wire Line
+	2800 6800 2850 6800
+Wire Wire Line
+	2850 6800 2850 6500
+Connection ~ 2850 6500
 $EndSCHEMATC
