File: Circuit_layout/PowerSystem.sch (KiCad schematic (older format))
At the start: 8 parts, among them U13 PDQ10-D, U14 PDQ15-D

Commit message: current sensor enable
Parts:
- removed C21, C9: 6.8uF, Capacitors_SMD:C_0805_HandSoldering, symbol C
- removed C36: 0.1u, Capacitors_SMD:C_0805_HandSoldering, symbol C
- removed U14: PDQ15-D, custom_footprints:PDQ_DCDC, symbol PDQ
Connections:
- net labels removed: +12V
- wire segments 30 -> 16
- no-connect marks 4 -> 2
Other:
- note removed: "DC DC Converter\n9V-36V to 12V"
- moved on the sheet: C10, C11, C37, U13

Commit message: added footprint to DPDT switch, test points, DRC passes
Parts:
- added W?: +5DC/DC, Measurement_Points:Measurement_Point_Round-SMD-Pad_Big, symbol TEST_1P
- added W?: +5DC/DC_GND, Measurement_Points:Measurement_Point_Square-SMD-Pad_Big, symbol TEST_1P
Connections:
- net +5V: now also W?.1
- net GND: now also W?.1
Changed lines of the file:
@@
 LIBS:xilinx
 LIBS:Zilog
+LIBS:pacman-main-cache
 LIBS:bss84
 LIBS:+10v
@@
 NoConn ~ 3450 1200
 $Comp
-L +24V #PWR050
+L +24V #PWR051
 U 1 1 58AF1DD3
 P 2150 950
-F 0 "#PWR050" H 2150 800 50  0001 C CNN
+F 0 "#PWR051" H 2150 800 50  0001 C CNN
 F 1 "+24V" H 2150 1090 50  0000 C CNN
 F 2 "" H 2150 950 50  0000 C CNN
@@
 LV_RTN
 $Comp
-L +5V #PWR051
+L +5V #PWR052
 U 1 1 58AF2067
 P 5350 900
-F 0 "#PWR051" H 5350 750 50  0001 C CNN
+F 0 "#PWR052" H 5350 750 50  0001 C CNN
 F 1 "+5V" H 5350 1040 50  0000 C CNN
 F 2 "" H 5350 900 50  0000 C CNN
@@
 $EndComp
 $Comp
-L GND #PWR052
+L GND #PWR053
 U 1 1 58B9D18E
 P 5900 1350
-F 0 "#PWR052" H 5900 1100 50  0001 C CNN
+F 0 "#PWR053" H 5900 1100 50  0001 C CNN
 F 1 "GND" H 5900 1200 50  0000 C CNN
 F 2 "" H 5900 1350 50  0000 C CNN
@@
 $EndComp
 $Comp
-L +5V #PWR053
+L +5V #PWR054
 U 1 1 58B9D1D5
 P 5900 850
-F 0 "#PWR053" H 5900 700 50  0001 C CNN
+F 0 "#PWR054" H 5900 700 50  0001 C CNN
 F 1 "+5V" H 5900 990 50  0000 C CNN
 F 2 "" H 5900 850 50  0000 C CNN
@@
 	5900 1350 5900 1250
 $Comp
-L GND #PWR054
+L GND #PWR055
 U 1 1 58D1E1EA
 P 5350 1300
-F 0 "#PWR054" H 5350 1050 50  0001 C CNN
+F 0 "#PWR055" H 5350 1050 50  0001 C CNN
 F 1 "GND" H 5350 1150 50  0000 C CNN
 F 2 "" H 5350 1300 50  0000 C CNN
@@
 	1    0    0    -1
 $EndComp
+$Comp
+L TEST_1P W?
+U 1 1 58D4724A
+P 5050 900
+F 0 "W?" H 5050 1170 50  0000 C CNN
+F 1 "+5DC/DC" H 5050 1100 50  0000 C CNN
+F 2 "Measurement_Points:Measurement_Point_Round-SMD-Pad_Big" H 5250 900 50  0001 C CNN
+F 3 "" H 5250 900 50  0000 C CNN
+	1    5050 900
+	1    0    0    -1
+$EndComp
+Wire Wire Line
+	5050 1000 5050 900
+Connection ~ 5050 1000
+$Comp
+L TEST_1P W?
+U 1 1 58D4731B
+P 5000 1300
+F 0 "W?" H 5000 1570 50  0000 C CNN
+F 1 "+5DC/DC_GND" H 5000 1500 50  0000 C CNN
+F 2 "Measurement_Points:Measurement_Point_Square-SMD-Pad_Big" H 5200 1300 50  0001 C CNN
+F 3 "" H 5200 1300 50  0000 C CNN
+	1    5000 1300
+	-1   0    0    1
+$EndComp
+Wire Wire Line
+	5000 1300 5000 1200
+Connection ~ 5000 1200
 $EndSCHEMATC

Commit message: cleaned up footprints of more testpoints. ran DRC again, passed
Parts:
- gave numbers to parts that had none: 2
Changed lines of the file:
@@
 NoConn ~ 3450 1200
 $Comp
-L +24V #PWR051
+L +24V #PWR049
 U 1 1 58AF1DD3
 P 2150 950
-F 0 "#PWR051" H 2150 800 50  0001 C CNN
+F 0 "#PWR049" H 2150 800 50  0001 C CNN
 F 1 "+24V" H 2150 1090 50  0000 C CNN
 F 2 "" H 2150 950 50  0000 C CNN
@@
 LV_RTN
 $Comp
-L +5V #PWR052
+L +5V #PWR050
 U 1 1 58AF2067
 P 5350 900
-F 0 "#PWR052" H 5350 750 50  0001 C CNN
+F 0 "#PWR050" H 5350 750 50  0001 C CNN
 F 1 "+5V" H 5350 1040 50  0000 C CNN
 F 2 "" H 5350 900 50  0000 C CNN
@@
 $EndComp
 $Comp
-L GND #PWR053
+L GND #PWR051
 U 1 1 58B9D18E
 P 5900 1350
-F 0 "#PWR053" H 5900 1100 50  0001 C CNN
+F 0 "#PWR051" H 5900 1100 50  0001 C CNN
 F 1 "GND" H 5900 1200 50  0000 C CNN
 F 2 "" H 5900 1350 50  0000 C CNN
@@
 $EndComp
 $Comp
-L +5V #PWR054
+L +5V #PWR052
 U 1 1 58B9D1D5
 P 5900 850
-F 0 "#PWR054" H 5900 700 50  0001 C CNN
+F 0 "#PWR052" H 5900 700 50  0001 C CNN
 F 1 "+5V" H 5900 990 50  0000 C CNN
 F 2 "" H 5900 850 50  0000 C CNN
@@
 	5900 1350 5900 1250
 $Comp
-L GND #PWR055
+L GND #PWR053
 U 1 1 58D1E1EA
 P 5350 1300
-F 0 "#PWR055" H 5350 1050 50  0001 C CNN
+F 0 "#PWR053" H 5350 1050 50  0001 C CNN
 F 1 "GND" H 5350 1150 50  0000 C CNN
 F 2 "" H 5350 1300 50  0000 C CNN
@@
 $EndComp
 $Comp
-L TEST_1P W?
+L TEST_1P W22
 U 1 1 58D4724A
 P 5050 900
-F 0 "W?" H 5050 1170 50  0000 C CNN
+F 0 "W22" H 5050 1170 50  0000 C CNN
 F 1 "+5DC/DC" H 5050 1100 50  0000 C CNN
 F 2 "Measurement_Points:Measurement_Point_Round-SMD-Pad_Big" H 5250 900 50  0001 C CNN
@@
 Connection ~ 5050 1000
 $Comp
-L TEST_1P W?
+L TEST_1P W21
 U 1 1 58D4731B
 P 5000 1300
-F 0 "W?" H 5000 1570 50  0000 C CNN
+F 0 "W21" H 5000 1570 50  0000 C CNN
 F 1 "+5DC/DC_GND" H 5000 1500 50  0000 C CNN
 F 2 "Measurement_Points:Measurement_Point_Square-SMD-Pad_Big" H 5200 1300 50  0001 C CNN
