File: Circuit_layout/StatusLights.sch (KiCad schematic (older format))
At the start: 17 parts

Commit message: KiCad BOM
Parts:
- U11, U12: renamed from U?; Field5 http://www.digikey.com/product-detail/en/toshiba-semiconduc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 -> (none); Man P/N TLP293(GB-TPL,E -> TLP293(GB-TPLE; URL (none) -> http://www.digikey.com/product-detail/en/toshiba-semiconduc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
- gave numbers to parts that had none: 15
Changed lines of the file:
@@
 EESchema Schematic File Version 2
 LIBS:Circuit_layout-rescue
+LIBS:TSI_KiCad_Lib
 LIBS:TSI_HV_Isolater-cache
 LIBS:74xgxx
@@
 Comp "Lafayette College"
 Comment1 "Spring 2017"
-Comment2 "Jack Plumb"
+Comment2 "Jack Plumb and Adam Ness"
 Comment3 ""
 Comment4 "DEVELOPMENT ONLY"
 $EndDescr
 $Comp
-L TLP291 U?
+L TLP291 U12
 U 1 1 58AF31A2
 P 5450 1950
-F 0 "U?" H 5250 2150 50  0000 L CNN
+F 0 "U12" H 5250 2150 50  0000 L CNN
 F 1 "TLP293" H 5450 2150 50  0000 L CNN
 F 2 "SOP-4" H 5250 1750 50  0000 L CIN
 F 3 "" H 5450 1950 50  0000 L CNN
 F 4 "TLP293(GB-TPLECT-ND" H 5450 1950 60  0001 C CNN "DigiKey P/N"
-F 5 "http://www.digikey.com/product-detail/en/toshiba-semiconductor-and-storage/TLP293(GB-TPL,E/TLP293(GB-TPLECT-ND/4562965" H 5450 1950 60  0001 C CNN "Field5"
-F 6 "TLP293(GB-TPL,E" H 5450 1950 60  0001 C CNN "Man P/N"
+F 5 "http://www.digikey.com/product-detail/en/toshiba-semiconductor-and-storage/TLP293(GB-TPL,E/TLP293(GB-TPLECT-ND/4562965" H 5450 1950 60  0001 C CNN "URL"
+F 6 "TLP293(GB-TPLE" H 5450 1950 60  0001 C CNN "Man P/N"
 F 7 "http://www.digikey.com/product-detail/en/toshiba-semiconductor-and-storage/TLP291(GB-TP,SE/TLP291(GB-TPSECT-ND/4562949" H 5450 1950 60  0001 C CNN "TLP291"
 	1    5450 1950
@@
 	5150 1850 4900 1850
 $Comp
-L R R?
+L R R14
 U 1 1 58AF3371
 P 4750 1850
-F 0 "R?" V 4830 1850 50  0000 C CNN
+F 0 "R14" V 4830 1850 50  0000 C CNN
 F 1 "150" V 4750 1850 50  0000 C CNN
 F 2 "" V 4680 1850 50  0000 C CNN
@@
 	5050 2050 5050 2150
 $Comp
-L GND #PWR?
+L GND #PWR021
 U 1 1 58AF33D9
 P 5050 2150
-F 0 "#PWR?" H 5050 1900 50  0001 C CNN
+F 0 "#PWR021" H 5050 1900 50  0001 C CNN
 F 1 "GND" H 5050 2000 50  0000 C CNN
 F 2 "" H 5050 2150 50  0000 C CNN
@@
 	5750 1850 6050 1850
 $Comp
-L +24V #PWR?
+L +24V #PWR022
 U 1 1 58AF3526
 P 6450 1700
-F 0 "#PWR?" H 6450 1550 50  0001 C CNN
+F 0 "#PWR022" H 6450 1550 50  0001 C CNN
 F 1 "+24V" H 6450 1840 50  0000 C CNN
 F 2 "" H 6450 1700 50  0000 C CNN
@@
 RTDS
 $Comp
-L TLP291 U?
+L TLP291 U11
 U 1 1 58AF4260
 P 5400 3100
-F 0 "U?" H 5200 3300 50  0000 L CNN
+F 0 "U11" H 5200 3300 50  0000 L CNN
 F 1 "TLP293" H 5400 3300 50  0000 L CNN
 F 2 "SOP-4" H 5200 2900 50  0000 L CIN
 F 3 "" H 5400 3100 50  0000 L CNN
 F 4 "TLP293(GB-TPLECT-ND" H 5400 3100 60  0001 C CNN "DigiKey P/N"
-F 5 "http://www.digikey.com/product-detail/en/toshiba-semiconductor-and-storage/TLP293(GB-TPL,E/TLP293(GB-TPLECT-ND/4562965" H 5400 3100 60  0001 C CNN "Field5"
-F 6 "TLP293(GB-TPL,E" H 5400 3100 60  0001 C CNN "Man P/N"
+F 5 "http://www.digikey.com/product-detail/en/toshiba-semiconductor-and-storage/TLP293(GB-TPL,E/TLP293(GB-TPLECT-ND/4562965" H 5400 3100 60  0001 C CNN "URL"
+F 6 "TLP293(GB-TPLE" H 5400 3100 60  0001 C CNN "Man P/N"
 F 7 "http://www.digikey.com/product-detail/en/toshiba-semiconductor-and-storage/TLP291(GB-TP,SE/TLP291(GB-TPSECT-ND/4562949" H 5400 3100 60  0001 C CNN "TLP291"
 	1    5400 3100
@@
 	5050 3200 5050 3300
 $Comp
-L GND #PWR?
+L GND #PWR023
 U 1 1 58AF4273
 P 5050 3300
-F 0 "#PWR?" H 5050 3050 50  0001 C CNN
+F 0 "#PWR023" H 5050 3050 50  0001 C CNN
 F 1 "GND" H 5050 3150 50  0000 C CNN
 F 2 "" H 5050 3300 50  0000 C CNN
@@
 	5700 3000 6000 3000
 $Comp
-L +24V #PWR?
+L +24V #PWR024
 U 1 1 58AF427B
 P 6450 2850
-F 0 "#PWR?" H 6450 2700 50  0001 C CNN
+F 0 "#PWR024" H 6450 2700 50  0001 C CNN
 F 1 "+24V" H 6450 2990 50  0000 C CNN
 F 2 "" H 6450 2850 50  0000 C CNN
@@
 Drive_LED
 $Comp
-L R R?
+L R R12
 U 1 1 58AF4E42
 P 4700 3000
-F 0 "R?" V 4780 3000 50  0000 C CNN
+F 0 "R12" V 4780 3000 50  0000 C CNN
 F 1 "150" V 4700 3000 50  0000 C CNN
 F 2 "" V 4630 3000 50  0000 C CNN
@@
 $EndComp
 $Comp
-L R R?
+L R R16
 U 1 1 58AF50A8
 P 6150 3000
-F 0 "R?" V 6230 3000 50  0000 C CNN
+F 0 "R16" V 6230 3000 50  0000 C CNN
 F 1 "2k" V 6150 3000 50  0000 C CNN
 F 2 "" V 6080 3000 50  0000 C CNN
@@
 	6450 3000 6450 2850
 $Comp
-L R R?
+L R R17
 U 1 1 58AF51A7
 P 6200 1850
-F 0 "R?" V 6280 1850 50  0000 C CNN
+F 0 "R17" V 6280 1850 50  0000 C CNN
 F 1 "2k" V 6200 1850 50  0000 C CNN
 F 2 "" V 6130 1850 50  0000 C CNN
@@
 RTDS_CTRL
 $Comp
-L R R?
+L R R15
 U 1 1 58B1EEB2
 P 5300 4350
-F 0 "R?" V 5380 4350 50  0000 C CNN
+F 0 "R15" V 5380 4350 50  0000 C CNN
 F 1 "DNP" V 5300 4350 50  0000 C CNN
 F 2 "Resistors_SMD:R_0805_HandSoldering" V 5230 4350 50  0001 C CNN
@@
 Confirm sizing of R:\nDatasheet lists 10mA/220mA as current draw of light.\nDesign for max?
 $Comp
-L MMBF170 Q?
+L MMBF170 Q1
 U 1 1 58B25E37
 P 5200 4950
-F 0 "Q?" H 5400 5025 50  0000 L CNN
+F 0 "Q1" H 5400 5025 50  0000 L CNN
 F 1 "MMBF170" H 5400 4950 50  0000 L CNN
 F 2 "SOT-23" H 5400 4875 50  0000 L CIN
@@
 $EndComp
 $Comp
-L R R?
+L R R18
 U 1 1 58B266DE
 P 9850 1800
-F 0 "R?" V 9930 1800 50  0000 C CNN
+F 0 "R18" V 9930 1800 50  0000 C CNN
 F 1 "1k" V 9850 1800 50  0000 C CNN
 F 2 "Resistors_SMD:R_0805_HandSoldering" V 9780 1800 50  0001 C CNN
@@
 $EndComp
 $Comp
-L LED D?
+L LED D1
 U 1 1 58B26743
 P 9300 1800
-F 0 "D?" H 9300 1900 50  0000 C CNN
+F 0 "D1" H 9300 1900 50  0000 C CNN
 F 1 "Power" H 9300 1700 50  0000 C CNN
 F 2 "LEDs:LED_0805" H 9300 1800 50  0001 C CNN
@@
 	8800 1800 8800 1900
 $Comp
-L GND #PWR?
+L GND #PWR025
 U 1 1 58B26825
 P 8800 1900
-F 0 "#PWR?" H 8800 1650 50  0001 C CNN
+F 0 "#PWR025" H 8800 1650 50  0001 C CNN
 F 1 "GND" H 8800 1750 50  0000 C CNN
 F 2 "" H 8800 1900 50  0000 C CNN
@@
 Green
 $Comp
-L LED D?
+L LED D2
 U 1 1 58B26F44
 P 9300 2250
-F 0 "D?" H 9300 2350 50  0000 C CNN
+F 0 "D2" H 9300 2350 50  0000 C CNN
 F 1 "Heartbeat" H 9300 2150 50  0000 C CNN
 F 2 "LEDs:LED_0805" H 9300 2250 50  0001 C CNN
@@
 	8800 2250 8800 2350
 $Comp
-L GND #PWR?
+L GND #PWR026
 U 1 1 58B26F4E
 P 8800 2350
-F 0 "#PWR?" H 8800 2100 50  0001 C CNN
+F 0 "#PWR026" H 8800 2100 50  0001 C CNN
 F 1 "GND" H 8800 2200 50  0000 C CNN
 F 2 "" H 8800 2350 50  0000 C CNN
@@
 Yellow
 $Comp
-L LED D?
+L LED D3
 U 1 1 58B272A0
 P 9300 2700
-F 0 "D?" H 9300 2800 50  0000 C CNN
+F 0 "D3" H 9300 2800 50  0000 C CNN
 F 1 "Spare/Fault" H 9300 2600 50  0000 C CNN
 F 2 "LEDs:LED_0805" H 9300 2700 50  0001 C CNN
@@
 	8800 2700 8800 2800
 $Comp
-L GND #PWR?
+L GND #PWR027
 U 1 1 58B272AA
 P 8800 2800
-F 0 "#PWR?" H 8800 2550 50  0001 C CNN
+F 0 "#PWR027" H 8800 2550 50  0001 C CNN
 F 1 "GND" H 8800 2650 50  0000 C CNN
 F 2 "" H 8800 2800 50  0000 C CNN
@@
 Red
 $Comp
-L LED D?
+L LED D4
 U 1 1 58B27326
 P 9300 3150
-F 0 "D?" H 9300 3250 50  0000 C CNN
+F 0 "D4" H 9300 3250 50  0000 C CNN
 F 1 "Power" H 9300 3050 50  0000 C CNN
 F 2 "LEDs:LED_0805" H 9300 3150 50  0001 C CNN
@@
 	8800 3150 8800 3250
 $Comp
-L GND #PWR?
+L GND #PWR028
 U 1 1 58B27330
 P 8800 3250
-F 0 "#PWR?" H 8800 3000 50  0001 C CNN
+F 0 "#PWR028" H 8800 3000 50  0001 C CNN
 F 1 "GND" H 8800 3100 50  0000 C CNN
 F 2 "" H 8800 3250 50  0000 C CNN
@@
 Blue
 $Comp
-L R R?
+L R R19
 U 1 1 58B27F91
 P 9850 2250
-F 0 "R?" V 9930 2250 50  0000 C CNN
+F 0 "R19" V 9930 2250 50  0000 C CNN
 F 1 "1k" V 9850 2250 50  0000 C CNN
 F 2 "Resistors_SMD:R_0805_HandSoldering" V 9780 2250 50  0001 C CNN
@@
 $EndComp
 $Comp
-L R R?
+L R R20
 U 1 1 58B27FEF
 P 9850 2700
-F 0 "R?" V 9930 2700 50  0000 C CNN
+F 0 "R20" V 9930 2700 50  0000 C CNN
 F 1 "1k" V 9850 2700 50  0000 C CNN
 F 2 "Resistors_SMD:R_0805_HandSoldering" V 9780 2700 50  0001 C CNN
@@
 $EndComp
 $Comp
-L R R?
+L R R21
 U 1 1 58B28050
 P 9850 3150
-F 0 "R?" V 9930 3150 50  0000 C CNN
+F 0 "R21" V 9930 3150 50  0000 C CNN
 F 1 "1k" V 9850 3150 50  0000 C CNN
 F 2 "Resistors_SMD:R_0805_HandSoldering" V 9780 3150 50  0001 C CNN
@@
 $EndComp
 $Comp
-L +5V #PWR?
+L +5V #PWR029
 U 1 1 58B2809B
 P 10300 1800
-F 0 "#PWR?" H 10300 1650 50  0001 C CNN
+F 0 "#PWR029" H 10300 1650 50  0001 C CNN
 F 1 "+5V" H 10300 1940 50  0000 C CNN
 F 2 "" H 10300 1800 50  0000 C CNN
@@
 Text Notes 8800 1500 0    99   ~ 0
 Status/Debug LEDs
-Text Notes 7250 3600 0    60   ~ 0
+Text Notes 7300 3550 0    60   ~ 0
 Can these resistors be internal pull-down/pull-up resistors in the microcontroller?
 $Comp
-L GND #PWR?
+L GND #PWR030
 U 1 1 58B21DFD
 P 5300 5350
-F 0 "#PWR?" H 5300 5100 50  0001 C CNN
+F 0 "#PWR030" H 5300 5100 50  0001 C CNN
 F 1 "GND" H 5300 5200 50  0000 C CNN
 F 2 "" H 5300 5350 50  0000 C CNN
@@
 Brake_Light
 $Comp
-L +12V #PWR?
+L +12V #PWR031
 U 1 1 58B22590
 P 5300 3950
-F 0 "#PWR?" H 5300 3800 50  0001 C CNN
+F 0 "#PWR031" H 5300 3800 50  0001 C CNN
 F 1 "+12V" H 5300 4090 50  0000 C CNN
 F 2 "" H 5300 3950 50  0000 C CNN
@@
 $EndComp
 $Comp
-L R R?
+L R R13
 U 1 1 58B5DC19
 P 4700 5000
-F 0 "R?" V 4780 5000 50  0000 C CNN
+F 0 "R13" V 4780 5000 50  0000 C CNN
 F 1 "1k" V 4700 5000 50  0000 C CNN
 F 2 "Resistors_SMD:R_0805_HandSoldering" V 4630 5000 50  0001 C CNN

Commit message: finished adding footprints/info to all parts that I can
Parts:
- removed Q1: MMBF170, SOT-23, symbol MMBF170
- removed R14: 150, symbol R
- removed R15: DNP, Resistors_SMD:R_0805_HandSoldering, symbol R
- removed R17: 2k, symbol R
- added Q?: MMBF170, TO_SOT_Packages_SMD:SOT-23, symbol MMBF170
- added R? (x2): 150, Resistors_SMD:R_0805_HandSoldering, symbol R
- added R?: 2k, Resistors_SMD:R_0805_HandSoldering, symbol R
- R12, R16: footprint (none) -> Resistors_SMD:R_0805_HandSoldering
Connections:
- net +12V: now also R?.2
- net +24V: now also R?.1
- net Brake_Light: now also Q?.3 (D), R?.1
- net GND: now also Q?.2 (S)
- net RTDS_CTRL: now also R?.2
- net at U12.1: now also R?.1
- net at U12.4: now also R?.2
- net at R13.1: now also Q?.1 (G)
Other:
- note added: "Confirm sizing of R:\nDatasheet lists 10mA/220mA as current draw of light.\nDesign for max? Currently roughly 80mA"
- note removed: "Confirm sizing of R:\nDatasheet lists 10mA/220mA as current draw of light.\nDesign for max?"
Changed lines of the file:
@@
 EESchema Schematic File Version 2
 LIBS:Circuit_layout-rescue
-LIBS:TSI_KiCad_Lib
 LIBS:TSI_HV_Isolater-cache
 LIBS:74xgxx
@@
 Wire Wire Line
 	5150 1850 4900 1850
-$Comp
-L R R14
-U 1 1 58AF3371
-P 4750 1850
-F 0 "R14" V 4830 1850 50  0000 C CNN
-F 1 "150" V 4750 1850 50  0000 C CNN
-F 2 "" V 4680 1850 50  0000 C CNN
-F 3 "" H 4750 1850 50  0000 C CNN
-F 4 "311-150CRCT-ND" V 4750 1850 60  0001 C CNN "DigiKey P/N"
-F 5 "http://www.digikey.com/product-detail/en/yageo/RC0805FR-07150RL/311-150CRCT-ND/730560" V 4750 1850 60  0001 C CNN "URL"
-F 6 "RC0805FR-07150RL" V 4750 1850 60  0001 C CNN "Man P/N"
-	1    4750 1850
-	0    1    1    0
-$EndComp
 Wire Wire Line
 	5050 2050 5050 2150
@@
 F 0 "R12" V 4780 3000 50  0000 C CNN
 F 1 "150" V 4700 3000 50  0000 C CNN
-F 2 "" V 4630 3000 50  0000 C CNN
+F 2 "Resistors_SMD:R_0805_HandSoldering" V 4630 3000 50  0001 C CNN
 F 3 "" H 4700 3000 50  0000 C CNN
 F 4 "311-150CRCT-ND" V 4700 3000 60  0001 C CNN "DigiKey P/N"
@@
 F 0 "R16" V 6230 3000 50  0000 C CNN
 F 1 "2k" V 6150 3000 50  0000 C CNN
-F 2 "" V 6080 3000 50  0000 C CNN
+F 2 "Resistors_SMD:R_0805_HandSoldering" V 6080 3000 50  0001 C CNN
 F 3 "" H 6150 3000 50  0000 C CNN
 F 4 "P2.00KCCT-ND" V 6150 3000 60  0001 C CNN "DigiKey P/N"
@@
 Wire Wire Line
 	6450 3000 6450 2850
-$Comp
-L R R17
-U 1 1 58AF51A7
-P 6200 1850
-F 0 "R17" V 6280 1850 50  0000 C CNN
-F 1 "2k" V 6200 1850 50  0000 C CNN
-F 2 "" V 6130 1850 50  0000 C CNN
-F 3 "" H 6200 1850 50  0000 C CNN
-F 4 "P2.00KCCT-ND" V 6200 1850 60  0001 C CNN "DigiKey P/N"
-F 5 "http://www.digikey.com/product-detail/en/panasonic-electronic-components/ERJ-6ENF2001V/P2.00KCCT-ND/119044" V 6200 1850 60  0001 C CNN "URL"
-F 6 "ERJ-6ENF2001V" V 6200 1850 60  0001 C CNN "Man P/N"
-	1    6200 1850
-	0    1    1    0
-$EndComp
 Wire Wire Line
 	6350 1850 6450 1850
@@
 Text HLabel 4100 1850 0    60   Input ~ 0
 RTDS_CTRL
-$Comp
-L R R15
-U 1 1 58B1EEB2
-P 5300 4350
-F 0 "R15" V 5380 4350 50  0000 C CNN
-F 1 "DNP" V 5300 4350 50  0000 C CNN
-F 2 "Resistors_SMD:R_0805_HandSoldering" V 5230 4350 50  0001 C CNN
-F 3 "" H 5300 4350 50  0000 C CNN
-	1    5300 4350
-	-1   0    0    1
-$EndComp
 Wire Wire Line
 	5300 4750 5300 4500
@@
 Wire Wire Line
 	5300 5150 5300 5350
-Text Label 3950 5000 0    60   ~ 0
-BP_uC
 Text Notes 5450 4500 0    60   ~ 0
-Confirm sizing of R:\nDatasheet lists 10mA/220mA as current draw of light.\nDesign for max?
-$Comp
-L MMBF170 Q1
-U 1 1 58B25E37
-P 5200 4950
-F 0 "Q1" H 5400 5025 50  0000 L CNN
-F 1 "MMBF170" H 5400 4950 50  0000 L CNN
-F 2 "SOT-23" H 5400 4875 50  0000 L CIN
-F 3 "" H 5200 4950 50  0000 L CNN
-	1    5200 4950
-	1    0    0    -1
-$EndComp
+Confirm sizing of R:\nDatasheet lists 10mA/220mA as current draw of light.\nDesign for max? Currently roughly 80mA
 $Comp
 L R R18
@@
 	5300 4700 5850 4700
 Connection ~ 5300 4700
-Text Label 5850 4700 0    60   ~ 0
-Brake_Light
 $Comp
 L +12V #PWR031
@@
 	0    1    1    0
 $EndComp
+$Comp
+L MMBF170 Q?
+U 1 1 58B375B3
+P 5200 4950
+F 0 "Q?" H 5400 5025 50  0000 L CNN
+F 1 "MMBF170" H 5400 4950 50  0000 L CNN
+F 2 "TO_SOT_Packages_SMD:SOT-23" H 5400 4875 50  0001 L CIN
+F 3 "https://www.fairchildsemi.com/datasheets/MM/MMBF170.pdf" H 5200 4950 50  0001 L CNN
+F 4 "MMBF170CT-ND" H 5200 4950 60  0001 C CNN "Digikey P/N"
+F 5 "http://www.digikey.com/product-detail/en/fairchild-on-semiconductor/MMBF170/MMBF170CT-ND/244295" H 5200 4950 60  0001 C CNN "URL"
+F 6 "MMBF170" H 5200 4950 60  0001 C CNN "Man P/N"
+	1    5200 4950
+	1    0    0    -1
+$EndComp
+$Comp
+L R R?
+U 1 1 58B384ED
+P 5300 4350
+F 0 "R?" V 5380 4350 50  0000 C CNN
+F 1 "150" V 5300 4350 50  0000 C CNN
+F 2 "Resistors_SMD:R_0805_HandSoldering" V 5230 4350 50  0001 C CNN
+F 3 "" H 5300 4350 50  0000 C CNN
+F 4 "311-150CRCT-ND" V 5300 4350 60  0001 C CNN "DigiKey P/N"
+F 5 "http://www.digikey.com/product-detail/en/yageo/RC0805FR-07150RL/311-150CRCT-ND/730560" V 5300 4350 60  0001 C CNN "URL"
+F 6 "RC0805FR-07150RL" V 5300 4350 60  0001 C CNN "Man P/N"
+	1    5300 4350
+	-1   0    0    1
+$EndComp
+$Comp
+L R R?
+U 1 1 58B38BE5
+P 4750 1850
+F 0 "R?" V 4830 1850 50  0000 C CNN
+F 1 "150" V 4750 1850 50  0000 C CNN
+F 2 "Resistors_SMD:R_0805_HandSoldering" V 4680 1850 50  0001 C CNN
+F 3 "" H 4750 1850 50  0000 C CNN
+F 4 "311-150CRCT-ND" V 4750 1850 60  0001 C CNN "DigiKey P/N"
+F 5 "http://www.digikey.com/product-detail/en/yageo/RC0805FR-07150RL/311-150CRCT-ND/730560" V 4750 1850 60  0001 C CNN "URL"
+F 6 "RC0805FR-07150RL" V 4750 1850 60  0001 C CNN "Man P/N"
+	1    4750 1850
+	0    1    1    0
+$EndComp
+$Comp
+L R R?
+U 1 1 58B38C61
+P 6200 1850
+F 0 "R?" V 6280 1850 50  0000 C CNN
+F 1 "2k" V 6200 1850 50  0000 C CNN
+F 2 "Resistors_SMD:R_0805_HandSoldering" V 6130 1850 50  0001 C CNN
+F 3 "" H 6200 1850 50  0000 C CNN
+F 4 "P2.00KCCT-ND" V 6200 1850 60  0001 C CNN "DigiKey P/N"
+F 5 "http://www.digikey.com/product-detail/en/panasonic-electronic-components/ERJ-6ENF2001V/P2.00KCCT-ND/119044" V 6200 1850 60  0001 C CNN "URL"
+F 6 "ERJ-6ENF2001V" V 6200 1850 60  0001 C CNN "Man P/N"
+	1    6200 1850
+	0    1    1    0
+$EndComp
+Text HLabel 3950 5000 0    60   Input ~ 0
+BP_uC
+Text HLabel 5850 4700 2    60   Output ~ 0
+Brake_Light
 $EndSCHEMATC

Commit message: took notes w/ greg
Parts:
- gave numbers to parts that had none: 4
Other:
- note added: "Make 100ohm"
- note removed: "Can these resistors be internal pull-down/pull-up resistors in the microcontroller?"
Changed lines of the file:
@@
 	5050 2050 5050 2150
 $Comp
-L GND #PWR021
+L GND #PWR025
 U 1 1 58AF33D9
 P 5050 2150
-F 0 "#PWR021" H 5050 1900 50  0001 C CNN
+F 0 "#PWR025" H 5050 1900 50  0001 C CNN
 F 1 "GND" H 5050 2000 50  0000 C CNN
 F 2 "" H 5050 2150 50  0000 C CNN
@@
 	5750 1850 6050 1850
 $Comp
-L +24V #PWR022
+L +24V #PWR026
 U 1 1 58AF3526
 P 6450 1700
-F 0 "#PWR022" H 6450 1550 50  0001 C CNN
+F 0 "#PWR026" H 6450 1550 50  0001 C CNN
 F 1 "+24V" H 6450 1840 50  0000 C CNN
 F 2 "" H 6450 1700 50  0000 C CNN
@@
 	5050 3200 5050 3300
 $Comp
-L GND #PWR023
+L GND #PWR027
 U 1 1 58AF4273
 P 5050 3300
-F 0 "#PWR023" H 5050 3050 50  0001 C CNN
+F 0 "#PWR027" H 5050 3050 50  0001 C CNN
 F 1 "GND" H 5050 3150 50  0000 C CNN
 F 2 "" H 5050 3300 50  0000 C CNN
@@
 	5700 3000 6000 3000
 $Comp
-L +24V #PWR024
+L +24V #PWR028
 U 1 1 58AF427B
 P 6450 2850
-F 0 "#PWR024" H 6450 2700 50  0001 C CNN
+F 0 "#PWR028" H 6450 2700 50  0001 C CNN
 F 1 "+24V" H 6450 2990 50  0000 C CNN
 F 2 "" H 6450 2850 50  0000 C CNN
@@
 	8800 1800 8800 1900
 $Comp
-L GND #PWR025
+L GND #PWR029
 U 1 1 58B26825
 P 8800 1900
-F 0 "#PWR025" H 8800 1650 50  0001 C CNN
+F 0 "#PWR029" H 8800 1650 50  0001 C CNN
 F 1 "GND" H 8800 1750 50  0000 C CNN
 F 2 "" H 8800 1900 50  0000 C CNN
@@
 	8800 2250 8800 2350
 $Comp
-L GND #PWR026
+L GND #PWR030
 U 1 1 58B26F4E
 P 8800 2350
-F 0 "#PWR026" H 8800 2100 50  0001 C CNN
+F 0 "#PWR030" H 8800 2100 50  0001 C CNN
 F 1 "GND" H 8800 2200 50  0000 C CNN
 F 2 "" H 8800 2350 50  0000 C CNN
@@
 	8800 2700 8800 2800
 $Comp
-L GND #PWR027
+L GND #PWR031
 U 1 1 58B272AA
 P 8800 2800
-F 0 "#PWR027" H 8800 2550 50  0001 C CNN
+F 0 "#PWR031" H 8800 2550 50  0001 C CNN
 F 1 "GND" H 8800 2650 50  0000 C CNN
 F 2 "" H 8800 2800 50  0000 C CNN
@@
 	8800 3150 8800 3250
 $Comp
-L GND #PWR028
+L GND #PWR032
 U 1 1 58B27330
 P 8800 3250
-F 0 "#PWR028" H 8800 3000 50  0001 C CNN
+F 0 "#PWR032" H 8800 3000 50  0001 C CNN
 F 1 "GND" H 8800 3100 50  0000 C CNN
 F 2 "" H 8800 3250 50  0000 C CNN
@@
 $EndComp
 $Comp
-L +5V #PWR029
+L +5V #PWR033
 U 1 1 58B2809B
 P 10300 1800
-F 0 "#PWR029" H 10300 1650 50  0001 C CNN
+F 0 "#PWR033" H 10300 1650 50  0001 C CNN
 F 1 "+5V" H 10300 1940 50  0000 C CNN
 F 2 "" H 10300 1800 50  0000 C CNN
@@
 Text Notes 8800 1500 0    99   ~ 0
 Status/Debug LEDs
-Text Notes 7300 3550 0    60   ~ 0
-Can these resistors be internal pull-down/pull-up resistors in the microcontroller?
-$Comp
-L GND #PWR030
+Text Notes 9800 3550 0    60   ~ 0
+Make 100ohm
+$Comp
+L GND #PWR034
 U 1 1 58B21DFD
 P 5300 5350
-F 0 "#PWR030" H 5300 5100 50  0001 C CNN
+F 0 "#PWR034" H 5300 5100 50  0001 C CNN
 F 1 "GND" H 5300 5200 50  0000 C CNN
 F 2 "" H 5300 5350 50  0000 C CNN
@@
 Connection ~ 5300 4700
 $Comp
-L +12V #PWR031
+L +12V #PWR035
 U 1 1 58B22590
 P 5300 3950
-F 0 "#PWR031" H 5300 3800 50  0001 C CNN
+F 0 "#PWR035" H 5300 3800 50  0001 C CNN
 F 1 "+12V" H 5300 4090 50  0000 C CNN
 F 2 "" H 5300 3950 50  0000 C CNN
@@
 $EndComp
 $Comp
-L MMBF170 Q?
+L MMBF170 Q1
 U 1 1 58B375B3
 P 5200 4950
-F 0 "Q?" H 5400 5025 50  0000 L CNN
+F 0 "Q1" H 5400 5025 50  0000 L CNN
 F 1 "MMBF170" H 5400 4950 50  0000 L CNN
 F 2 "TO_SOT_Packages_SMD:SOT-23" H 5400 4875 50  0001 L CIN
@@
 $EndComp
 $Comp
-L R R?
+L R R17
 U 1 1 58B384ED
 P 5300 4350
-F 0 "R?" V 5380 4350 50  0000 C CNN
+F 0 "R17" V 5380 4350 50  0000 C CNN
 F 1 "150" V 5300 4350 50  0000 C CNN
 F 2 "Resistors_SMD:R_0805_HandSoldering" V 5230 4350 50  0001 C CNN
@@
 $EndComp
 $Comp
-L R R?
+L R R15
 U 1 1 58B38BE5
 P 4750 1850
-F 0 "R?" V 4830 1850 50  0000 C CNN
+F 0 "R15" V 4830 1850 50  0000 C CNN
 F 1 "150" V 4750 1850 50  0000 C CNN
 F 2 "Resistors_SMD:R_0805_HandSoldering" V 4680 1850 50  0001 C CNN
@@
 $EndComp
 $Comp
-L R R?
+L R R35
 U 1 1 58B38C61
 P 6200 1850
-F 0 "R?" V 6280 1850 50  0000 C CNN
+F 0 "R35" V 6280 1850 50  0000 C CNN
 F 1 "2k" V 6200 1850 50  0000 C CNN
 F 2 "Resistors_SMD:R_0805_HandSoldering" V 6130 1850 50  0001 C CNN
