File: Circuit_layout/Circuit_layout.kicad_pcb (KiCad board)
At the start: 2 copper layers, 203.2 x 152.4 mm, 193 parts, among them CON1 AVR-JTAG-10, J1 Spare_Conns, J10 AIRs, J3 CAN, J4 Motor_Ctrl, J5 RJ12, P1 TSV, P2 HVPL, P3 IMD, P4 GLV, P5 Cockpit, P6 Pedals, P7 RTDS, Q1 ZVP4525G, Q2 MMBF170, Q3 MMBF170, SW1 SW_PUSH, SW2 TS5A3159-Q1, SW3 JS202011CQN, U1 PDM2-S24-S12, U10 MCP2551-I/SN, U11 TLP293, U12 TLP293, U13 PDQ10-D, U15 TLP293, U16 LTC3638, U17 MCP6004, U18 TS912, U19 ACPL-C870, U2 MCP6002, U20 ACPL-C870, U21 MCP6001, U22 TS372, U23 TLP293, U24 TLP293, U3 MCP6004, U5 LM7810CT, U6 TS912, U7 AT90CAN128-A, U8 74ACT11030, U9 TLP293, Y1 10MHz

Commit message: made changes discussed in sch review w/ prof. added back +5 plane
Parts:
- removed C1, C2: 0.1u, Capacitors_SMD:C_0805_HandSoldering
- removed J10: AIRs, custom_footprints:TerminalBlock_Pheonix_MPT-5.08mm_2pol
- removed J3: CAN, custom_footprints:TerminalBlock_Pheonix_MPT-5.08mm_2pol
- removed P4: GLV, custom_footprints:TerminalBlock_Pheonix_MPT-5.08mm_3pol
- removed P5: Cockpit, custom_footprints:TerminalBlock_Pheonix_MPT-5.08mm_6pol
- removed P6: Pedals, custom_footprints:mkds_1,5-8
- removed P7: RTDS, custom_footprints:TerminalBlock_Pheonix_MPT-5.08mm_2pol
- removed R27: 137k, Resistors_SMD:R_0805_HandSoldering
- removed R46, R48, R84: 1k, Resistors_SMD:R_0805_HandSoldering
- removed U15: TLP293, Housings_SSOP:SOP-4_4.4x2.8mm_Pitch1.27mm
- added R17: 10k, Resistors_SMD:R_0805_HandSoldering, F.Cu at (144.8, 47.0)
- added R21: 10k, Resistors_SMD:R_0805_HandSoldering, F.Cu at (38.1, 125.7)
- J1: footprint custom_footprints:mkds_1,5-8 -> custom_footprints:Molex_8x1_2.54mm
- P2: value HVPL -> CONN_02X10; footprint custom_footprints:TerminalBlock_Pheonix_MPT-5.08mm_4pol -> Connect:IDC_Header_Straight_20pins
- P3: value IMD -> CONN_02X07; footprint custom_footprints:TerminalBlock_Pheonix_MPT-5.08mm_2pol -> Connect:IDC_Header_Straight_14pins
- R1: value 10k -> 665k
- R5: value 1k -> 10k
- R9: value 137k -> 665k
- U5: footprint Power_Integrations:TO-220 -> TO_SOT_Packages_THT:TO-220_Horizontal
- Y1: footprint Crystals:Crystal_SMD_HC49-SD_HandSoldering -> custom_footprints:crystal_TXC_7A
- moved P2 230.5 mm to (20.3, 116.8), turned to 90 degrees
- moved R5 153.1 mm to (53.3, 119.4)
- moved U1 130.0 mm to (62.2, 144.8)
- moved APPS2_b 122.6 mm to (29.2, 82.5)
- moved +10V 122.3 mm to (62.2, 82.5)
- moved W4 120.3 mm to (62.2, 87.6)
- moved C3 108.8 mm to (179.1, 129.5)
- moved Q1 100.2 mm to (141.0, 36.8), turned to 90 degrees
- moved W1 97.2 mm to (121.9, 128.3)
- moved U12 96.7 mm to (132.1, 49.5)
- moved R15 94.3 mm to (141.0, 50.8)
- moved P1 94.0 mm to (110.5, 158.8)
- moved APPS1_b 93.7 mm to (29.2, 88.9)
- moved C4 92.7 mm to (139.7, 127.0), turned to 180 degrees
- moved C25 88.4 mm to (130.8, 132.1)
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- renumbered W5 to +10V, W7 to APPS1_b, W6 to APPS2_b, W10 to Thrt_LPF, W11 to Thrt_LV, W9 to Thrt_PL, W8 to Thrt_uC
Connections:
- C15 pad 1: I_+5 -> /ThrottlePlausibility/APPS1_ISO
- C15 pad 2: CH_GND -> Net-(C15-Pad2)
- C18 pad 1: I_+5 -> +5V
- C25 pad 1: I_+5 -> +5V
- C27 pad 1: I_+5 -> +5V
- C32 pad 1: I_+5 -> +5V
- C33 pad 1: I_+5 -> +5V
- C37 pad 1: I_+5 -> +5V
- C42 pad 1: I_+5 -> +5V
- C43 pad 1: I_+5 -> +5V
- C44 pad 1: I_+5 -> +5V
- C45 pad 1: I_+5 -> +5V
- C7 pad 1: I_+5 -> +5V
- CON1 pad 4: I_+5 -> +5V
- J5 pad 5: I_+5 -> +5V
- P2 pad 1: HVPL -> +24V
- P2 pad 3: CH_GND -> BOT
- P2 pad 4: CH_GND -> HVPL
- P3 pad 1: IMD_Status -> CH_GND
- P3 pad 2: IMD_PWM -> CH_GND
- R1 pad 1: Net-(R1-Pad1) -> CH_GND
- R1 pad 2: CH_GND -> Net-(R1-Pad2)
- R10 pad 1: I_+5 -> +5V
- R10 pad 2: Net-(R10-Pad2) -> Net-(R1-Pad2)
- R11 pad 2: I_+5 -> +5V
- R13 pad 1: I_+5 -> +5V
- R23 pad 1: I_+5 -> +5V
- R23 pad 2: Net-(R23-Pad2) -> Net-(C15-Pad2)
- R28 pad 1: Net-(R22-Pad2) -> CH_GND
- R28 pad 2: CH_GND -> Net-(R22-Pad2)
- R29 pad 1: Net-(R23-Pad2) -> Net-(C15-Pad2)
- R40 pad 2: I_+5 -> +5V
- R41 pad 2: I_+5 -> +5V
- R47 pad 2: I_+5 -> +5V
- R5 pad 1: Net-(R5-Pad1) -> /ThrottlePlausibility/APPS2_b
- R5 pad 2: I_+5 -> Net-(Q2-Pad3)
- R55 pad 2: Net-(R55-Pad2) -> Net-(C29-Pad1)
- R56 pad 1: Net-(C29-Pad1) -> Net-(R56-Pad1)
- R56 pad 2: Net-(R55-Pad2) -> Net-(C29-Pad1)
- R62 pad 1: Net-(C46-Pad1) -> Net-(R62-Pad1)
- R62 pad 2: Net-(R62-Pad2) -> Net-(C46-Pad1)
- R64 pad 2: Net-(R62-Pad2) -> Net-(C46-Pad1)
- R71 pad 1: I_+5 -> +5V
- R79 pad 2: I_+5 -> +5V
- R8 pad 2: I_+5 -> +5V
- R82 pad 2: I_+5 -> +5V
- R9 pad 2: Net-(R5-Pad1) -> IMD_PWM
- SW2 pad 5: I_+5 -> +5V
- U10 pad 3: I_+5 -> +5V
- U13 pad 3: I_+5 -> +5V
- U17 pad 10: Net-(R55-Pad2) -> Net-(C29-Pad1)
- U17 pad 4: I_+5 -> +5V
- U17 pad 5: Net-(R10-Pad2) -> Net-(R1-Pad2)
- U18 pad 2: Net-(R23-Pad2) -> Net-(C15-Pad2)
- U19 pad 1: I_+5 -> +5V
- U19 pad 7: Net-(C46-Pad1) -> Net-(R62-Pad1)
- U2 pad 8: I_+5 -> +5V
- U20 pad 7: Net-(C29-Pad1) -> Net-(R56-Pad1)
- U20 pad 8: I_+5 -> +5V
- U21 pad 3: Net-(R62-Pad2) -> Net-(C46-Pad1)
- U3 pad 4: I_+5 -> +5V
- U7 pad 21: I_+5 -> +5V
- U7 pad 52: I_+5 -> +5V
- U7 pad 64: I_+5 -> +5V
- U8 pad 1: I_+5 -> +5V
- U8 pad 11: I_+5 -> +5V
- U8 pad 2: I_+5 -> +5V
- W22 pad 1: I_+5 -> +5V
Routing:
- net /ThrottlePlausibility/Throttle_PL: track 0.08 -> 67.4 mm, vias 0 -> 2
- net Net-(R40-Pad1): track 3.18 -> 49.7 mm, vias 2 -> 5
- net Net-(C26-Pad1): track 0.00 -> 41.7 mm, vias 0 -> 8
- net Net-(U3-Pad1): track 0.00 -> 40.6 mm, vias 0 -> 4
- net /ThrottlePlausibility/APPS1_ISO: track 3.83 -> 41.6 mm, vias 0 -> 5
- net Net-(C30-Pad1): track 0.00 -> 33.2 mm, vias 0 -> 5
- net Net-(U3-Pad7): track 0.00 -> 31.7 mm, vias 0 -> 6
- net +5V: track 0.00 -> 29.2 mm, vias 0 -> 9
- net Net-(Q2-Pad3): track 0.00 -> 28.2 mm, vias 0 -> 4
- net +24V: track 0.00 -> 28.0 mm, vias 0 -> 4
- net Net-(U3-Pad14): track 0.00 -> 26.3 mm, vias 0 -> 2
- net /ThrottlePlausibility/APPS2_b: track 51.0 -> 77.3 mm, vias 9 -> 12
- net Net-(R41-Pad1): track 4.70 -> 30.3 mm, vias 2 -> 4
- net /ThrottlePlausibility/Throttle_SEL: track 0.00 -> 22.8 mm, vias 0 -> 4
- net Net-(R52-Pad2): track 0.00 -> 21.2 mm
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- added copper zone on B.Cu, net +5V

Commit message: organized sheet more, updated some footprints
Parts:
- removed +10V: +10V, Measurement_Points:Measurement_Point_Round-SMD-Pad_Big
- removed APPS1_b: APPS1_b, Measurement_Points:Measurement_Point_Round-SMD-Pad_Big
- removed APPS2_b: APPS2_b, Measurement_Points:Measurement_Point_Round-SMD-Pad_Big
- removed C27, C7: 0.1u, Capacitors_SMD:C_0805_HandSoldering
- removed Thrt_LPF: Throttle_LPF, Measurement_Points:Measurement_Point_Round-SMD-Pad_Big
- removed Thrt_LV: Throttle_LV, Measurement_Points:Measurement_Point_Round-SMD-Pad_Big
- removed Thrt_PL: Throttle_PL, Measurement_Points:Measurement_Point_Round-SMD-Pad_Big
- removed Thrt_uC: Throttle_uC, Measurement_Points:Measurement_Point_Round-SMD-Pad_Big
- added W10: Throttle_LPF, Measurement_Points:Measurement_Point_Round-SMD-Pad_Big, F.Cu at (114.3, 175.2)
- added W11: Throttle_LV, Measurement_Points:Measurement_Point_Round-SMD-Pad_Big, F.Cu at (45.7, 123.2)
- added W5: +10V, Measurement_Points:Measurement_Point_Round-SMD-Pad_Big, F.Cu at (62.2, 81.9)
- added W6: APPS2_b, Measurement_Points:Measurement_Point_Round-SMD-Pad_Big, F.Cu at (31.1, 89.5)
- added W7: APPS1_b, Measurement_Points:Measurement_Point_Round-SMD-Pad_Big, F.Cu at (31.1, 83.8)
- added W8: Throttle_uC, Measurement_Points:Measurement_Point_Round-SMD-Pad_Big, F.Cu at (74.9, 131.4)
- added W9: Throttle_PL, Measurement_Points:Measurement_Point_Round-SMD-Pad_Big, F.Cu at (94.0, 108.6)
- U1: footprint Converters_DCDC_ACDC:DCDC-Conv_TRACO_TMR_1-xxxx_Single -> custom_footprints:DCDC-Conv_TRACO_TMR_1-xxxx_Single
- moved J4 265.0 mm to (12.1, 158.8), turned to 0 degrees
- moved C10 154.3 mm to (168.3, 64.8), turned to 270 degrees
- moved C3 152.4 mm to (26.7, 132.7), turned to 270 degrees
- moved W16 147.2 mm to (165.7, 57.1), turned to 180 degrees
- moved C11 144.3 mm to (163.2, 64.8), turned to 270 degrees
- moved W19 143.5 mm to (26.7, 127.0)
- moved J1 132.5 mm to (74.9, 44.5)
- moved U13 110.3 mm to (144.8, 64.8), turned to 270 degrees
- moved R44 108.8 mm to (94.6, 127.0)
- moved U10 108.2 mm to (94.0, 131.4), turned to 90 degrees
- moved C18 103.0 mm to (101.6, 130.2)
- moved R37 101.9 mm to (103.5, 122.6)
- moved W22 80.2 mm to (136.5, 48.3), turned to 180 degrees
- moved W12 69.9 mm to (240.0, 137.2)
- moved P3 65.5 mm to (179.1, 72.4), turned to 90 degrees
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Connections:
- P2 pad 1: +24V -> CANH
- P2 pad 16: (no net) -> BP
- P2 pad 18: CANH -> BOT
- P2 pad 20: CANL -> +24V
- P2 pad 3: BOT -> CANL
- P2 pad 5: BP -> (no net)
- U1 pad 1: /Status Lights/HV- -> Net-(C19-Pad1)
- U1 pad 2: Net-(C19-Pad1) -> /Status Lights/HV-
- U1 pad 4: (no net) -> CH_GND
- U1 pad 6: (no net) -> HVPL
Routing:
- net Net-(C19-Pad1): track 0.00 -> 95.0 mm, vias 0 -> 7
- net /IMD: track 0.00 -> 70.4 mm, vias 0 -> 4
- net Net-(R76-Pad2): track 0.00 -> 28.5 mm, vias 0 -> 5
- net Net-(C46-Pad1): track 0.00 -> 24.2 mm, vias 0 -> 6
- net Net-(D5-Pad1): track 0.00 -> 22.9 mm, vias 0 -> 3
- net +5V: track 29.2 -> 50.9 mm, vias 9 -> 13
- net HVPL: track 0.00 -> 15.2 mm, vias 0 -> 3
- net Net-(U16-Pad10): track 0.00 -> 15.0 mm, vias 0 -> 4
- net Net-(C47-Pad2): track 0.00 -> 14.4 mm, vias 0 -> 6
- net Net-(C41-Pad1): track 0.00 -> 14.1 mm, vias 0 -> 6
- net Net-(R69-Pad1): track 0.00 -> 13.9 mm, vias 0 -> 4
- net APPS1_10: track 23.2 -> 35.9 mm, vias 6 -> 8
- net APPS2_5: track 0.00 -> 12.7 mm, vias 0 -> 2
- net /Isolators/Throttle_LV: track 19.5 -> 6.78 mm, vias 6 -> 4
- net +5HV: track 0.00 -> 11.8 mm, vias 0 -> 4
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- removed copper zone on B.Cu, net +5V
Other:
- board text added: "The MC connections can move down. Not sure what connector youre currently thinking. This would be a nice spot, since can can all come in here"

Commit message: added more tracks
Parts:
- removed W1: I_Measure, Measurement_Points:Measurement_Point_Round-SMD-Pad_Big
- removed W10: Throttle_LPF, Measurement_Points:Measurement_Point_Round-SMD-Pad_Big
- removed W11: Throttle_LV, Measurement_Points:Measurement_Point_Round-SMD-Pad_Big
- removed W12: V_Measure, Measurement_Points:Measurement_Point_Round-SMD-Pad_Big
- removed W13: Throttle_HV, Measurement_Points:Measurement_Point_Round-SMD-Pad_Big
- removed W14: +5HV, Measurement_Points:Measurement_Point_Round-SMD-Pad_Big
- removed W15: I/O_Ground, Measurement_Points:Measurement_Point_Round-SMD-Pad_Big
- removed W16: +24V, Measurement_Points:Measurement_Point_Round-SMD-Pad_Big
- removed W17: CH_GND, Measurement_Points:Measurement_Point_Square-SMD-Pad_Big
- removed W18: HV_GND, Measurement_Points:Measurement_Point_Square-SMD-Pad_Big
- removed W19: HVPL_LV, Measurement_Points:Measurement_Point_Round-SMD-Pad_Big
- removed W2: IMD_uC, Measurement_Points:Measurement_Point_Round-SMD-Pad_Big
- removed W20: GLV_GND, Measurement_Points:Measurement_Point_Square-SMD-Pad_Big
- removed W21: +5DC/DC_GND, Measurement_Points:Measurement_Point_Square-SMD-Pad_Big
- removed W22: +5DC/DC, Measurement_Points:Measurement_Point_Round-SMD-Pad_Big
- removed W23: V_Meas_GND, Measurement_Points:Measurement_Point_Square-SMD-Pad_Big
- removed W4: +10_GND, Measurement_Points:Measurement_Point_Square-SMD-Pad_Big
- removed W5: +10V, Measurement_Points:Measurement_Point_Round-SMD-Pad_Big
- removed W6: APPS2_b, Measurement_Points:Measurement_Point_Round-SMD-Pad_Big
- removed W7: APPS1_b, Measurement_Points:Measurement_Point_Round-SMD-Pad_Big
- removed W8: Throttle_uC, Measurement_Points:Measurement_Point_Round-SMD-Pad_Big
- removed W9: Throttle_PL, Measurement_Points:Measurement_Point_Round-SMD-Pad_Big
- added +10V1: +10V, Measurement_Points:Measurement_Point_Round-SMD-Pad_Big, F.Cu at (59.1, 63.5)
- added +10_GND1: +10_GND, Measurement_Points:Measurement_Point_Square-SMD-Pad_Big, F.Cu at (-17.1, 125.7)
- added +24V1: +24V, Measurement_Points:Measurement_Point_Round-SMD-Pad_Big, F.Cu at (162.6, 55.2)
- added +5DC/DC1: +5DC/DC, Measurement_Points:Measurement_Point_Round-SMD-Pad_Big, F.Cu at (132.7, 48.3)
- added +5HV1: +5HV, Measurement_Points:Measurement_Point_Round-SMD-Pad_Big, F.Cu at (30.5, 146.1)
- added ?: , custom_footprints:Symbol_HighVoltage_Type2_FSilk_VerySmall, F.Cu at (180.3, 148.0)
- added APPS1_b1: APPS1_b, Measurement_Points:Measurement_Point_Round-SMD-Pad_Big, F.Cu at (27.9, 81.3)
- added APPS2_b1: APPS2_b, Measurement_Points:Measurement_Point_Round-SMD-Pad_Big, F.Cu at (64.8, 62.9)
- added C1: 0.1u, Capacitors_SMD:C_0805_HandSoldering, F.Cu at (91.4, 94.0)
- added CH_GND1: CH_GND, Measurement_Points:Measurement_Point_Square-SMD-Pad_Big, F.Cu at (-17.1, 130.8)
- added DC/DC_GND1: +5DC/DC_GND, Measurement_Points:Measurement_Point_Square-SMD-Pad_Big, F.Cu at (-16.5, 119.4)
- added G***: LOGO, custom_footprints:ROHS, F.Cu at (163.2, 44.5)
- added G***: LOGO, custom_footprints:logo_lafayette_ece_20mmx7mm, F.Cu at (37.5, 45.7)
- added GLV_GND1: GLV_GND, Measurement_Points:Measurement_Point_Square-SMD-Pad_Big, F.Cu at (-15.9, 139.1)
- added HVPL_LV1: HVPL_LV, Measurement_Points:Measurement_Point_Round-SMD-Pad_Big, F.Cu at (26.7, 125.7)
- added HV_GND1: HV_GND, Measurement_Points:Measurement_Point_Square-SMD-Pad_Big, F.Cu at (28.6, 151.1)
- added IMD_uC1: IMD_uC, Measurement_Points:Measurement_Point_Round-SMD-Pad_Big, F.Cu at (175.3, 106.0)
- added IO_GND1: I/O_Ground, Measurement_Points:Measurement_Point_Round-SMD-Pad_Big, F.Cu at (52.7, 158.8)
- added I_Meas1: I_Meas, Measurement_Points:Measurement_Point_Round-SMD-Pad_Big, F.Cu at (168.9, 111.1)
- added REF**: MountingHole_3.5mm_Pad, Mounting_Holes:MountingHole_3.5mm_Pad, F.Cu at (180.3, 158.8)
- added REF**: MountingHole_3.5mm_Pad, Mounting_Holes:MountingHole_3.5mm_Pad, F.Cu at (18.4, 159.4)
- added REF**: MountingHole_3.5mm_Pad, Mounting_Holes:MountingHole_3.5mm_Pad, F.Cu at (19.7, 45.7)
- added REF**: Symbol_OSHW-Logo_SilkScreen, custom_footprints:Symbol_OSHW-Logo_SilkScreen, F.Cu at (19.7, 59.1)
- added Thrtl_HV1: Throttle_HV, Measurement_Points:Measurement_Point_Round-SMD-Pad_Big, F.Cu at (52.7, 150.5)
- added Thrtl_LPF1: Throttle_LPF, Measurement_Points:Measurement_Point_Round-SMD-Pad_Big, F.Cu at (82.5, 119.4)
- added Thrtl_LV1: Throttle_LV, Measurement_Points:Measurement_Point_Round-SMD-Pad_Big, F.Cu at (15.9, 124.5)
- added Thrtl_PL1: Throttle_PL, Measurement_Points:Measurement_Point_Round-SMD-Pad_Big, F.Cu at (93.3, 107.3)
- added Thrtl_uC1: Throttle_uC, Measurement_Points:Measurement_Point_Round-SMD-Pad_Big, F.Cu at (93.3, 101.0)
- added U4: LM95071-Q1, TO_SOT_Packages_SMD:SOT-23-5_HandSoldering, F.Cu at (91.4, 89.5)
- added VAL: REF, custom_footprints:lafLogo, F.Cu at (174.0, 140.3)
- added V_Meas1: V_Measure, Measurement_Points:Measurement_Point_Round-SMD-Pad_Big, F.Cu at (151.1, 121.3)
- added V_Meas_GND1: V_Meas_GND, Measurement_Points:Measurement_Point_Square-SMD-Pad_Big, F.Cu at (-16.5, 145.4)
- moved J4 56.5 mm to (68.6, 160.0), turned to 90 degrees
- moved C25 46.8 mm to (161.9, 111.8), turned to 270 degrees
- moved R44 21.9 mm to (116.2, 123.2)
- moved P1 21.6 mm to (132.1, 158.1)
- moved C19 21.6 mm to (108.0, 155.6)
- moved C24 21.6 mm to (123.2, 158.1)
- moved D5 21.6 mm to (79.4, 153.0)
- moved L1 21.6 mm to (99.1, 154.3)
- moved R19 21.6 mm to (106.7, 161.9)
- moved R20 21.6 mm to (97.8, 161.9)
- moved R69 21.6 mm to (88.9, 161.9)
- moved R70 21.6 mm to (88.9, 159.4)
- moved R76 21.6 mm to (108.0, 150.5)
- moved R77 21.6 mm to (108.0, 153.0)
- moved R16 21.6 mm to (115.6, 161.9)
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Connections:
- U7 pad 10: (no net) -> /~SS
- U7 pad 11: (no net) -> /SCK
- U7 pad 13: (no net) -> /MISO
Routing:
- net CANH: track 0.00 -> 122.6 mm, vias 0 -> 4
- net CANL: track 0.00 -> 118.9 mm, vias 0 -> 4
- net /I_Measure: track 0.00 -> 98.5 mm, vias 0 -> 11
- net /ThrottlePlausibility/BOT_uC: track 0.00 -> 83.9 mm, vias 0 -> 4
- net /ThrottlePlausibility/BP_uC: track 0.00 -> 60.9 mm, vias 0 -> 4
- net /ThrottlePlausibility/Throttle_uC: track 0.00 -> 58.4 mm, vias 0 -> 2
- net Net-(C4-Pad2): track 0.00 -> 47.6 mm, vias 0 -> 7
- net /IMD: track 70.4 -> 25.1 mm, vias 4 -> 2
- net /PIN54: track 0.00 -> 45.2 mm, vias 0 -> 2
- net /Safety_Loop: track 0.00 -> 45.2 mm, vias 0 -> 2
- net /PIN55: track 0.00 -> 42.1 mm, vias 0 -> 4
- net /CAN Transceiver/CANRX: track 0.00 -> 36.6 mm, vias 0 -> 2
- net /I_ENB: track 0.00 -> 33.1 mm, vias 0 -> 4
- net Net-(C29-Pad1): track 0.00 -> 31.4 mm, vias 0 -> 9
- net Net-(R1-Pad2): track 0.00 -> 30.8 mm, vias 0 -> 6
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- removed copper zone on F.Cu, net CH_GND
Other:
- board size 203.2 x 152.4 mm -> 177.8 x 127 mm
- board text added: "Made in U.S.A."

Commit message: working on pcb
Parts:
- moved C5 7.10 mm to (109.2, 105.4), turned to 270 degrees
- moved Y1 5.12 mm to (104.1, 106.7)
- moved C6 2.01 mm to (102.9, 103.5), turned to 0 degrees
- moved C18 1.91 mm to (102.9, 123.2), turned to 90 degrees
- moved R11 1.90 mm to (108.6, 111.1)
- moved Thrtl_LPF1 1.27 mm to (82.5, 118.1)
- moved R8 0.64 mm to (111.1, 111.1)
- moved C31 0.63 mm to (103.5, 78.1)
- turned C42 to 180 degrees
- turned R34 to 0 degrees
- turned R43 to 180 degrees
- turned R59 to 0 degrees
- turned R81 to 0 degrees
Routing:
- net /ThrottlePlausibility/Throttle_SEL: track 22.8 -> 98.6 mm, vias 4 -> 6
- net CH_GND: track 0.00 -> 42.8 mm, vias 0 -> 10
- net /ThrottlePlausibility/Throttle_PL: track 71.9 -> 92.2 mm, vias 2 -> 4
- net +5V: track 70.2 -> 78.5 mm, vias 19 -> 33
- net Net-(C30-Pad1): track 33.2 -> 40.9 mm
- net TDO: track 13.9 -> 21.4 mm
- net IMD_Fault_LED: track 6.35 -> 0.00 mm, vias 2 -> 0
- net Net-(C28-Pad2): track 28.5 -> 33.6 mm, vias 8 -> 6
- net Net-(R56-Pad1): track 6.14 -> 11.1 mm
- net Net-(R57-Pad1): track 8.68 -> 12.3 mm
- net Net-(C6-Pad1): track 8.86 -> 12.1 mm, vias 2 -> 0
- net /CAN Transceiver/CANRX: track 36.6 -> 33.4 mm, vias 2 -> 4
- net Net-(C26-Pad1): track 49.3 -> 51.7 mm, vias 9 -> 7
- net Net-(C5-Pad1): track 10.5 -> 8.05 mm, vias 2 -> 0
- net Net-(C29-Pad1): track 31.4 -> 33.8 mm, vias 9 -> 8
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- added copper zone on B.Cu, net +5V
- added copper zone on F.Cu, net CH_GND
