File: Circuit_layout/Circuit_layout.kicad_pcb (KiCad board)
At the start: 2 copper layers, 177.8 x 127 mm, 190 parts, among them CON1 AVR-JTAG-10, J1 Spare_Conns, J4 Motor_Ctrl, J5 RJ12, P1 TSV, P2 CONN_02X10, P3 CONN_02X07, Q1 ZVP4525G, Q2 MMBF170, Q3 MMBF170, SW1 SW_PUSH, SW2 TS5A3159-Q1, SW3 JS202011CQN, U1 PDM2-S24-S12, U10 MCP2551-I/SN, U11 TLP293, U12 TLP293, U13 PDQ10-D, U16 LTC3638, U17 MCP6004, U18 TS912, U19 ACPL-C870, U2 MCP6002, U20 ACPL-C870, U21 MCP6001, U22 TS372, U23 TLP293, U24 TLP293, U3 MCP6004, U4 LM95071-Q1, U5 LM7810CT, U6 TS912, U7 AT90CAN128-A, U8 74ACT11030, U9 TLP293, Y1 10MHz

Commit message: working on pcb
Parts:
- J4: footprint custom_footprints:TerminalBlock_Pheonix_MPT-5.08mm_4pol -> custom_footprints:Molex_4x1_2.54mm
- P1: footprint custom_footprints:TerminalBlock_Pheonix_MPT-5.08mm_2pol -> custom_footprints:AMPCONN_2
- moved HVPL_HV1 126.2 mm to (101.6, 168.9)
- moved P3 40.7 mm to (138.4, 69.8)
- moved C37 27.6 mm to (147.3, 61.0), turned to 270 degrees
- moved R65 21.6 mm to (151.1, 144.8)
- moved R67 20.1 mm to (144.8, 144.8)
- moved P1 19.1 mm to (151.1, 156.2), turned to 180 degrees
- moved R68 18.8 mm to (138.4, 144.8)
- moved U13 18.0 mm to (162.6, 62.2)
- moved C11 16.7 mm to (179.7, 62.2)
- moved C10 16.7 mm to (184.8, 62.2)
- moved +24V1 16.5 mm to (179.1, 55.2)
- moved R61 15.9 mm to (157.5, 144.8)
- moved +5DC/DC1 14.7 mm to (147.3, 47.0)
- moved Thrtl_LV1 13.1 mm to (28.6, 127.6)
- moved J1 12.1 mm to (66.0, 52.7), turned to 0 degrees
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Connections:
- CON1 pad 7: (no net) -> Net-(CON1-Pad7)
- CON1 pad 8: (no net) -> Net-(CON1-Pad8)
- J5 pad 1: (no net) -> Net-(J5-Pad1)
- J5 pad 6: (no net) -> Net-(J5-Pad6)
- P2 pad 14: (no net) -> Net-(P2-Pad14)
- P2 pad 19: (no net) -> Net-(P2-Pad19)
- P2 pad 5: (no net) -> Net-(P2-Pad5)
- U10 pad 5: (no net) -> Net-(U10-Pad5)
- U13 pad 4: (no net) -> Net-(U13-Pad4)
- U13 pad 6: (no net) -> Net-(U13-Pad6)
- U7 pad 12: (no net) -> Net-(U7-Pad12)
- U7 pad 18: (no net) -> Net-(U7-Pad18)
- U7 pad 19: (no net) -> Net-(U7-Pad19)
- U7 pad 27: (no net) -> Net-(U7-Pad27)
- U7 pad 28: (no net) -> Net-(U7-Pad28)
- U7 pad 29: (no net) -> Net-(U7-Pad29)
- U7 pad 32: (no net) -> Net-(U7-Pad32)
- U7 pad 33: (no net) -> Net-(U7-Pad33)
- U7 pad 34: (no net) -> Net-(U7-Pad34)
- U7 pad 35: /ThrottlePlausibility/BOT_uC -> Net-(U7-Pad35)
- U7 pad 39: (no net) -> Net-(U7-Pad39)
- U7 pad 4: (no net) -> Net-(U7-Pad4)
- U7 pad 40: (no net) -> Net-(U7-Pad40)
- U7 pad 41: (no net) -> Net-(U7-Pad41)
- U7 pad 42: (no net) -> Net-(U7-Pad42)
- U7 pad 43: (no net) -> Net-(U7-Pad43)
- U7 pad 45: (no net) -> Net-(U7-Pad45)
- U7 pad 49: (no net) -> Net-(U7-Pad49)
- U7 pad 50: (no net) -> Net-(U7-Pad50)
- U7 pad 51: (no net) -> Net-(U7-Pad51)
- U7 pad 6: (no net) -> Net-(U7-Pad6)
- U7 pad 8: (no net) -> /ThrottlePlausibility/BOT_uC
Routing:
- net +24V: track 33.0 -> 305.3 mm, vias 4 -> 11
- net APPS2: track 0.00 -> 102.7 mm, vias 0 -> 2
- net /IMD: track 25.1 -> 124.3 mm, vias 2 -> 8
- net /Isolators/V_Measure: track 27.5 -> 109.6 mm, vias 7 -> 11
- net IMD_PWM: track 0.00 -> 74.8 mm, vias 0 -> 4
- net UART_TX: track 0.00 -> 69.7 mm, vias 0 -> 1
- net UART_RX: track 0.00 -> 69.3 mm, vias 0 -> 1
- net Spare_ICP: track 0.00 -> 65.4 mm, vias 0 -> 3
- net Spare_OC: track 0.00 -> 61.7 mm, vias 0 -> 1
- net Drive_BTN: track 0.00 -> 45.7 mm, vias 0 -> 2
- net IMD_Fault_LED: track 0.00 -> 44.9 mm, vias 0 -> 2
- net BP: track 0.00 -> 43.1 mm, vias 0 -> 2
- net +24V_RTN: track 5.08 -> 47.9 mm
- net BOT: track 0.00 -> 42.7 mm, vias 0 -> 1
- net RTDS: track 0.00 -> 41.9 mm, vias 0 -> 2
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
Commit message: small changes to pcb
Other:
- net class TSV added: clearance 0.5, trace_width 0.5, via_dia 0.6, via_drill 0.4
Changed lines of the file:
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@@
     (trace_clearance 0.2)
     (zone_clearance 0.508)
-    (zone_45_only no)
+    (zone_45_only yes)
     (trace_min 0.2)
     (segment_width 0.2)
@@
     (add_net Drive_BTN)
     (add_net Drive_LED)
-    (add_net HV+)
     (add_net HV-)
     (add_net HVPL)
@@
     (add_net ~RESET_AVR)
   )
+  (net_class TSV ""
+    (clearance 0.5)
+    (trace_width 0.5)
+    (via_dia 0.6)
+    (via_drill 0.4)
+    (uvia_dia 0.3)
+    (uvia_drill 0.1)
+    (add_net HV+)
+  )
   (module Housings_QFP:TQFP-64_14x14mm_Pitch0.8mm (layer F.Cu)
     (at 108.585 92.71)
@@
       )
     )
+  )
+  (zone (net 0) (net_name "") (layer F.Cu) (hatch edge 0.508)
+    (connect_pads (clearance 0.508))
+    (min_thickness 0.254)
+    (keepout (tracks allowed) (vias allowed) (copperpour not_allowed))
+    (fill (arc_segments 16) (thermal_gap 0.508) (thermal_bridge_width 0.508))
+    (polygon
+      (pts
+        (xy 114.935 99.06) (xy 102.235 99.06) (xy 102.235 86.36) (xy 114.935 86.36) (xy 114.935 99.06)
+      )
+    )

Commit message: finishing rev 0 of pcb
Parts:
- removed the G*** at (37.5, 45.7)
- removed R35: 2k, Resistors_SMD:R_0805_HandSoldering
- removed the REF** at (180.3, 158.8)
- removed the REF** at (18.4, 159.4)
- removed the REF** at (19.7, 45.7)
- added ?: , custom_footprints:Symbol_HighVoltage_Type2_BSilk_VerySmall, F.Cu at (200.0, 148.6)
- added G***: LOGO, custom_footprints:logo_lafayette_ece_32mmx11mm, F.Cu at (47.0, 35.6)
- moved DC/DC_GND1 223.2 mm to (199.4, 62.9)
- moved V_Meas_GND1 216.2 mm to (196.2, 106.7)
- moved VAL 109.0 mm to (204.5, 32.4)
- moved GLV_GND1 100.0 mm to (40.6, 56.5)
- moved G*** 92.9 mm to (71.1, 32.4)
- moved REF** 66.2 mm to (80.0, 31.8)
- moved HVPL_HV1 63.5 mm to (43.2, 144.1)
- moved +5HV1 62.7 mm to (92.7, 138.4)
- moved +5DC/DC1 61.7 mm to (196.8, 83.8)
- moved IO_GND1 40.0 mm to (92.1, 151.8)
- moved APPS2_b1 34.9 mm to (45.7, 92.1)
- moved Thrtl_HV1 34.6 mm to (85.1, 138.4)
- moved I_Meas1 30.2 mm to (196.8, 99.7)
- moved APPS1_b1 26.7 mm to (47.6, 82.5)
- moved C23 22.2 mm to (71.8, 71.1)
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Connections:
- C19 pad 2: /Status Lights/HV- -> HV-
- C24 pad 1: /Status Lights/HV+ -> HV+
- C24 pad 2: /Status Lights/HV- -> HV-
- D5 pad 2: /Status Lights/HV- -> HV-
- HV_GND1 pad 1: /Status Lights/HV- -> HV-
- R16 pad 2: /Status Lights/HV+ -> HV+
- R70 pad 2: /Status Lights/HV- -> HV-
- R77 pad 2: /Status Lights/HV- -> HV-
- U1 pad 2: /Status Lights/HV- -> HV-
- U12 pad 4: Net-(R35-Pad2) -> +24V
- U16 pad 12: /Status Lights/HV- -> HV-
- U16 pad 16: /Status Lights/HV- -> HV-
- U16 pad 17: /Status Lights/HV- -> HV-
- U16 pad 3: /Status Lights/HV+ -> HV+
- U16 pad 6: /Status Lights/HV- -> HV-
- U16 pad 8: /Status Lights/HV- -> HV-
Routing:
- net +5HV: track 8.02 -> 156.0 mm, vias 2 -> 1
- net SCL: track 13.5 -> 146.1 mm, vias 2 -> 4
- net SDA: track 11.6 -> 137.4 mm, vias 2 -> 4
- net I/O_Ground: track 4.17 -> 122.2 mm, vias 2 -> 10
- net HV+: track 0.00 -> 105.9 mm, vias 0 -> 2
- net APPS1_10: track 40.9 -> 141.3 mm, vias 9 -> 14
- net CH_GND: track 40.0 -> 104.2 mm, vias 9 -> 18
- net ~RESET_AVR: track 42.7 -> 88.3 mm, vias 2 -> 4
- net Throttle_HV: track 10.2 -> 43.8 mm, vias 2 -> 3
- net /ThrottlePlausibility/APPS2_b: track 78.9 -> 102.9 mm, vias 11 -> 10
- net Net-(C41-Pad1): track 0.00 -> 20.6 mm, vias 0 -> 2
- net HV-: track 0.00 -> 20.5 mm, vias 0 -> 2
- net Net-(C19-Pad1): track 118.0 -> 135.4 mm, vias 9 -> 5
- net /Isolators/Throttle_LV: track 9.06 -> 25.1 mm, vias 2 -> 4
- net Net-(R35-Pad2): track 15.9 -> 0.00 mm, vias 4 -> 0
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Other:
- board text added: "High Voltage"
- board text added: "Low Voltage"
- board text added: "Tractive System Interface"
- board text removed: "The MC connections can move down. Not sure what connector youre currently thinking. This would be a nice spot, since can can all come in here"

Commit message: adding silkscreen
Parts:
- added ?: MountingHole_3.5mm_Pad, Mounting_Holes:MountingHole_3.5mm_Pad, F.Cu at (35.6, 34.3)
- added ?: MountingHole_3.5mm_Pad, Mounting_Holes:MountingHole_3.5mm_Pad, F.Cu at (203.2, 34.3)
- added ?: MountingHole_3.5mm_Pad, Mounting_Holes:MountingHole_3.5mm_Pad, F.Cu at (35.6, 151.1)
- added REF**: MountingHole_3.5mm_Pad, Mounting_Holes:MountingHole_3.5mm_Pad, F.Cu at (203.2, 151.1)
- moved VAL 93.3 mm to (204.5, 125.7)
- moved G*** 22.9 mm to (94.0, 34.3)
- moved ? 11.4 mm to (200.0, 137.2)
- moved ? 11.4 mm to (200.7, 137.2)
- moved G*** 10.2 mm to (57.1, 35.6)
- moved REF** 5.24 mm to (85.1, 33.0)
Changed lines of the file:
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@@
     (links 405)
     (no_connects 3)
-    (area 30.404999 29.134999 208.355001 156.285001)
+    (area -39.052858 17.47 231.825715 156.905)
     (thickness 1.6)
-    (drawings 12)
+    (drawings 13)
     (tracks 1531)
     (zones 0)
-    (modules 187)
+    (modules 191)
     (nets 167)
   )
@@
     (visible_elements 7FFEFFFF)
     (pcbplotparams
-      (layerselection 0x00030_80000001)
+      (layerselection 0x0003c_80000001)
       (usegerberextensions false)
       (excludeedgelayer true)
@@
   )
   (module custom_footprints:ROHS (layer F.Cu)
-    (at 71.12 32.385)
+    (at 93.98 34.29)
     (fp_text reference G*** (at 0 0) (layer F.SilkS) hide
       (effects (font (thickness 0.3)))
@@
   )
   (module custom_footprints:Symbol_HighVoltage_Type2_FSilk_VerySmall (layer F.Cu)
-    (at 199.39 148.59)
+    (at 200.025 137.16)
     (descr "Symbol, High Voltage, Type 2, Copper Top, Very Small,")
     (tags "Symbol, High Voltage, Type 2, Copper Top, Very Small,")
@@
   )
   (module custom_footprints:Symbol_HighVoltage_Type2_BSilk_VerySmall (layer F.Cu)
-    (at 200.025 148.59)
+    (at 200.66 137.16)
     (descr "Symbol, High Voltage, Type 2, Copper Top, Very Small,")
     (tags "Symbol, High Voltage, Type 2, Copper Top, Very Small,")
@@
   )
   (module custom_footprints:Symbol_OSHW-Logo_SilkScreen (layer F.Cu)
-    (at 80.01 31.75)
+    (at 85.09 33.02)
     (descr "Symbol, OSHW-Logo, Silk Screen,")
     (tags "Symbol, OSHW-Logo, Silk Screen,")
@@
   )
   (module custom_footprints:logo_lafayette_ece_32mmx11mm (layer F.Cu)
-    (at 46.99 35.56)
+    (at 57.15 35.56)
     (fp_text reference G*** (at 0 0) (layer F.SilkS) hide
       (effects (font (thickness 0.3)))
@@
   )
   (module custom_footprints:lafLogo (layer F.Cu)
-    (at 204.47 32.385)
+    (at 204.47 125.73)
     (fp_text reference VAL (at 0 0) (layer F.SilkS) hide
       (effects (font (size 0.381 0.381) (thickness 0.127)))
@@
       (xy 1.65862 -1.25476) (xy 1.66878 -1.13792) (xy 1.66878 -1.13792)) (layer F.Cu) (width 0.00254))
   )
+  (module Mounting_Holes:MountingHole_3.5mm_Pad (layer F.Cu)
+    (at 35.56 34.29)
+    (descr "Mounting Hole 3.5mm")
+    (tags "mounting hole 3.5mm")
+    (fp_text reference "" (at 0 -4.5) (layer F.SilkS)
+      (effects (font (size 1 1) (thickness 0.15)))
+    )
+    (fp_text value MountingHole_3.5mm_Pad (at 0 4.5) (layer F.Fab)
+      (effects (font (size 1 1) (thickness 0.15)))
+    )
+    (fp_circle (center 0 0) (end 3.5 0) (layer Cmts.User) (width 0.15))
+    (fp_circle (center 0 0) (end 3.75 0) (layer F.CrtYd) (width 0.05))
+    (pad 1 thru_hole circle (at 0 0) (size 7 7) (drill 3.5) (layers *.Cu *.Mask))
+  )
+  (module Mounting_Holes:MountingHole_3.5mm_Pad (layer F.Cu)
+    (at 203.2 34.29)
+    (descr "Mounting Hole 3.5mm")
+    (tags "mounting hole 3.5mm")
+    (fp_text reference "" (at 0 -4.5) (layer F.SilkS)
+      (effects (font (size 1 1) (thickness 0.15)))
+    )
+    (fp_text value MountingHole_3.5mm_Pad (at 0 4.5) (layer F.Fab)
+      (effects (font (size 1 1) (thickness 0.15)))
+    )
+    (fp_circle (center 0 0) (end 3.5 0) (layer Cmts.User) (width 0.15))
+    (fp_circle (center 0 0) (end 3.75 0) (layer F.CrtYd) (width 0.05))
+    (pad 1 thru_hole circle (at 0 0) (size 7 7) (drill 3.5) (layers *.Cu *.Mask))
+  )
+  (module Mounting_Holes:MountingHole_3.5mm_Pad (layer F.Cu)
+    (at 203.2 151.13)
+    (descr "Mounting Hole 3.5mm")
+    (tags "mounting hole 3.5mm")
+    (fp_text reference REF** (at 0 -4.5) (layer F.SilkS)
+      (effects (font (size 1 1) (thickness 0.15)))
+    )
+    (fp_text value MountingHole_3.5mm_Pad (at 0 4.5) (layer F.Fab)
+      (effects (font (size 1 1) (thickness 0.15)))
+    )
+    (fp_circle (center 0 0) (end 3.5 0) (layer Cmts.User) (width 0.15))
+    (fp_circle (center 0 0) (end 3.75 0) (layer F.CrtYd) (width 0.05))
+    (pad 1 thru_hole circle (at 0 0) (size 7 7) (drill 3.5) (layers *.Cu *.Mask))
+  )
+  (module Mounting_Holes:MountingHole_3.5mm_Pad (layer F.Cu)
+    (at 35.56 151.13)
+    (descr "Mounting Hole 3.5mm")
+    (tags "mounting hole 3.5mm")
+    (fp_text reference "" (at 0 -4.5) (layer F.SilkS)
+      (effects (font (size 1 1) (thickness 0.15)))
+    )
+    (fp_text value MountingHole_3.5mm_Pad (at 0 4.5) (layer F.Fab)
+      (effects (font (size 1 1) (thickness 0.15)))
+    )
+    (fp_circle (center 0 0) (end 3.5 0) (layer Cmts.User) (width 0.15))
+    (fp_circle (center 0 0) (end 3.75 0) (layer F.CrtYd) (width 0.05))
+    (pad 1 thru_hole circle (at 0 0) (size 7 7) (drill 3.5) (layers *.Cu *.Mask))
+  )
+  (dimension 6.35 (width 0.3) (layer Dwgs.User)
+    (gr_text "6.350 mm" (at 13.97 128.27 270) (layer Dwgs.User)
+      (effects (font (size 1.5 1.5) (thickness 0.3)))
+    )
+    (feature1 (pts (xy 29.21 130.81) (xy 16.35 130.81)))
+    (feature2 (pts (xy 29.21 124.46) (xy 16.35 124.46)))
+    (crossbar (pts (xy 19.05 124.46) (xy 19.05 130.81)))
+    (arrow1a (pts (xy 19.05 130.81) (xy 18.463579 129.683496)))
+    (arrow1b (pts (xy 19.05 130.81) (xy 19.636421 129.683496)))
+    (arrow2a (pts (xy 19.05 124.46) (xy 18.463579 125.586504)))
+    (arrow2b (pts (xy 19.05 124.46) (xy 19.636421 125.586504)))
+  )
   (gr_text "Low Voltage" (at 128.905 126.365) (layer F.SilkS)
     (effects (font (size 3 3) (thickness 0.3)))
@@
     (arrow2b (pts (xy 224.79 156.21) (xy 224.203579 155.083496)))
   )
-  (gr_text "Made in U.S.A." (at 46.99 42.545) (layer F.SilkS)
+  (gr_text "Made in U.S.A." (at 57.15 41.91) (layer F.SilkS)
     (effects (font (size 1.5 1.5) (thickness 0.3)))
   )
@@
   (segment (start 124.46 139.7) (end 124.46 139.78) (width 0.25) (layer F.Cu) (net 121))
   (via (at 103.505 139.7) (size 0.6) (drill 0.4) (layers F.Cu B.Cu) (net 121))
-  (segment (start 103.505 139.7) (end 103.505 142.24) (width 0.25) (layer B.Cu) (net 121))
-  (via (at 103.505 142.24) (size 0.6) (drill 0.4) (layers F.Cu B.Cu) (net 121))
-  (segment (start 103.3045 142.4405) (end 103.505 142.24) (width 0.25) (layer F.Cu) (net 121))
+  (segment (start 103.505 139.7) (end 103.505 141.605) (width 0.25) (layer B.Cu) (net 121))
+  (via (at 103.505 141.605) (size 0.6) (drill 0.4) (layers F.Cu B.Cu) (net 121))
+  (segment (start 103.3045 141.8055) (end 103.505 141.605) (width 0.25) (layer F.Cu) (net 121))
   (segment (start 124.46 139.7) (end 103.505 139.7) (width 0.25) (layer F.Cu) (net 121))
   (segment (start 124.46 139.78) (end 126.285 141.605) (width 0.25) (layer F.Cu) (net 121))
-  (segment (start 103.3045 142.4405) (end 103.3045 142.57) (width 0.25) (layer F.Cu) (net 121))
+  (segment (start 103.3045 141.8055) (end 103.3045 142.57) (width 0.25) (layer F.Cu) (net 121))
   (segment (start 54.21 102.87) (end 52.705 102.87) (width 0.25) (layer F.Cu) (net 122))
   (via (at 52.705 102.87) (size 0.6) (drill 0.4) (layers F.Cu B.Cu) (net 122))
@@
   (via (at 106.68 84.455) (size 0.6) (drill 0.4) (layers F.Cu B.Cu) (net 135))
   (segment (start 107 84.775) (end 106.68 84.455) (width 0.25) (layer F.Cu) (net 135))
-  (zone (net 24) (net_name HV-) (layer F.Cu) (hatch edge 0.508)
-    (connect_pads (clearance 0.508))
-    (min_thickness 0.254)
-    (fill yes (arc_segments 16) (thermal_gap 0.508) (thermal_bridge_width 0.508))
-    (polygon
-      (pts
-        (xy 206.375 154.94) (xy 31.75 154.94) (xy 31.75 131.445) (xy 206.375 131.445) (xy 206.375 154.94)
-      )
-    )
-  )
   (zone (net 1) (net_name CH_GND) (layer F.Cu) (hatch edge 0.508)
     (connect_pads (clearance 0.508))
@@
       )
     )
+  )
+  (zone (net 24) (net_name HV-) (layer F.Cu) (hatch edge 0.508)
+    (connect_pads (clearance 0.508))
+    (min_thickness 0.254)
+    (fill yes (arc_segments 16) (thermal_gap 0.508) (thermal_bridge_width 0.508))
+    (polygon
+      (pts
+        (xy 206.375 154.94) (xy 31.75 154.94) (xy 31.75 131.445) (xy 206.375 131.445) (xy 206.375 154.94)
+      )
+    )

Commit message: review pcb, made notes
Parts:
- removed +10_GND1: +10_GND, Measurement_Points:Measurement_Point_Square-SMD-Pad_Big
- removed CH_GND1: CH_GND, Measurement_Points:Measurement_Point_Square-SMD-Pad_Big
- removed W3: uC_GND, Measurement_Points:Measurement_Point_Square-SMD-Pad_Big
- moved R61 5.85 mm to (171.4, 138.4)
- moved R65 5.85 mm to (165.1, 138.4)
- moved R67 5.85 mm to (158.8, 138.4)
- moved R68 5.85 mm to (152.4, 138.4)
- renumbered APPS1_b1 to APPS1_b, APPS2_b1 to APPS2_b
Routing:
- net Net-(C19-Pad1): track 135.4 -> 152.1 mm
- net HV-: track 20.5 -> 35.1 mm
- net Net-(R80-Pad2): track 16.7 -> 29.7 mm, vias 3 -> 4
- net CH_GND: track 104.2 -> 115.5 mm
- net Net-(C26-Pad2): track 16.9 -> 23.7 mm
- net +5V: track 75.8 -> 78.8 mm
- net HV+: track 105.9 -> 103.0 mm
- net BP: track 43.1 -> 41.6 mm, vias 2 -> 1
- net Net-(Q2-Pad1): track 7.56 -> 8.58 mm
- net Net-(R50-Pad2): track 24.0 -> 24.8 mm
- net /ThrottlePlausibility/Throttle_SEL: track 98.6 -> 97.8 mm
- net Net-(C41-Pad1): track 20.6 -> 20.0 mm
Other:
- net class Default: clearance 0.2 -> 0.254
- rule trace_clearance: 0.2 -> 0.254
