File: Circuit_layout/Circuit_layout.kicad_pcb (KiCad board)
At the start: 2 copper layers, 177.8 x 127 mm, 193 parts, among them CON1 AVR-JTAG-10, J1 Spare_Conns, J4 Motor_Ctrl, J5 RJ12, P1 TSV, P2 CONN_02X10, P3 CONN_02X07, Q1 ZVP4525G, Q2 MMBF170, Q3 MMBF170, SW1 SW_PUSH, SW2 TS5A3159-Q1, SW3 JS202011CQN, U1 PDM2-S24-S12, U10 MCP2551-I/SN, U11 TLP293, U12 TLP293, U13 PDQ10-D, U14 Mounting_hole, U15 Mounting_hole, U16 LTC3638, U17 MCP6004, U18 TS912, U19 ACPL-C870, U2 MCP6002, U20 ACPL-C870, U21 MCP6001, U22 TS372, U23 TLP293, U24 TLP293, U25 Mounting_hole, U26 Mounting_hole, U27 TLP293, U3 MCP6004, U4 LM95071-Q1, U5 LM7810CT, U6 TS912, U7 AT90CAN128-A, U8 74ACT11030, U9 TLP293, Y1 10MHz

Commit message: final changes to pcb. working on BOM
Routing:
- net (no net): track 0.65 -> 3.47 mm, vias 0 -> 2
Other:
- board text added: "HEART"
- board text added: "L17_TSI_001"
- board text added: "REV 0"
- board text added: "SN"
- board text added: "SP"
- board text added: "SP/FLT"
- board text removed: "Heart"
- board text removed: "Sp"
- board text removed: "Sp/Flt"
Changed lines of the file:
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@@
     (links 413)
     (no_connects 0)
-    (area -39.052858 17.47 231.825715 156.905)
+    (area -20.013201 17.47 231.825715 156.905)
     (thickness 1.6)
-    (drawings 21)
-    (tracks 1612)
+    (drawings 24)
+    (tracks 1618)
     (zones 0)
     (modules 193)
@@
     (41 Cmts.User user)
     (42 Eco1.User user)
-    (43 Eco2.User user hide)
+    (43 Eco2.User user)
     (44 Edge.Cuts user)
     (45 Margin user)
@@
       (effects (font (size 1 1) (thickness 0.15)))
     )
-    (fp_text user 1 (at -1.5 -1.5 90) (layer F.SilkS)
+    (fp_text user 1 (at -3.5306 -1.7018 90) (layer F.SilkS)
       (effects (font (size 1 1) (thickness 0.15)))
     )
-    (fp_text user Vout (at 10.25 4 90) (layer F.SilkS)
+    (fp_text user Vout (at 12.2936 7.1374 90) (layer F.SilkS)
       (effects (font (size 1 1) (thickness 0.15)))
     )
-    (fp_text user Vin (at 1.25 4 90) (layer F.SilkS)
+    (fp_text user Vin (at -0.254 7.6454 90) (layer F.SilkS)
       (effects (font (size 1 1) (thickness 0.15)))
     )
-    (fp_text user + (at 12.7 2.54 90) (layer F.SilkS)
+    (fp_text user + (at 14.732 7.112 90) (layer F.SilkS)
       (effects (font (size 1 1) (thickness 0.15)))
     )
-    (fp_text user - (at 7.62 2.54 90) (layer F.SilkS)
+    (fp_text user - (at 10.0076 7.1374 90) (layer F.SilkS)
       (effects (font (size 1 1) (thickness 0.15)))
     )
-    (fp_text user - (at 2.54 2.54 90) (layer F.SilkS)
+    (fp_text user - (at 1.6764 7.6454 90) (layer F.SilkS)
       (effects (font (size 1 1) (thickness 0.15)))
     )
-    (fp_text user + (at 0 2.54 90) (layer F.SilkS)
+    (fp_text user + (at -2.2352 7.5692 90) (layer F.SilkS)
       (effects (font (size 1 1) (thickness 0.15)))
     )
@@
     (tags "capacitor 0805")
     (attr smd)
-    (fp_text reference C42 (at 3.81 0 180) (layer F.SilkS)
+    (fp_text reference C42 (at 3.7338 0.4826 180) (layer F.SilkS)
       (effects (font (size 1 1) (thickness 0.15)))
     )
@@
     (tags "resistor 0805")
     (attr smd)
-    (fp_text reference R32 (at -3.81 0 180) (layer F.SilkS)
+    (fp_text reference R32 (at -3.8608 1.016 180) (layer F.SilkS)
       (effects (font (size 1 1) (thickness 0.15)))
     )
@@
     (tags "resistor 0805")
     (attr smd)
-    (fp_text reference R34 (at -3.81 0) (layer F.SilkS)
+    (fp_text reference R34 (at -3.8862 -0.889) (layer F.SilkS)
       (effects (font (size 1 1) (thickness 0.15)))
     )
@@
     (descr "20 pins through hole IDC header")
     (tags "IDC header socket VASCH")
-    (fp_text reference P2 (at 11.43 -7.62 90) (layer F.SilkS)
+    (fp_text reference P2 (at 29.4386 -5.3594 180) (layer F.SilkS)
       (effects (font (size 1 1) (thickness 0.15)))
     )
@@
     (fp_line (start 28.44 3.78) (end -5.58 3.78) (layer F.CrtYd) (width 0.05))
     (fp_line (start -5.58 3.78) (end -5.58 -6.32) (layer F.CrtYd) (width 0.05))
-    (fp_text user 1 (at 0.02 1.72 90) (layer F.SilkS)
+    (fp_text user 1 (at -0.1778 4.7752 90) (layer F.SilkS)
       (effects (font (size 1 1) (thickness 0.12)))
     )
@@
     (fp_line (start 20.82 3.78) (end -5.58 3.78) (layer F.CrtYd) (width 0.05))
     (fp_line (start -5.58 3.78) (end -5.58 -6.32) (layer F.CrtYd) (width 0.05))
-    (fp_text user 1 (at 0.02 1.72 90) (layer F.SilkS)
+    (fp_text user 1 (at -0.1524 4.8514 90) (layer F.SilkS)
       (effects (font (size 1 1) (thickness 0.12)))
     )
@@
       (xy 0.465667 0.021167)) (layer F.SilkS) (width 0.01))
   )
+  (gr_text "REV 0" (at 168.91 34.29) (layer B.Cu)
+    (effects (font (size 1.5 1.5) (thickness 0.3)) (justify mirror))
+  )
+  (gr_text L17_TSI_001 (at 184.15 34.29) (layer B.Cu)
+    (effects (font (size 1.5 1.5) (thickness 0.3)) (justify mirror))
+  )
+  (gr_text SN (at 34.925 47.625) (layer F.SilkS)
+    (effects (font (size 2.54 2.54) (thickness 0.508)))
+  )
   (gr_text "High Voltage" (at 128.905 133.35) (layer B.SilkS)
     (effects (font (size 3 3) (thickness 0.3)) (justify mirror))
@@
     (effects (font (size 2 2) (thickness 0.3)))
   )
-  (gr_text Sp (at 156.21 83.82) (layer F.SilkS)
+  (gr_text SP (at 156.21 83.82) (layer F.SilkS)
     (effects (font (size 1 1) (thickness 0.15)))
   )
-  (gr_text Sp/Flt (at 157.48 86.36) (layer F.SilkS)
+  (gr_text SP/FLT (at 157.8102 86.3854) (layer F.SilkS)
     (effects (font (size 1 1) (thickness 0.15)))
   )
-  (gr_text Heart (at 157.48 88.9) (layer F.SilkS)
+  (gr_text HEART (at 157.4292 88.9254) (layer F.SilkS)
     (effects (font (size 1 1) (thickness 0.15)))
   )
-  (gr_text PWR (at 156.845 91.44) (layer F.SilkS)
+  (gr_text PWR (at 156.7434 91.3638) (layer F.SilkS)
     (effects (font (size 1 1) (thickness 0.15)))
   )
@@
   (segment (start -19.685 151.13) (end -19.665 151.13) (width 0.25) (layer F.Cu) (net 0))
   (segment (start 121.285 71.12) (end 120.65 71.12) (width 0.25) (layer B.Cu) (net 0))
+  (segment (start 126.0602 81.4324) (end 126.1618 81.4324) (width 0.25) (layer F.Cu) (net 0))
+  (via (at 126.2126 84.074) (size 0.6) (drill 0.4) (layers F.Cu B.Cu) (net 0))
+  (segment (start 126.2126 81.4324) (end 126.2126 84.074) (width 0.25) (layer B.Cu) (net 0))
+  (segment (start 126.1872 81.407) (end 126.2126 81.4324) (width 0.25) (layer B.Cu) (net 0))
+  (via (at 126.1872 81.407) (size 0.6) (drill 0.4) (layers F.Cu B.Cu) (net 0))
+  (segment (start 126.1618 81.4324) (end 126.1872 81.407) (width 0.25) (layer F.Cu) (net 0))
   (segment (start 125.095 89.535) (end 125.095 89.515) (width 0.25) (layer B.Cu) (net 1))
-  (segment (start 124.365 90.265) (end 125.095 89.535) (width 0.25) (layer F.Cu) (net 1))
-  (via (at 125.095 89.535) (size 0.6) (drill 0.4) (layers F.Cu B.Cu) (net 1))
-  (segment (start 124.365 91.52) (end 124.365 90.265) (width 0.25) (layer F.Cu) (net 1))
   (segment (start 125.095 89.515) (end 126.345 88.265) (width 0.25) (layer B.Cu) (net 1))
+  (segment (start 124.365 91.52) (end 124.365 90.265) (width 0.25) (layer F.Cu) (net 1))
+  (via (at 125.095 89.535) (size 0.6) (drill 0.4) (layers F.Cu B.Cu) (net 1))
+  (segment (start 124.365 90.265) (end 125.095 89.535) (width 0.25) (layer F.Cu) (net 1))
   (segment (start 129.54 74.295) (end 129.54 70.485) (width 0.25) (layer B.Cu) (net 1))
   (segment (start 129.165 74.67) (end 129.54 74.295) (width 0.25) (layer F.Cu) (net 1))
@@
       )
     )
+  )
+  (zone (net 0) (net_name "") (layer F.Mask) (hatch edge 0.508)
+    (connect_pads (clearance 6.35))
+    (min_thickness 0.254)
+    (fill yes (arc_segments 16) (thermal_gap 0.508) (thermal_bridge_width 0.508))
+    (polygon
+      (pts
+        (xy 205.74 125.73) (xy 199.39 125.73) (xy 199.39 119.38) (xy 205.74 119.38) (xy 205.74 125.73)
+      )
+    )
+  )
+  (zone (net 0) (net_name "") (layer F.Mask) (hatch edge 0.508)
+    (connect_pads (clearance 6.35))
+    (min_thickness 0.254)
+    (fill yes (arc_segments 16) (thermal_gap 0.508) (thermal_bridge_width 0.508))
+    (polygon
+      (pts
+        (xy 38.1 45.085) (xy 38.1 52.07) (xy 53.34 52.07) (xy 53.34 43.815) (xy 38.1 43.815)
+        (xy 38.1 45.085)
+      )
+    )
