File: Circuit_layout/_autosave-Circuit_layout.kicad_pcb (KiCad board)
At the start: 2 copper layers, 168 parts, among them CON1 AVR-JTAG-10, J1 Spare_Conns, J10 AIRs, J3 CAN, J4 Motor_Ctrl, J5 RJ12, P1 TSV, P2 HVPL, P3 IMD, P4 GLV, P5 Cockpit, P6 Pedals, P7 BrakeLight/RTDS, Q1 MMBF170, Q2 MMBF170, Q3 BSS84, SW1 TS5A3159-Q1, U1 LM7332, U10 MCP2551-I/SN, U11 TLP293, U12 TLP293, U13 PDQ10-D, U14 PDQ15-D, U15 TLP293, U16 LTC3638, U17 MCP6004, U18 PDQ10-Q24-S12-D, U19 ACPL-C870, U2 LM7810CT, U20 ACPL-C870, U21 MCP6001, U3 MCP6004, U4 MCP6004, U5 LM7332, U6 LM339, U7 AT90CAN128-A, U8 74ACT11030, U9 TLP293, Y1 10MHz

Commit message: working on top level schematic
Parts:
- removed C13, C27, C36, C39: 0.1u, Capacitors_SMD:C_0805_HandSoldering
- removed C20: 15p, Capacitors_SMD:C_0805_HandSoldering
- removed C21, C9: 6.8uF, Capacitors_SMD:C_0805_HandSoldering
- removed C48: 10uF, Capacitors_SMD:C_0805_HandSoldering
- removed J10: AIRs, custom_footprints:TerminalBlock_Pheonix_MPT-5.08mm_2pol
- removed J3: CAN, custom_footprints:TerminalBlock_Pheonix_MPT-5.08mm_2pol
- removed P4: GLV, custom_footprints:TerminalBlock_Pheonix_MPT-5.08mm_3pol
- removed P5: Cockpit, custom_footprints:TerminalBlock_Pheonix_MPT-5.08mm_6pol
- removed P6: Pedals, custom_footprints:mkds_1,5-8
- removed P7: BrakeLight/RTDS, custom_footprints:TerminalBlock_Pheonix_MPT-5.08mm_4pol
- removed R35, R85: 2k, Resistors_SMD:R_0805_HandSoldering
- removed R46, R48, R84: 1k, Resistors_SMD:R_0805_HandSoldering
- removed R86: 100, Resistors_SMD:R_0805_HandSoldering
- added +10V1: +10V, Measurement_Points:Measurement_Point_Round-SMD-Pad_Big, F.Cu at (74.3, 55.9)
- added +24V1: +24V, Measurement_Points:Measurement_Point_Round-SMD-Pad_Big, F.Cu at (197.5, 46.4)
- added +5DC/DC1: +5DC/DC, Measurement_Points:Measurement_Point_Round-SMD-Pad_Big, F.Cu at (196.8, 83.8)
- added +5HV1: +5HV, Measurement_Points:Measurement_Point_Round-SMD-Pad_Big, F.Cu at (92.7, 138.4)
- added ?: , custom_footprints:Symbol_HighVoltage_Type2_FSilk_VerySmall, F.Cu at (200.7, 141.0)
- added ?: , custom_footprints:Symbol_HighVoltage_Type2_BSilk_VerySmall, F.Cu at (201.3, 141.0)
- added APPS1_b1: APPS1_b, Measurement_Points:Measurement_Point_Round-SMD-Pad_Big, F.Cu at (45.7, 81.9)
- added APPS2_b1: APPS2_b, Measurement_Points:Measurement_Point_Round-SMD-Pad_Big, F.Cu at (45.7, 87.6)
- added DC/DC_GND1: +5DC/DC_GND, Measurement_Points:Measurement_Point_Square-SMD-Pad_Big, F.Cu at (199.4, 62.9)
- added G***: LOGO, custom_footprints:logo_lafayette_ece_24mmx9mm, F.Cu at (56.5, 35.6)
- added G***: LOGO, custom_footprints:ROHS, F.Cu at (193.7, 111.8)
- added GLV_GND1: GLV_GND, Measurement_Points:Measurement_Point_Square-SMD-Pad_Big, F.Cu at (40.6, 56.5)
- added HVPL_HV1: TEST_1P, Measurement_Points:Measurement_Point_Round-SMD-Pad_Big, F.Cu at (43.2, 144.1)
- added HVPL_LV1: HVPL_LV, Measurement_Points:Measurement_Point_Round-SMD-Pad_Big, F.Cu at (38.1, 117.5)
- added HV_GND1: HV_GND, Measurement_Points:Measurement_Point_Square-SMD-Pad_Big, F.Cu at (35.6, 144.1)
- added IMD_uC1: IMD_uC, Measurement_Points:Measurement_Point_Round-SMD-Pad_Big, F.Cu at (196.8, 91.4)
- added IO_GND1: I/O_Ground, Measurement_Points:Measurement_Point_Round-SMD-Pad_Big, F.Cu at (92.1, 151.8)
- added I_Meas1: I_Meas, Measurement_Points:Measurement_Point_Round-SMD-Pad_Big, F.Cu at (196.8, 99.7)
- added JP1: JUMPER3, Pin_Headers:Pin_Header_Straight_1x03_Pitch2.54mm, F.Cu at (63.5, 102.9)
- added L1: 100uH, Inductors:Inductor_Taiyo-Yuden_NR-80xx_HandSoldering, F.Cu at (116.8, 145.4)
- added R69: 250k, Resistors_SMD:R_0805_HandSoldering, F.Cu at (106.7, 153.0)
- added R70: 47k, Resistors_SMD:R_0805_HandSoldering, F.Cu at (106.7, 150.5)
- added R71: 330, Resistors_SMD:R_0805_HandSoldering, F.Cu at (142.9, 91.4)
- added R72: 330, Resistors_SMD:R_0805_HandSoldering, F.Cu at (142.9, 88.9)
- added R73: 330, Resistors_SMD:R_0805_HandSoldering, F.Cu at (142.9, 86.4)
- added R74: 330, Resistors_SMD:R_0805_HandSoldering, F.Cu at (142.9, 83.8)
- added R76: 750k, Resistors_SMD:R_0805_HandSoldering, F.Cu at (127.6, 141.6)
- added R77: 196k, Resistors_SMD:R_0805_HandSoldering, F.Cu at (127.6, 144.1)
- added REF**: Symbol_OSHW-Logo_SilkScreen, custom_footprints:Symbol_OSHW-Logo_SilkScreen, F.Cu at (193.7, 120.7)
- added SW2: TS5A3159-Q1, TO_SOT_Packages_SMD:SOT-23-6_Handsoldering, F.Cu at (55.9, 104.1)
- added SW3: JS202011CQN, custom_footprints:CK_DPDT_Switch, F.Cu at (110.5, 49.5)
- added Thrtl_HV1: Throttle_HV, Measurement_Points:Measurement_Point_Round-SMD-Pad_Big, F.Cu at (85.1, 138.4)
- added Thrtl_LPF1: Throttle_LPF, Measurement_Points:Measurement_Point_Round-SMD-Pad_Big, F.Cu at (100.3, 109.2)
- added Thrtl_LV1: Throttle_LV, Measurement_Points:Measurement_Point_Round-SMD-Pad_Big, F.Cu at (46.4, 117.5)
- added Thrtl_PL1: Throttle_PL, Measurement_Points:Measurement_Point_Round-SMD-Pad_Big, F.Cu at (111.1, 96.5)
- added Thrtl_uC1: Throttle_uC, Measurement_Points:Measurement_Point_Round-SMD-Pad_Big, F.Cu at (111.1, 92.1)
- added U22: TS372, Housings_SOIC:SOIC-8_3.9x4.9mm_Pitch1.27mm, F.Cu at (81.3, 90.2)
- added U23: TLP293, Housings_SSOP:SOP-4_4.4x2.8mm_Pitch1.27mm, F.Cu at (76.2, 67.3)
- added U24: TLP293, Housings_SSOP:SOP-4_4.4x2.8mm_Pitch1.27mm, F.Cu at (76.2, 62.2)
- added U25: Mounting_hole, Mounting_Holes:MountingHole_3.5mm_Pad, F.Cu at (35.6, 34.3)
- added U26: Mounting_hole, Mounting_Holes:MountingHole_3.5mm_Pad, F.Cu at (202.6, 34.3)
- added U27: TLP293, Housings_SSOP:SOP-4_4.4x2.8mm_Pitch1.27mm, F.Cu at (161.3, 75.6)
- added VAL: REF, custom_footprints:lafLogo, F.Cu at (202.6, 122.6)
- added V_Meas1: V_Measure, Measurement_Points:Measurement_Point_Round-SMD-Pad_Big, F.Cu at (168.9, 112.4)
- added V_Meas_GND1: V_Meas_GND, Measurement_Points:Measurement_Point_Square-SMD-Pad_Big, F.Cu at (196.2, 106.7)
- C2, C31, C7: moved to B.Cu
- C22: value DNP -> 0.1u
- C23: value 10uF -> 0.1u
- C24: value 15p -> 1uF; footprint Capacitors_SMD:C_0805_HandSoldering -> Capacitors_SMD:C_2220_HandSoldering
- C3: value 0.1u -> 2.2uF
- C8: value 1uF -> 0.1u; footprint Capacitors_SMD:C_2220_HandSoldering -> Capacitors_SMD:C_0805_HandSoldering; moved to B.Cu
- J1: footprint custom_footprints:mkds_1,5-8 -> custom_footprints:Molex_8x1_2.54mm
- J4: footprint custom_footprints:TerminalBlock_Pheonix_MPT-5.08mm_4pol -> custom_footprints:Molex_4x1_2.54mm
- P1: footprint custom_footprints:TerminalBlock_Pheonix_MPT-5.08mm_2pol -> custom_footprints:AMPCONN_2
- P2: value HVPL -> CONN_02X10; footprint custom_footprints:TerminalBlock_Pheonix_MPT-5.08mm_4pol -> Connect:IDC_Header_Straight_20pins
- P3: value IMD -> CONN_02X07; footprint custom_footprints:TerminalBlock_Pheonix_MPT-5.08mm_2pol -> Connect:IDC_Header_Straight_14pins
- Q1: value MMBF170 -> ZVP4525G; footprint TO_SOT_Packages_SMD:SOT-23 -> TO_SOT_Packages_SMD:SOT-223-3Lead_TabPin2
- Q3: value BSS84 -> MMBF170
- R1: value 1k -> 665k
- R13, R21, R22, R23, R28, R29, R3, R31, R4, R5, R6, R7: value 1k -> 10k
- R14: value 47k -> 10k
- R16: value 2k -> 250k
- R17: value 150 -> 10k
- R18: value 100 -> 10k
- R19, R20: value 100 -> 250k
- R2: value 1k -> 250k
- R24, R30: value 1k -> 100k
- R27: value 137k -> 150
- R39: value 750k -> 10k
- R42: value 196k -> 10k
- R51, R52: value 0 -> 250k
- R8: value 1M -> 10k
- R9: value 137k -> 665k
- SW1: value TS5A3159-Q1 -> SW_PUSH; footprint TO_SOT_Packages_SMD:SOT-23-6_Handsoldering -> custom_footprints:SW_RACON_8
- U1: value LM7332 -> PDM2-S24-S12; footprint Housings_SOIC:SOIC-8_3.9x4.9mm_Pitch1.27mm -> custom_footprints:DCDC-Conv_TRACO_TMR_1-xxxx_Single
- U14: value PDQ15-D -> Mounting_hole; footprint custom_footprints:PDQ_DCDC -> Mounting_Holes:MountingHole_3.5mm_Pad
- U15: value TLP293 -> Mounting_hole; footprint Housings_SSOP:SOP-4_4.4x2.8mm_Pitch1.27mm -> Mounting_Holes:MountingHole_3.5mm_Pad
- U18: value PDQ10-Q24-S12-D -> TS912; footprint custom_footprints:PDQ_DCDC -> Housings_SOIC:SOIC-8_3.9x4.9mm_Pitch1.27mm
- U2: value LM7810CT -> MCP6002; footprint TO_SOT_Packages_THT:TO-220_Vertical -> Housings_SOIC:SOIC-8_3.9x4.9mm_Pitch1.27mm
- U4: value MCP6004 -> LM95071-Q1; footprint Housings_SOIC:SOIC-14_3.9x8.7mm_Pitch1.27mm -> TO_SOT_Packages_SMD:SOT-23-5_HandSoldering
- U5: value LM7332 -> LM7810CT; footprint Housings_SOIC:SOIC-8_3.9x4.9mm_Pitch1.27mm -> custom_footprints:TO-220_Horizontal_Plated_Hole
- U6: value LM339 -> TS912; footprint Housings_SOIC:SOIC-14_3.9x8.7mm_Pitch1.27mm -> Housings_SOIC:SOIC-8_3.9x4.9mm_Pitch1.27mm
- Y1: footprint Crystals:Crystal_SMD_HC49-SD_HandSoldering -> custom_footprints:crystal_TXC_7A
- moved P2 210.6 mm to (38.1, 108.0), turned to 90 degrees
- moved J4 191.9 mm to (83.8, 144.8), turned to 180 degrees
- moved U14 188.5 mm to (202.6, 151.1)
- moved C34 185.4 mm to (62.2, 139.7), turned to 0 degrees
- moved C47 182.5 mm to (55.9, 147.3)
- moved U16 179.8 mm to (105.4, 144.1), turned to 180 degrees
- moved U21 179.7 mm to (62.2, 143.5), turned to 0 degrees
- moved D5 178.4 mm to (97.2, 144.1)
- moved R64 177.6 mm to (62.2, 149.9)
- moved R62 177.3 mm to (55.9, 142.2), turned to 180 degrees
- moved R63 177.0 mm to (55.9, 144.8)
- moved R66 176.5 mm to (62.2, 147.3), turned to 0 degrees
- moved C19 175.9 mm to (125.7, 146.7)
- moved C46 174.8 mm to (62.2, 137.2)
- moved R39 174.5 mm to (66.0, 83.8), turned to 270 degrees
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Connections:
- C1 pad 1: CH_GND -> +5V
- C1 pad 2: A1_LV -> CH_GND
- C15 pad 1: APPS1 -> /ThrottlePlausibility/APPS1_ISO
- C15 pad 2: CH_GND -> Net-(C15-Pad2)
- C16 pad 1: APPS2 -> Net-(C16-Pad1)
- C19 pad 2: /Status Lights/HV- -> HV-
- C2 pad 1: A2_LV -> +5V
- C22 pad 1: /Status Lights/BP_uC -> Net-(C22-Pad1)
- C23 pad 1: Net-(C19-Pad1) -> APPS1_10
- C23 pad 2: /Status Lights/HV- -> CH_GND
- C24 pad 1: Net-(C24-Pad1) -> HV+
- C24 pad 2: CH_GND -> HV-
- C3 pad 1: IMD_PWM -> HVPL
- C38 pad 1: +5V -> APPS1_10
- C8 pad 1: /Status Lights/HV+ -> +5V
- C8 pad 2: /Status Lights/HV- -> CH_GND
- D5 pad 2: /Status Lights/HV- -> HV-
- J5 pad 4: CH_GND -> I_RTN
- P2 pad 1: HVPL -> CANH
- P2 pad 3: CH_GND -> CANL
- P2 pad 4: CH_GND -> HVPL
- P3 pad 1: IMD_Status -> CH_GND
- P3 pad 2: IMD_PWM -> CC_LED
- Q1 pad 2: CH_GND -> IMD_Fault_LED
- Q1 pad 3: Brake_Light -> +24V
- Q3 pad 2: IMD_Fault_LED -> CH_GND
- Q3 pad 3: +12V -> I_RTN
- R10 pad 2: Net-(R10-Pad2) -> Net-(R1-Pad2)
- R11 pad 1: SDA -> SCL
- R13 pad 1: Net-(Q1-Pad1) -> +5V
- R13 pad 2: /Status Lights/BP_uC -> ~RESET_AVR
- R14 pad 1: Net-(R14-Pad1) -> Net-(Q3-Pad1)
- R14 pad 2: /Status Lights/HV- -> /I_ENB
- R16 pad 1: +24V -> Net-(R16-Pad1)
- R16 pad 2: Net-(R16-Pad2) -> HV+
- R17 pad 1: Brake_Light -> Net-(Q1-Pad1)
- R17 pad 2: +12V -> IMD_Status
- R18 pad 1: +5V -> CH_GND
- R18 pad 2: Net-(D1-Pad2) -> Net-(Q3-Pad1)
- R19 pad 1: /Status Lights/Spare_Red -> Net-(R19-Pad1)
- R19 pad 2: Net-(D3-Pad2) -> Net-(R16-Pad1)
- R2 pad 1: Net-(R2-Pad1) -> AIRs+
- R2 pad 2: A1_LV -> Net-(R2-Pad2)
- R20 pad 1: /Status Lights/Spare_Blue -> Net-(R20-Pad1)
- R20 pad 2: Net-(D4-Pad2) -> Net-(R19-Pad1)
- R21 pad 1: Net-(R21-Pad1) -> Net-(Q2-Pad1)
- R21 pad 2: APPS1 -> /ThrottlePlausibility/Throttle_PL
- R22 pad 1: Net-(R22-Pad1) -> /ThrottlePlausibility/APPS1_b
- R22 pad 2: +5V -> Net-(R22-Pad2)
- R23 pad 1: Net-(R21-Pad1) -> +5V
- R23 pad 2: CH_GND -> Net-(C15-Pad2)
- R24 pad 1: /ThrottlePlausibility/APPS1_ISO -> APPS2
- R24 pad 2: Net-(R22-Pad1) -> Net-(C16-Pad1)
- R27 pad 1: Net-(R10-Pad2) -> Net-(R27-Pad1)
- R27 pad 2: CH_GND -> /Status Lights/CC_LED_CTRL
- R28 pad 1: Net-(R28-Pad1) -> CH_GND
- R28 pad 2: APPS1 -> Net-(R22-Pad2)
- R29 pad 1: Net-(R29-Pad1) -> Net-(C15-Pad2)
- R29 pad 2: APPS2 -> /ThrottlePlausibility/APPS1_ISO
- R3 pad 2: A2_LV -> A1_LV
- R30 pad 1: Net-(R28-Pad1) -> APPS1
- R30 pad 2: CH_GND -> Net-(C22-Pad1)
- R31 pad 1: Net-(R31-Pad1) -> /ThrottlePlausibility/APPS1_b
- R31 pad 2: Net-(R29-Pad1) -> Net-(R31-Pad2)
- R39 pad 1: Net-(C19-Pad1) -> /ThrottlePlausibility/APPS2_b
- R4 pad 1: Net-(R2-Pad1) -> Net-(R4-Pad1)
- R4 pad 2: CH_GND -> A2_LV
- R40 pad 1: Net-(C20-Pad1) -> Net-(R40-Pad1)
- R41 pad 1: Net-(C24-Pad1) -> Net-(R41-Pad1)
- R42 pad 1: Net-(R39-Pad2) -> Net-(R31-Pad2)
- R42 pad 2: /Status Lights/HV- -> CH_GND
- R43 pad 1: SCL -> /ThrottlePlausibility/Throttle_SEL
- R43 pad 2: +5V -> CH_GND
- R5 pad 1: Net-(R5-Pad1) -> /ThrottlePlausibility/APPS2_b
- R5 pad 2: +5V -> Net-(Q2-Pad3)
- R50 pad 1: CH_GND -> Net-(R39-Pad2)
- R50 pad 2: BP -> Net-(R50-Pad2)
- R51 pad 2: /Status Lights/BP_uC -> Net-(R51-Pad2)
- R52 pad 1: CH_GND -> BOT
- R52 pad 2: CH_GND -> Net-(R52-Pad2)
- R55 pad 2: Net-(R55-Pad2) -> Net-(C29-Pad1)
- R56 pad 1: Net-(C29-Pad1) -> Net-(R56-Pad1)
- R56 pad 2: Net-(R55-Pad2) -> Net-(C29-Pad1)
- R6 pad 1: /I_Measure -> CH_GND
- R62 pad 1: Net-(C46-Pad1) -> Net-(R62-Pad1)
- R62 pad 2: Net-(R62-Pad2) -> Net-(C46-Pad1)
- R64 pad 2: Net-(R62-Pad2) -> Net-(C46-Pad1)
- R7 pad 1: Net-(R7-Pad1) -> /I_Measure
- R7 pad 2: AIRs+ -> Net-(R4-Pad1)
- R8 pad 1: /Status Lights/HV+ -> SDA
- R8 pad 2: Net-(R14-Pad1) -> +5V
- R9 pad 2: Net-(R5-Pad1) -> IMD_PWM
- SW1 pad 1: /ThrottlePlausibility/Pedal_Out -> ~RESET_AVR
- U1 pad 1: /ThrottlePlausibility/APPS1_ISO -> Net-(C19-Pad1)
- U1 pad 2: Net-(R22-Pad1) -> HV-
- U1 pad 6: (no net) -> HVPL
- U11 pad 4: Net-(R16-Pad2) -> +24V
- U12 pad 4: Net-(R35-Pad2) -> +24V
- U14 pad 1: +24V -> (no net)
- U15 pad 1: IMD_PWM -> (no net)
- U16 pad 12: /Status Lights/HV- -> HV-
- U16 pad 14: Net-(R14-Pad1) -> Net-(R69-Pad1)
- U16 pad 16: /Status Lights/HV- -> HV-
- U16 pad 17: /Status Lights/HV- -> HV-
- U16 pad 3: /Status Lights/HV+ -> HV+
- U16 pad 6: /Status Lights/HV- -> HV-
- U16 pad 8: /Status Lights/HV- -> HV-
- U16 pad 9: Net-(R39-Pad2) -> Net-(R76-Pad2)
- U17 pad 10: Net-(R55-Pad2) -> Net-(C29-Pad1)
- U17 pad 12: Net-(R79-Pad1) -> (no net)
- U17 pad 13: /ThrottlePlausibility/APPS1_ISO -> (no net)
- U17 pad 14: Net-(U17-Pad14) -> (no net)
- U17 pad 2: Net-(R3-Pad1) -> Net-(R4-Pad1)
- U17 pad 3: Net-(R2-Pad1) -> Net-(R3-Pad1)
- U17 pad 5: Net-(R10-Pad2) -> Net-(R1-Pad2)
- U18 pad 1: /Status Lights/HV- -> /ThrottlePlausibility/APPS1_ISO
- U18 pad 2: Net-(C19-Pad1) -> Net-(C15-Pad2)
- U18 pad 3: /Status Lights/HVPL -> Net-(R22-Pad2)
- U18 pad 4: Net-(U18-Pad4) -> CH_GND
- U18 pad 5: CH_GND -> Net-(R31-Pad2)
- U18 pad 6: (no net) -> Net-(R39-Pad2)
- U19 pad 7: Net-(C46-Pad1) -> Net-(R62-Pad1)
- U2 pad 1: +24V -> /ThrottlePlausibility/Pedal_Out
- U2 pad 2: CH_GND -> /ThrottlePlausibility/Pedal_Out
- U2 pad 3: APPS1_10 -> Net-(Q2-Pad3)
- U20 pad 7: Net-(C29-Pad1) -> Net-(R56-Pad1)
- U21 pad 3: Net-(R62-Pad2) -> Net-(C46-Pad1)
- U3 pad 10: APPS2 -> Net-(R38-Pad1)
- U3 pad 12: (no net) -> /ThrottlePlausibility/APPS2_b
- U3 pad 13: (no net) -> Net-(R38-Pad2)
- U3 pad 14: (no net) -> Net-(U3-Pad14)
- U3 pad 2: Net-(R80-Pad2) -> /ThrottlePlausibility/APPS1_ISO
- U3 pad 3: /ThrottlePlausibility/APPS1_ISO -> Net-(R79-Pad1)
- U3 pad 5: Net-(R38-Pad1) -> /ThrottlePlausibility/APPS1_ISO
- U3 pad 6: APPS2 -> Net-(R80-Pad2)
- U3 pad 9: Net-(R38-Pad2) -> /ThrottlePlausibility/APPS2_b
- U4 pad 1: Net-(C26-Pad1) -> /~SS
- U4 pad 2: Net-(C26-Pad2) -> CH_GND
- U4 pad 3: Net-(R47-Pad1) -> /MISO
- U4 pad 4: +5V -> /SCK
- U4 pad 5: (no net) -> +5V
- U5 pad 1: Net-(R31-Pad1) -> +24V
- U5 pad 2: Net-(R29-Pad1) -> CH_GND
- U5 pad 3: Net-(R28-Pad1) -> APPS1_10
- U6 pad 1: Net-(C24-Pad1) -> /ThrottlePlausibility/APPS1_b
- U6 pad 2: Net-(C20-Pad1) -> /ThrottlePlausibility/APPS1_b
- U6 pad 3: APPS1_10 -> Net-(C22-Pad1)
- U6 pad 4: Net-(R31-Pad1) -> CH_GND
- U6 pad 5: Net-(R32-Pad1) -> Net-(C16-Pad1)
- U6 pad 6: Net-(R33-Pad1) -> /ThrottlePlausibility/APPS2_b
- U6 pad 7: Net-(R31-Pad1) -> /ThrottlePlausibility/APPS2_b
- U6 pad 8: (no net) -> APPS1_10
- U7 pad 10: Net-(U7-Pad10) -> /~SS
- U7 pad 11: Net-(U7-Pad11) -> /SCK
- U7 pad 13: Net-(U7-Pad13) -> /MISO
- U7 pad 14: /Status Lights/BP_uC -> /ThrottlePlausibility/BP_uC
- U7 pad 44: Net-(U7-Pad44) -> /I_ENB
- U7 pad 49: Net-(U7-Pad49) -> /Status Lights/CC_LED_CTRL
- U7 pad 51: /Safety_Loop -> Net-(U7-Pad51)
- U7 pad 54: TDI -> /PIN54
- U7 pad 55: TDO -> /PIN55
- U7 pad 7: Net-(U7-Pad7) -> /Safety_Loop
- U7 pad 8: Net-(U7-Pad8) -> /ThrottlePlausibility/BOT_uC
- U8 pad 12: Net-(U3-Pad1) -> Net-(U3-Pad7)
- U8 pad 13: Net-(U3-Pad7) -> Net-(U3-Pad8)
- U8 pad 14: Net-(U3-Pad8) -> Net-(U3-Pad14)
- U8 pad 3: Net-(C20-Pad1) -> Net-(R40-Pad1)
- U8 pad 8: Net-(C24-Pad1) -> Net-(R41-Pad1)
- U8 pad 9: Net-(U17-Pad14) -> Net-(U3-Pad1)
- U9 pad 1: Net-(R7-Pad1) -> Net-(R2-Pad2)
Routing:
- net +24V: track 0.00 -> 315.4 mm, vias 0 -> 12
- net +5HV: track 0.00 -> 156.0 mm, vias 0 -> 1
- net Net-(C19-Pad1): track 0.00 -> 152.1 mm, vias 0 -> 5
- net SCL: track 0.00 -> 146.1 mm, vias 0 -> 4
- net APPS1_10: track 0.00 -> 141.3 mm, vias 0 -> 14
- net SDA: track 0.00 -> 137.4 mm, vias 0 -> 4
- net CH_GND: track 0.00 -> 128.9 mm, vias 0 -> 20
- net /IMD: track 0.00 -> 124.3 mm, vias 0 -> 8
- net CANH: track 0.00 -> 122.6 mm, vias 0 -> 4
- net I/O_Ground: track 0.00 -> 122.2 mm, vias 0 -> 10
- net CANL: track 0.00 -> 118.9 mm, vias 0 -> 4
- net /Isolators/V_Measure: track 0.00 -> 109.6 mm, vias 0 -> 11
- net /I_Measure: track 0.00 -> 106.7 mm, vias 0 -> 7
- net /ThrottlePlausibility/APPS2_b: track 0.00 -> 106.6 mm, vias 0 -> 10
- net HV+: track 0.00 -> 103.0 mm, vias 0 -> 2
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- added copper zone on B.Cu, net +5V
- added copper zone on F.Cu, net CH_GND
- added copper zone on F.Cu, net HV-
Other:
- board outline added: 177.8 x 127 mm
- net class Default: clearance 0.2 -> 0.2032
- net class TSV added: clearance 0.5, trace_width 0.5, via_dia 0.6, via_drill 0.4
- rule trace_clearance: 0.2 -> 0.2032
- board text added: "Designed by: Jack Plumb and Adam Ness"
- board text added: "HEART"
- board text added: "High Voltage"
- board text added: "L17_TSI_001"
- board text added: "Low Voltage"
- board text added: "Made in U.S.A."
- board text added: "PWR"
- board text added: "RESET"
- board text added: "REV 0"
- board text added: "SN"
- board text added: "SP"
- board text added: "SP/FLT"
- board text added: "Tractive System Interface"
